File: ice40_FPGA_Breakout/iCE40_FPGA_Module.sch (KiCad schematic (older format))
At the start: 101 parts

Commit message: global nets changed to hierarchy net, interconnects updated
Parts:
- added R?: 0, symbol R
- R?: value 10k -> 10K
- R?: value VAR -> 10K
Connections:
- net LVDS_13_D- is gone; now on net LVDS_D13-: R?.2
- net EXT_RESET: now also R?.1; no longer R?.1, TP?.1
- net LVDS_D13-: now reaches R?.2
- net 1V2_EXT_IN renamed 1V2_IN
- net 2V5_EXT_IN renamed 2V5_IN
- removed net 3V3_REF_IN: C?.1, C?.1, C?.1, C?.1, C?.1, C?.1, C?.1, C?.1, C?.1, C?.1, C?.1, C?.1, U?.A13 (VCCIO_0), U?.A3 (VCCIO_0), U?.A8 (VCCIO_0), U?.C15 (VCCIO_1), U?.E1 (VCCIO_3), U?.F8 (VCCIO_0), U?.G6 (VCCIO_3), U?.H10 (VCCIO_1), U?.H15 (VCCIO_1), U?.J6 (VCCIO_3), U?.K8 (VCCIO_2), U?.N1 (VCCIO_3), U?.N15 (VCCIO_1), U?.P3 (VCCIO_2), U?.R13 (VCCIO_2), U?.R8 (VCCIO_2)
- net FTDI_AD6_GPIO6 renamed FPGA_CDONE
- net LVDS_10_D+ renamed LVDS_D10+
- net LVDS_10_D- renamed LVDS_D10-
- net LVDS_11_D+ renamed LVDS_D11+
- net LVDS_11_D- renamed LVDS_D11-
- net LVDS_12_D+ renamed LVDS_D12+
- net LVDS_12_D- renamed LVDS_D12-
- net LVDS_13_D+ renamed LVDS_D13+
- net LVDS_14_D+ renamed LVDS_D14+
- net LVDS_14_D- renamed LVDS_D14-
- net LVDS_15_D+ renamed LVDS_D15+
- net LVDS_15_D- renamed LVDS_D15-
- net LVDS_16_D+ renamed LVDS_D16+
- net LVDS_16_D- renamed LVDS_D16-
- net LVDS_17_D+ renamed LVDS_D17+
- net LVDS_17_D- renamed LVDS_D17-
- net LVDS_18_D+ renamed LVDS_D18+
- net LVDS_18_D- renamed LVDS_D18-
- net LVDS_19_D+ renamed LVDS_D19+
- net LVDS_19_D- renamed LVDS_D19-
- net LVDS_1_D+ renamed LVDS_D1+
- net LVDS_1_D- renamed LVDS_D1-
- net LVDS_20_D+ renamed LVDS_D20+
- net LVDS_20_D- renamed LVDS_D20-
- net LVDS_2_D+ renamed LVDS_D2+
- net LVDS_2_D- renamed LVDS_D2-
- net LVDS_3_D+ renamed LVDS_D3+
- net LVDS_3_D- renamed LVDS_D3-
- net LVDS_4_D+ renamed LVDS_D4+
- net LVDS_4_D- renamed LVDS_D4-
- net LVDS_5_D+ renamed LVDS_D5+
- net LVDS_5_D- renamed LVDS_D5-
- net LVDS_6_D+ renamed LVDS_D6+
- net LVDS_6_D- renamed LVDS_D6-
- net LVDS_7_D+ renamed LVDS_D7+
- net LVDS_7_D- renamed LVDS_D7-
- net LVDS_8_D+ renamed LVDS_D8+
- net LVDS_8_D- renamed LVDS_D8-
- net LVDS_9_D+ renamed LVDS_D9+
- net LVDS_9_D- renamed LVDS_D9-
- net LVPECLK- renamed LVDSCLK-
- new net FPGA_CRST: R?.1, R?.2, TP?.1
- new net VCCIO_0_IN: C?.1, C?.1, C?.1, U?.A13 (VCCIO_0), U?.A3 (VCCIO_0), U?.A8 (VCCIO_0), U?.F8 (VCCIO_0)
- new net VCCIO_1_IN: C?.1, C?.1, C?.1, U?.C15 (VCCIO_1), U?.H10 (VCCIO_1), U?.H15 (VCCIO_1), U?.N15 (VCCIO_1)
- new net VCCIO_2_IN: C?.1, C?.1, C?.1, U?.K8 (VCCIO_2), U?.P3 (VCCIO_2), U?.R13 (VCCIO_2), U?.R8 (VCCIO_2)
- new net VCCIO_3_IN: C?.1, C?.1, C?.1, U?.E1 (VCCIO_3), U?.G6 (VCCIO_3), U?.J6 (VCCIO_3), U?.N1 (VCCIO_3)

Commit message: post review fix
Connections:
- net 1V2_REF_IN is gone; now on net 1V2_IN: R?.2, R?.2
- net 3V3_EXT_IN is gone; now on net 3V3_IN: R?.2, R?.2
- net LVDS_D3+: now also R?.2
- net VCCIO_0_IN renamed VCCIO_0_REFIN
- net VCCIO_1_IN renamed VCCIO_1_REFIN
- net VCCIO_2_IN renamed VCCIO_2_REFIN
- net VCCIO_3_IN renamed VCCIO_3_REFIN
Other:
- note added: "Differential Pair"
