File: ice40_FPGA_Breakout/_saved_USB_FTDI.sch (KiCad schematic (older format))
At the start: 52 parts, among them J1 USB_B_Micro, J2 3pos_Jumper, J3 3pos_Jumper, U5 93LCxxC, U6 FT2232H, Y1 ABM10AIG-12.000MHZ-4Z-T3

Commit message: Component Annotated and R/C/Conn/TP CVPCB mapping
Parts:
- C22, C23, C25, C26, C28, C30, C31, C33, C34, C35, C36, C37, C38, C39, C40: footprint (none) -> Capacitor_SMD:C_0402_1005Metric
- C24, C27, C29, C32: footprint (none) -> Capacitor_SMD:C_0603_1608Metric
- D4, D5: footprint (none) -> LED_SMD:LED_0402_1005Metric
- R110, R111, R112, R113, R114, R115, R116, R117, R118, R119, R120, R121, R122, R123, R124, R125, R126: footprint (none) -> Resistor_SMD:R_0402_1005Metric
- TP11: footprint (none) -> Conn_PinHeader_2.00mm:PinHeader_1x01_P2.00mm_Vertical
Changed lines of the file:
@@
 F 0 "C22" V 2100 1600 50  0000 L CNN
 F 1 "0.1uF" V 2200 1600 50  0000 L CNN
-F 2 "" H 2288 1350 50  0001 C CNN
+F 2 "Capacitor_SMD:C_0402_1005Metric" H 2288 1350 50  0001 C CNN
 F 3 "" H 2250 1500 50  0001 C CNN
 	1    2250 1500
@@
 F 0 "C23" H 3175 4900 50  0000 L CNN
 F 1 "0.1uF" H 3175 4700 50  0000 L CNN
-F 2 "" H 3188 4650 50  0001 C CNN
+F 2 "Capacitor_SMD:C_0402_1005Metric" H 3188 4650 50  0001 C CNN
 F 3 "" H 3150 4800 50  0001 C CNN
 	1    3150 4800
@@
 F 0 "C37" H 8700 1150 50  0000 L CNN
 F 1 "0.1uF" H 8600 1350 50  0000 L CNN
-F 2 "" H 8888 1100 50  0001 C CNN
+F 2 "Capacitor_SMD:C_0402_1005Metric" H 8888 1100 50  0001 C CNN
 F 3 "" H 8850 1250 50  0001 C CNN
 	1    8850 1250
@@
 F 0 "C39" H 9475 1350 50  0000 L CNN
 F 1 "0.1uF" H 9475 1150 50  0000 L CNN
-F 2 "" H 9488 1100 50  0001 C CNN
+F 2 "Capacitor_SMD:C_0402_1005Metric" H 9488 1100 50  0001 C CNN
 F 3 "" H 9450 1250 50  0001 C CNN
 	1    9450 1250
@@
 F 0 "C36" H 8575 1350 50  0000 L CNN
 F 1 "0.1uF" H 8575 1150 50  0000 L CNN
-F 2 "" H 8588 1100 50  0001 C CNN
+F 2 "Capacitor_SMD:C_0402_1005Metric" H 8588 1100 50  0001 C CNN
 F 3 "" H 8550 1250 50  0001 C CNN
 	1    8550 1250
@@
 F 0 "C40" H 9775 1350 50  0000 L CNN
 F 1 "0.1uF" H 9775 1150 50  0000 L CNN
-F 2 "" H 9788 1100 50  0001 C CNN
+F 2 "Capacitor_SMD:C_0402_1005Metric" H 9788 1100 50  0001 C CNN
 F 3 "" H 9750 1250 50  0001 C CNN
 	1    9750 1250
@@
 F 0 "C35" H 8275 1350 50  0000 L CNN
 F 1 "0.1uF" H 8275 1150 50  0000 L CNN
-F 2 "" H 8288 1100 50  0001 C CNN
+F 2 "Capacitor_SMD:C_0402_1005Metric" H 8288 1100 50  0001 C CNN
 F 3 "" H 8250 1250 50  0001 C CNN
 	1    8250 1250
@@
 F 0 "C34" H 7975 1350 50  0000 L CNN
 F 1 "0.1uF" H 7975 1150 50  0000 L CNN
-F 2 "" H 7988 1100 50  0001 C CNN
+F 2 "Capacitor_SMD:C_0402_1005Metric" H 7988 1100 50  0001 C CNN
 F 3 "" H 7950 1250 50  0001 C CNN
 	1    7950 1250
@@
 F 0 "C27" H 5575 1300 50  0000 L CNN
 F 1 "4.7uf" H 5575 1100 50  0000 L CNN
-F 2 "" H 5588 1050 50  0001 C CNN
+F 2 "Capacitor_SMD:C_0603_1608Metric" H 5588 1050 50  0001 C CNN
 F 3 "" H 5550 1200 50  0001 C CNN
 	1    5550 1200
@@
 F 0 "C30" H 5875 1300 50  0000 L CNN
 F 1 "0.1uF" H 5875 1100 50  0000 L CNN
-F 2 "" H 5888 1050 50  0001 C CNN
+F 2 "Capacitor_SMD:C_0402_1005Metric" H 5888 1050 50  0001 C CNN
 F 3 "" H 5850 1200 50  0001 C CNN
 	1    5850 1200
@@
 F 0 "C32" H 6175 1300 50  0000 L CNN
 F 1 "4.7uF" H 6175 1100 50  0000 L CNN
-F 2 "" H 6188 1050 50  0001 C CNN
+F 2 "Capacitor_SMD:C_0603_1608Metric" H 6188 1050 50  0001 C CNN
 F 3 "" H 6150 1200 50  0001 C CNN
 	1    6150 1200
@@
 F 0 "C33" H 6475 1300 50  0000 L CNN
 F 1 "0.1uF" H 6475 1100 50  0000 L CNN
-F 2 "" H 6488 1050 50  0001 C CNN
+F 2 "Capacitor_SMD:C_0402_1005Metric" H 6488 1050 50  0001 C CNN
 F 3 "" H 6450 1200 50  0001 C CNN
 	1    6450 1200
@@
 F 0 "C38" H 9175 1350 50  0000 L CNN
 F 1 "0.1uF" H 9175 1150 50  0000 L CNN
-F 2 "" H 9188 1100 50  0001 C CNN
+F 2 "Capacitor_SMD:C_0402_1005Metric" H 9188 1100 50  0001 C CNN
 F 3 "" H 9150 1250 50  0001 C CNN
 	1    9150 1250
@@
 F 0 "C25" H 5525 2400 50  0000 L CNN
 F 1 "0.1uF" H 5525 2200 50  0000 L CNN
-F 2 "" H 5538 2150 50  0001 C CNN
+F 2 "Capacitor_SMD:C_0402_1005Metric" H 5538 2150 50  0001 C CNN
 F 3 "" H 5500 2300 50  0001 C CNN
 	1    5500 2300
@@
 F 0 "C29" H 5775 2400 50  0000 L CNN
 F 1 "3.3uF" H 5775 2200 50  0000 L CNN
-F 2 "" H 5788 2150 50  0001 C CNN
+F 2 "Capacitor_SMD:C_0603_1608Metric" H 5788 2150 50  0001 C CNN
 F 3 "" H 5750 2300 50  0001 C CNN
 	1    5750 2300
@@
 F 0 "C26" H 5400 5950 50  0000 L CNN
 F 1 "10pF" H 5300 5750 50  0000 L CNN
-F 2 "" H 5538 5700 50  0001 C CNN
+F 2 "Capacitor_SMD:C_0402_1005Metric" H 5538 5700 50  0001 C CNN
 F 3 "" H 5500 5850 50  0001 C CNN
 	1    5500 5850
@@
 F 0 "C24" H 4975 5950 50  0000 L CNN
 F 1 "10pF" H 4975 5750 50  0000 L CNN
-F 2 "" H 4988 5700 50  0001 C CNN
+F 2 "Capacitor_SMD:C_0603_1608Metric" H 4988 5700 50  0001 C CNN
 F 3 "" H 4950 5850 50  0001 C CNN
 	1    4950 5850
@@
 F 0 "R111" V 4080 3850 50  0000 C CNN
 F 1 "10K" V 4000 3850 50  0000 C CNN
-F 2 "" V 3930 3850 50  0001 C CNN
+F 2 "Resistor_SMD:R_0402_1005Metric" V 3930 3850 50  0001 C CNN
 F 3 "" H 4000 3850 50  0001 C CNN
 	1    4000 3850
@@
 F 0 "R110" V 3880 3850 50  0000 C CNN
 F 1 "10K" V 3800 3850 50  0000 C CNN
-F 2 "" V 3730 3850 50  0001 C CNN
+F 2 "Resistor_SMD:R_0402_1005Metric" V 3730 3850 50  0001 C CNN
 F 3 "" H 3800 3850 50  0001 C CNN
 	1    3800 3850
@@
 F 0 "R112" V 4280 3850 50  0000 C CNN
 F 1 "10K" V 4200 3850 50  0000 C CNN
-F 2 "" V 4130 3850 50  0001 C CNN
+F 2 "Resistor_SMD:R_0402_1005Metric" V 4130 3850 50  0001 C CNN
 F 3 "" H 4200 3850 50  0001 C CNN
 	1    4200 3850
@@
 F 0 "R113" V 4580 4650 50  0000 C CNN
 F 1 "2.2K" V 4500 4650 50  0000 C CNN
-F 2 "" V 4430 4650 50  0001 C CNN
+F 2 "Resistor_SMD:R_0402_1005Metric" V 4430 4650 50  0001 C CNN
 F 3 "" H 4500 4650 50  0001 C CNN
 	1    4500 4650
@@
 F 0 "R114" V 4950 2700 50  0000 C CNN
 F 1 "0" V 5050 2750 50  0000 C CNN
-F 2 "" V 4980 2750 50  0001 C CNN
+F 2 "Resistor_SMD:R_0402_1005Metric" V 4980 2750 50  0001 C CNN
 F 3 "" H 5050 2750 50  0001 C CNN
 	1    5050 2750
@@
 F 0 "R115" V 5150 2800 50  0000 C CNN
 F 1 "0" V 5050 2850 50  0000 C CNN
-F 2 "" V 4980 2850 50  0001 C CNN
+F 2 "Resistor_SMD:R_0402_1005Metric" V 4980 2850 50  0001 C CNN
 F 3 "" H 5050 2850 50  0001 C CNN
 	1    5050 2850
@@
 F 0 "R117" V 5930 3600 50  0000 C CNN
 F 1 "12K" V 5850 3600 50  0000 C CNN
-F 2 "" V 5780 3600 50  0001 C CNN
+F 2 "Resistor_SMD:R_0402_1005Metric" V 5780 3600 50  0001 C CNN
 F 3 "" H 5850 3600 50  0001 C CNN
 	1    5850 3600
@@
 F 0 "R116" V 5380 3350 50  0000 C CNN
 F 1 "1K" V 5300 3350 50  0000 C CNN
-F 2 "" V 5230 3350 50  0001 C CNN
+F 2 "Resistor_SMD:R_0402_1005Metric" V 5230 3350 50  0001 C CNN
 F 3 "" H 5300 3350 50  0001 C CNN
 	1    5300 3350
@@
 F 0 "C28" H 5575 3700 50  0000 L CNN
 F 1 "0.1uF" H 5575 3500 50  0000 L CNN
-F 2 "" H 5588 3450 50  0001 C CNN
+F 2 "Capacitor_SMD:C_0402_1005Metric" H 5588 3450 50  0001 C CNN
 F 3 "" H 5550 3600 50  0001 C CNN
 	1    5550 3600
@@
 F 0 "R118" V 8750 1700 50  0000 C CNN
 F 1 "0" V 8800 1850 50  0000 C CNN
-F 2 "" V 8730 1850 50  0001 C CNN
+F 2 "Resistor_SMD:R_0402_1005Metric" V 8730 1850 50  0001 C CNN
 F 3 "" H 8800 1850 50  0001 C CNN
 	1    8800 1850
@@
 F 0 "R119" V 8750 1800 50  0000 C CNN
 F 1 "0" V 8800 1950 50  0000 C CNN
-F 2 "" V 8730 1950 50  0001 C CNN
+F 2 "Resistor_SMD:R_0402_1005Metric" V 8730 1950 50  0001 C CNN
 F 3 "" H 8800 1950 50  0001 C CNN
 	1    8800 1950
@@
 F 0 "R120" V 8750 1900 50  0000 C CNN
 F 1 "0" V 8800 2050 50  0000 C CNN
-F 2 "" V 8730 2050 50  0001 C CNN
+F 2 "Resistor_SMD:R_0402_1005Metric" V 8730 2050 50  0001 C CNN
 F 3 "" H 8800 2050 50  0001 C CNN
 	1    8800 2050
@@
 F 0 "R121" V 8750 2000 50  0000 C CNN
 F 1 "0" V 8800 2150 50  0000 C CNN
-F 2 "" V 8730 2150 50  0001 C CNN
+F 2 "Resistor_SMD:R_0402_1005Metric" V 8730 2150 50  0001 C CNN
 F 3 "" H 8800 2150 50  0001 C CNN
 	1    8800 2150
@@
 F 0 "R123" V 8750 2300 50  0000 C CNN
 F 1 "0" V 8800 2450 50  0000 C CNN
-F 2 "" V 8730 2450 50  0001 C CNN
+F 2 "Resistor_SMD:R_0402_1005Metric" V 8730 2450 50  0001 C CNN
 F 3 "" H 8800 2450 50  0001 C CNN
 	1    8800 2450
@@
 F 0 "R124" V 8750 2400 50  0000 C CNN
 F 1 "0" V 8800 2550 50  0000 C CNN
-F 2 "" V 8730 2550 50  0001 C CNN
+F 2 "Resistor_SMD:R_0402_1005Metric" V 8730 2550 50  0001 C CNN
 F 3 "" H 8800 2550 50  0001 C CNN
 	1    8800 2550
@@
 F 0 "C31" H 6025 2400 50  0000 L CNN
 F 1 "0.1uF" H 6025 2200 50  0000 L CNN
-F 2 "" H 6038 2150 50  0001 C CNN
+F 2 "Capacitor_SMD:C_0402_1005Metric" H 6038 2150 50  0001 C CNN
 F 3 "" H 6000 2300 50  0001 C CNN
 	1    6000 2300
@@
 F 0 "R122" V 8750 2100 50  0000 C CNN
 F 1 "DNP" V 8800 2250 50  0000 C CNN
-F 2 "" V 8730 2250 50  0001 C CNN
+F 2 "Resistor_SMD:R_0402_1005Metric" V 8730 2250 50  0001 C CNN
 F 3 "" H 8800 2250 50  0001 C CNN
 	1    8800 2250
@@
 F 0 "R125" V 9500 4700 50  0000 C CNN
 F 1 "330" V 9550 4850 50  0000 C CNN
-F 2 "" V 9480 4850 50  0001 C CNN
+F 2 "Resistor_SMD:R_0402_1005Metric" V 9480 4850 50  0001 C CNN
 F 3 "" H 9550 4850 50  0001 C CNN
 	1    9550 4850
@@
 F 0 "R126" V 9500 4800 50  0000 C CNN
 F 1 "330" V 9550 4950 50  0000 C CNN
-F 2 "" V 9480 4950 50  0001 C CNN
+F 2 "Resistor_SMD:R_0402_1005Metric" V 9480 4950 50  0001 C CNN
 F 3 "" H 9550 4950 50  0001 C CNN
 	1    9550 4950
@@
 F 0 "D4" H 9000 4900 50  0000 C CNN
 F 1 "LED" H 8800 4850 50  0000 C CNN
-F 2 "" H 9000 4800 50  0001 C CNN
+F 2 "LED_SMD:LED_0402_1005Metric" H 9000 4800 50  0001 C CNN
 F 3 "" H 9000 4800 50  0001 C CNN
 	1    9000 4800
@@
 F 0 "D5" H 9000 5100 50  0000 C CNN
 F 1 "LED" H 8800 5050 50  0000 C CNN
-F 2 "" H 9000 5000 50  0001 C CNN
+F 2 "LED_SMD:LED_0402_1005Metric" H 9000 5000 50  0001 C CNN
 F 3 "" H 9000 5000 50  0001 C CNN
 	1    9000 5000
@@
 F 0 "TP11" H 2000 1620 50  0000 C CNN
 F 1 "Test_Point" H 2000 1550 50  0000 C CNN
-F 2 "" H 2200 1350 50  0001 C CNN
+F 2 "Conn_PinHeader_2.00mm:PinHeader_1x01_P2.00mm_Vertical" H 2200 1350 50  0001 C CNN
 F 3 "" H 2200 1350 50  0001 C CNN
 	1    2000 1350
