File: ice40_FPGA_Breakout/_saved_iCE40_FPGA_Module.sch (KiCad schematic (older format))
At the start: 100 parts, among them U1 iCE40HX8_CT256

Commit message: Component Annotated and R/C/Conn/TP CVPCB mapping
Parts:
- C1, C10, C11, C12, C13, C14, C15, C16, C17, C4, C5: footprint (none) -> Capacitor_SMD:C_0402_1005Metric
- C2, C3, C6, C7, C8, C9: footprint (none) -> Capacitor_SMD:C_0603_1608Metric
- R13, R14, R15, R16, R17, R18, R19, R20, R21, R22, R23, R24, R25, R26, R27, R28, R29, R30, R31, R32, R33, R34, R35, R36, R37, R38, R39, R40, R41, R42, R43, R44, R45, R46, R47, R48, R49, R50, R51, R52, R53, R54, R55, R56, R57, R58, R59, R66, R67, R68, R69, R70, R71, R72, R73, R74, R75, R76, R77, R78, R79, R80, R81, R82, R83, R84, R85, R86: footprint (none) -> Resistor_SMD:R_0402_1005Metric
- R60, R61, R62, R63, R64, R65: footprint (none) -> Resistor_SMD:R_0603_1608Metric
