File: ice40_FPGA_Breakout/_saved_iCE40_FPGA_Module.sch (KiCad schematic (older format))
At the start: 108 parts, among them U1 iCE40HX8_CT256

Commit message: grouping complete ready to route
Parts:
- gave numbers to parts that had none: 4
Changed lines of the file:
@@
 $EndComp
 $Comp
-L GND #PWR044
+L GND #PWR45
 U 1 1 5A263712
 P 4800 4150
-F 0 "#PWR044" H 4800 3900 50  0001 C CNN
+F 0 "#PWR45" H 4800 3900 50  0001 C CNN
 F 1 "GND" H 4800 4000 50  0000 C CNN
 F 2 "" H 4800 4150 50  0001 C CNN
@@
 $EndComp
 $Comp
-L GND #PWR045
+L GND #PWR48
 U 1 1 5A3E2FC7
 P 7450 6300
-F 0 "#PWR045" H 7450 6050 50  0001 C CNN
+F 0 "#PWR48" H 7450 6050 50  0001 C CNN
 F 1 "GND" H 7450 6150 50  0000 C CNN
 F 2 "" H 7450 6300 50  0001 C CNN
@@
 $EndComp
 $Comp
-L GND #PWR046
+L GND #PWR47
 U 1 1 5A3E512A
 P 7400 5400
-F 0 "#PWR046" H 7400 5150 50  0001 C CNN
+F 0 "#PWR47" H 7400 5150 50  0001 C CNN
 F 1 "GND" H 7400 5250 50  0000 C CNN
 F 2 "" H 7400 5400 50  0001 C CNN
@@
 $EndComp
 $Comp
-L GND #PWR047
+L GND #PWR52
 U 1 1 5A407417
 P 11075 6175
-F 0 "#PWR047" H 11075 5925 50  0001 C CNN
+F 0 "#PWR52" H 11075 5925 50  0001 C CNN
 F 1 "GND" H 11175 6175 50  0000 C CNN
 F 2 "" H 11075 6175 50  0001 C CNN
@@
 $EndComp
 $Comp
-L GND #PWR048
+L GND #PWR50
 U 1 1 5A40791C
 P 11075 5075
-F 0 "#PWR048" H 11075 4825 50  0001 C CNN
+F 0 "#PWR50" H 11075 4825 50  0001 C CNN
 F 1 "GND" H 11175 5075 50  0000 C CNN
 F 2 "" H 11075 5075 50  0001 C CNN
@@
 $EndComp
 $Comp
-L GND #PWR049
+L GND #PWR49
 U 1 1 5A407BD5
 P 11075 4475
-F 0 "#PWR049" H 11075 4225 50  0001 C CNN
+F 0 "#PWR49" H 11075 4225 50  0001 C CNN
 F 1 "GND" H 11175 4475 50  0000 C CNN
 F 2 "" H 11075 4475 50  0001 C CNN
@@
 $EndComp
 $Comp
-L GND #PWR050
+L GND #PWR51
 U 1 1 5A407D06
 P 11075 5625
-F 0 "#PWR050" H 11075 5375 50  0001 C CNN
+F 0 "#PWR51" H 11075 5375 50  0001 C CNN
 F 1 "GND" H 11175 5625 50  0000 C CNN
 F 2 "" H 11075 5625 50  0001 C CNN
@@
 	5150 7050 5150 7100
 $Comp
-L GND #PWR051
+L GND #PWR46
 U 1 1 5A2D5A99
 P 5150 7100
-F 0 "#PWR051" H 5150 6850 50  0001 C CNN
+F 0 "#PWR46" H 5150 6850 50  0001 C CNN
 F 1 "GND" H 5150 6950 50  0000 C CNN
 F 2 "" H 5150 7100 50  0001 C CNN
@@
 VCCIO_0_REFIN
 $Comp
-L GND #PWR052
+L GND #PWR44
 U 1 1 5A39D4DE
 P 2150 1000
-F 0 "#PWR052" H 2150 750 50  0001 C CNN
+F 0 "#PWR44" H 2150 750 50  0001 C CNN
 F 1 "GND" H 2150 850 50  0000 C CNN
 F 2 "" H 2150 1000 50  0001 C CNN
@@
 D4+
 $Comp
-L C C?
+L C C80
 U 1 1 5AF811E0
 P 10800 5975
-F 0 "C?" H 10825 6075 50  0000 L CNN
+F 0 "C80" H 10825 6075 50  0000 L CNN
 F 1 "0.01uF" H 10825 5875 50  0000 L CNN
 F 2 "Capacitor_SMD:C_0402_1005Metric" H 10838 5825 50  0001 C CNN
@@
 $EndComp
 $Comp
-L C C?
+L C C79
 U 1 1 5AF81632
 P 10775 5425
-F 0 "C?" H 10800 5525 50  0000 L CNN
+F 0 "C79" H 10800 5525 50  0000 L CNN
 F 1 "0.01uF" H 10800 5325 50  0000 L CNN
 F 2 "Capacitor_SMD:C_0402_1005Metric" H 10813 5275 50  0001 C CNN
@@
 $EndComp
 $Comp
-L C C?
+L C C78
 U 1 1 5AF817AA
 P 10775 4875
-F 0 "C?" H 10800 4975 50  0000 L CNN
+F 0 "C78" H 10800 4975 50  0000 L CNN
 F 1 "0.01uF" H 10800 4775 50  0000 L CNN
 F 2 "Capacitor_SMD:C_0402_1005Metric" H 10813 4725 50  0001 C CNN
@@
 $EndComp
 $Comp
-L C C?
+L C C77
 U 1 1 5AF81B3C
 P 10775 4275
-F 0 "C?" H 10800 4375 50  0000 L CNN
+F 0 "C77" H 10800 4375 50  0000 L CNN
 F 1 "0.01uF" H 10800 4175 50  0000 L CNN
 F 2 "Capacitor_SMD:C_0402_1005Metric" H 10813 4125 50  0001 C CNN
