File: ice40_FPGA_Breakout/_autosave-ice40-hx8K_breakout_brd.kicad_pcb (KiCad board)
At the start: 2 copper layers, 281 parts, among them J1 USB_B_Micro, J2 3pos_Jumper, J3 3pos_Jumper, J4 4POS_JUMPER, J5 4POS_JUMPER, J6 4POS_JUMPER, J7 4POS_JUMPER, J8 4POS_JUMPER, J9 SO-DIMM, U1 iCE40HX8_CT256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

Commit message: ftdi component placement
Parts:
- moved J9 211.4 mm to (214.2, 118.7)
- moved U1 129.3 mm to (78.8, 165.5)
- moved R37 112.3 mm to (67.1, 160.9)
- moved R33 109.1 mm to (67.1, 157.8)
- moved R36 106.3 mm to (67.1, 159.9)
- moved R34 100.7 mm to (68.9, 163.3)
- moved R32 95.6 mm to (68.9, 162.3)
- moved R35 88.6 mm to (67.1, 158.8)
Changed lines of the file:
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@@
   )
   (module Resistor_SMD:R_0402_1005Metric (layer F.Cu)
-    (at 47.427381 69.18)
+    (at 68.8875 162.3)
     (descr "Resistor SMD 0402 (1005 Metric), square (rectangular) end terminal, IPC_7351 nominal, (Body size source: http://www.tortai-tech.com/upload/download/2011102023233369053.pdf), generated with kicad-footprint-generator")
     (tags resistor)
@@
   )
   (module Resistor_SMD:R_0402_1005Metric (layer F.Cu)
-    (at 67.657381 48.68)
+    (at 67.0875 157.775)
     (descr "Resistor SMD 0402 (1005 Metric), square (rectangular) end terminal, IPC_7351 nominal, (Body size source: http://www.tortai-tech.com/upload/download/2011102023233369053.pdf), generated with kicad-footprint-generator")
     (tags resistor)
@@
   )
   (module Resistor_SMD:R_0402_1005Metric (layer F.Cu)
-    (at 51.967381 64.13)
+    (at 68.8875 163.35)
     (descr "Resistor SMD 0402 (1005 Metric), square (rectangular) end terminal, IPC_7351 nominal, (Body size source: http://www.tortai-tech.com/upload/download/2011102023233369053.pdf), generated with kicad-footprint-generator")
     (tags resistor)
@@
   )
   (module Resistor_SMD:R_0402_1005Metric (layer F.Cu)
-    (at 40.647381 74.23)
+    (at 67.0875 158.825)
     (descr "Resistor SMD 0402 (1005 Metric), square (rectangular) end terminal, IPC_7351 nominal, (Body size source: http://www.tortai-tech.com/upload/download/2011102023233369053.pdf), generated with kicad-footprint-generator")
     (tags resistor)
@@
   )
   (module Resistor_SMD:R_0402_1005Metric (layer F.Cu)
-    (at 60.827381 53.73)
+    (at 67.0875 159.875)
     (descr "Resistor SMD 0402 (1005 Metric), square (rectangular) end terminal, IPC_7351 nominal, (Body size source: http://www.tortai-tech.com/upload/download/2011102023233369053.pdf), generated with kicad-footprint-generator")
     (tags resistor)
@@
   )
   (module Resistor_SMD:R_0402_1005Metric (layer F.Cu)
-    (at 64.357381 48.68)
+    (at 67.0875 160.925)
     (descr "Resistor SMD 0402 (1005 Metric), square (rectangular) end terminal, IPC_7351 nominal, (Body size source: http://www.tortai-tech.com/upload/download/2011102023233369053.pdf), generated with kicad-footprint-generator")
     (tags resistor)
@@
   )
   (module GTI_Footprint_Lib:SO_DIMM_200 (layer F.Cu)
-    (at 36.830001 3.8)
+    (at 214.225 118.7)
     (fp_text reference J9 (at -9.6 -2.4) (layer F.SilkS)
       (effects (font (size 1 1) (thickness 0.15)))
@@
   )
   (module GTI_Footprint_Lib:BGA-256_12mmx12mm_Layout_14mmx14mm_P0.8mm_R0.5mm (layer F.Cu)
-    (at 10.575001 55.73)
+    (at 78.8 165.525)
     (fp_text reference U1 (at 0 -12) (layer F.SilkS)
       (effects (font (size 1 1) (thickness 0.15)))
