File: ice40_FPGA_Breakout/Parallel_SRAM.sch (KiCad schematic (older format))
At the start: 13 parts, among them U3 M25P20, U4 IDT71V016SA

Commit message: schematic clean up, label aligned
Parts:
- C21: footprint (none) -> Capacitor_SMD:C_0402_1005Metric
- R100, R101, R102, R103, R104, R105, R106, R107, R108, R109: footprint (none) -> Resistor_SMD:R_0402_1005Metric
Changed lines of the file:
@@
 U 1 1 5A55CAEB
 P 8150 3550
-F 0 "R109" V 8230 3550 50  0000 C CNN
+F 0 "R109" V 8050 3550 50  0000 C CNN
 F 1 "10K" V 8150 3550 50  0000 C CNN
-F 2 "" V 8080 3550 50  0001 C CNN
+F 2 "Resistor_SMD:R_0402_1005Metric" V 8080 3550 50  0001 C CNN
 F 3 "" H 8150 3550 50  0001 C CNN
 	1    8150 3550
@@
 U 1 1 5A55CB26
 P 7250 2650
-F 0 "R105" V 7330 2650 50  0000 C CNN
+F 0 "R105" V 7200 2850 50  0000 C CNN
 F 1 "10K" V 7250 2650 50  0000 C CNN
-F 2 "" V 7180 2650 50  0001 C CNN
+F 2 "Resistor_SMD:R_0402_1005Metric" V 7180 2650 50  0001 C CNN
 F 3 "" H 7250 2650 50  0001 C CNN
 	1    7250 2650
@@
 U 1 1 5A55CB43
 P 7400 2650
-F 0 "R106" V 7480 2650 50  0000 C CNN
+F 0 "R106" V 7350 2850 50  0000 C CNN
 F 1 "10K" V 7400 2650 50  0000 C CNN
-F 2 "" V 7330 2650 50  0001 C CNN
+F 2 "Resistor_SMD:R_0402_1005Metric" V 7330 2650 50  0001 C CNN
 F 3 "" H 7400 2650 50  0001 C CNN
 	1    7400 2650
@@
 U 1 1 5A55CB63
 P 7550 2650
-F 0 "R107" V 7630 2650 50  0000 C CNN
+F 0 "R107" V 7500 2850 50  0000 C CNN
 F 1 "10K" V 7550 2650 50  0000 C CNN
-F 2 "" V 7480 2650 50  0001 C CNN
+F 2 "Resistor_SMD:R_0402_1005Metric" V 7480 2650 50  0001 C CNN
 F 3 "" H 7550 2650 50  0001 C CNN
 	1    7550 2650
@@
 U 1 1 5A55CB8C
 P 7700 2650
-F 0 "R108" V 7780 2650 50  0000 C CNN
+F 0 "R108" V 7650 2850 50  0000 C CNN
 F 1 "10K" V 7700 2650 50  0000 C CNN
-F 2 "" V 7630 2650 50  0001 C CNN
+F 2 "Resistor_SMD:R_0402_1005Metric" V 7630 2650 50  0001 C CNN
 F 3 "" H 7700 2650 50  0001 C CNN
 	1    7700 2650
 	1    0    0    -1
 $EndComp
-Text HLabel 7250 2300 1    60   Input ~ 0
+Text HLabel 7250 2150 1    60   Input ~ 0
 +3V3
 Text HLabel 10100 1100 2    60   Input ~ 0
@@
 U 1 1 5A55FF49
 P 3450 1100
-F 0 "R101" V 3530 1100 50  0000 C CNN
+F 0 "R101" V 3400 900 50  0000 C CNN
 F 1 "10K" V 3450 1100 50  0000 C CNN
-F 2 "" V 3380 1100 50  0001 C CNN
+F 2 "Resistor_SMD:R_0402_1005Metric" V 3380 1100 50  0001 C CNN
 F 3 "" H 3450 1100 50  0001 C CNN
 	1    3450 1100
@@
 	8350 1200 8450 1200
 Wire Wire Line
-	8350 950  8350 1200
+	8350 950  8350 1100
+Wire Wire Line
+	8350 1100 8350 1200
 Wire Wire Line
 	8450 1100 8350 1100
@@
 	8450 3400 8350 3400
 Wire Wire Line
-	8350 3400 8350 3800
+	8350 3400 8350 3500
+Wire Wire Line
+	8350 3500 8350 3750
+Wire Wire Line
+	8350 3750 8350 3800
 Wire Wire Line
 	8450 3500 8350 3500
 Connection ~ 8350 3500
 Wire Wire Line
-	7000 2900 8450 2900
-Wire Wire Line
-	7000 3000 8450 3000
-Wire Wire Line
-	7000 3100 8450 3100
-Wire Wire Line
-	7000 3200 8450 3200
-Wire Wire Line
-	7000 3300 8450 3300
+	7000 2900 8150 2900
+Wire Wire Line
+	8150 2900 8450 2900
+Wire Wire Line
+	7000 3000 7700 3000
+Wire Wire Line
+	7700 3000 8450 3000
+Wire Wire Line
+	7000 3100 7550 3100
+Wire Wire Line
+	7550 3100 8450 3100
+Wire Wire Line
+	7000 3200 7400 3200
+Wire Wire Line
+	7400 3200 8450 3200
+Wire Wire Line
+	7000 3300 7250 3300
+Wire Wire Line
+	7250 3300 8450 3300
 Wire Wire Line
 	8150 3400 8150 2900
@@
 Connection ~ 8350 3750
 Wire Wire Line
-	7700 2400 7700 2500
-Wire Wire Line
-	7250 2400 7700 2400
-Wire Wire Line
-	7250 2300 7250 2500
-Connection ~ 7250 2400
-Wire Wire Line
-	7400 2500 7400 2400
-Connection ~ 7400 2400
-Wire Wire Line
-	7550 2500 7550 2400
-Connection ~ 7550 2400
+	7700 2250 7700 2500
+Wire Wire Line
+	7250 2250 7400 2250
+Wire Wire Line
+	7400 2250 7550 2250
+Wire Wire Line
+	7550 2250 7700 2250
+Wire Wire Line
+	7250 2150 7250 2250
+Wire Wire Line
+	7250 2250 7250 2500
+Connection ~ 7250 2250
+Wire Wire Line
+	7400 2500 7400 2250
+Connection ~ 7400 2250
+Wire Wire Line
+	7550 2500 7550 2250
+Connection ~ 7550 2250
 Wire Wire Line
 	9900 1100 10100 1100
@@
 	9900 2600 10100 2600
 Wire Wire Line
-	4200 2100 4550 2100
+	4200 2100 4400 2100
+Wire Wire Line
+	4400 2100 4550 2100
 Wire Wire Line
 	4400 2100 4400 1250
 Wire Wire Line
-	3000 1100 3000 2200
-Wire Wire Line
-	2600 2200 3200 2200
+	3000 1100 3000 1250
+Wire Wire Line
+	3000 1250 3000 1450
+Wire Wire Line
+	3000 1450 3000 2200
+Wire Wire Line
+	2600 2200 3000 2200
+Wire Wire Line
+	3000 2200 3200 2200
 Wire Wire Line
 	3200 2300 3050 2300
 Wire Wire Line
-	3050 2300 3050 2800
+	3050 2300 3050 2650
+Wire Wire Line
+	3050 2650 3050 2750
+Wire Wire Line
+	3050 2750 3050 2800
 Wire Wire Line
 	4300 2000 4200 2000
 Wire Wire Line
-	2600 2000 3200 2000
+	2600 2000 2900 2000
+Wire Wire Line
+	2900 2000 3150 2000
+Wire Wire Line
+	3150 2000 3200 2000
 Wire Wire Line
 	3200 2100 2600 2100
 Wire Wire Line
-	4200 2200 4550 2200
+	4200 2200 4250 2200
+Wire Wire Line
+	4250 2200 4550 2200
 Wire Wire Line
 	4200 2300 4550 2300
 Wire Wire Line
-	3600 1100 4400 1100
+	3600 1100 3750 1100
+Wire Wire Line
+	3750 1100 4300 1100
+Wire Wire Line
+	4300 1100 4400 1100
 Wire Wire Line
 	4400 1250 3000 1250
@@
 	4300 1100 4300 2000
 Wire Wire Line
-	2850 1100 3300 1100
+	2850 1100 3000 1100
+Wire Wire Line
+	3000 1100 3300 1100
 Connection ~ 3000 1250
 Connection ~ 4300 1100
@@
 F 0 "R100" V 2980 2400 50  0000 C CNN
 F 1 "10K" V 2900 2400 50  0000 C CNN
-F 2 "" V 2830 2400 50  0001 C CNN
+F 2 "Resistor_SMD:R_0402_1005Metric" V 2830 2400 50  0001 C CNN
 F 3 "" H 2900 2400 50  0001 C CNN
 	1    2900 2400
@@
 F 0 "R104" V 4330 2550 50  0000 C CNN
 F 1 "10K" V 4250 2550 50  0000 C CNN
-F 2 "" V 4180 2550 50  0001 C CNN
+F 2 "Resistor_SMD:R_0402_1005Metric" V 4180 2550 50  0001 C CNN
 F 3 "" H 4250 2550 50  0001 C CNN
 	1    4250 2550
@@
 F 0 "C21" H 2725 1200 50  0000 L CNN
 F 1 "0.1uF" H 2725 1000 50  0000 L CNN
-F 2 "" H 2738 950 50  0001 C CNN
+F 2 "Capacitor_SMD:C_0402_1005Metric" H 2738 950 50  0001 C CNN
 F 3 "" H 2700 1100 50  0001 C CNN
 	1    2700 1100
@@
 U 1 1 5A6077BD
 P 3450 1450
-F 0 "R102" V 3530 1450 50  0000 C CNN
+F 0 "R102" V 3400 1250 50  0000 C CNN
 F 1 "10K" V 3450 1450 50  0000 C CNN
-F 2 "" V 3380 1450 50  0001 C CNN
+F 2 "Resistor_SMD:R_0402_1005Metric" V 3380 1450 50  0001 C CNN
 F 3 "" H 3450 1450 50  0001 C CNN
 	1    3450 1450
@@
 U 1 1 5A60780F
 P 3450 1600
-F 0 "R103" V 3530 1600 50  0000 C CNN
+F 0 "R103" V 3400 1400 50  0000 C CNN
 F 1 "10K" V 3450 1600 50  0000 C CNN
-F 2 "" V 3380 1600 50  0001 C CNN
+F 2 "Resistor_SMD:R_0402_1005Metric" V 3380 1600 50  0001 C CNN
 F 3 "" H 3450 1600 50  0001 C CNN
 	1    3450 1600
@@
 	3600 1450 3750 1450
 Wire Wire Line
-	3750 1100 3750 1600
+	3750 1100 3750 1450
+Wire Wire Line
+	3750 1450 3750 1600
 Connection ~ 3750 1100
 Wire Wire Line

Commit message: assigned footprint to each component
Parts:
- U3: footprint (none) -> Package_SO:SOIC-8_3.9x4.9mm_P1.27mm
- U4: footprint (none) -> GTI_Footprint_Lib:44pin_400mil_TSOP_TypeII_SO44-2
Changed lines of the file:
@@
 F 0 "U4" H 8700 950 60  0000 C CNN
 F 1 "IDT71V016SA" H 9100 800 60  0000 C CNN
-F 2 "" H 9150 900 60  0001 C CNN
+F 2 "GTI_Footprint_Lib:44pin_400mil_TSOP_TypeII_SO44-2" H 9150 900 60  0001 C CNN
 F 3 "" H 9150 900 60  0001 C CNN
 	1    9150 900
@@
 F 0 "U3" H 3450 1900 60  0000 C CNN
 F 1 "M25P20" H 3700 1800 60  0000 C CNN
-F 2 "" H 3700 1900 60  0001 C CNN
+F 2 "Package_SO:SOIC-8_3.9x4.9mm_P1.27mm" H 3700 1900 60  0001 C CNN
 F 3 "" H 3700 1900 60  0001 C CNN
 	1    3700 1850
@@
 	8350 1200 8450 1200
 Wire Wire Line
-	8350 950  8350 1100
-Wire Wire Line
-	8350 1100 8350 1200
+	8350 950  8350 1200
 Wire Wire Line
 	8450 1100 8350 1100
@@
 	8450 3400 8350 3400
 Wire Wire Line
-	8350 3400 8350 3500
-Wire Wire Line
-	8350 3500 8350 3750
-Wire Wire Line
-	8350 3750 8350 3800
+	8350 3400 8350 3800
 Wire Wire Line
 	8450 3500 8350 3500
 Connection ~ 8350 3500
 Wire Wire Line
-	7000 2900 8150 2900
-Wire Wire Line
-	8150 2900 8450 2900
-Wire Wire Line
-	7000 3000 7700 3000
-Wire Wire Line
-	7700 3000 8450 3000
-Wire Wire Line
-	7000 3100 7550 3100
-Wire Wire Line
-	7550 3100 8450 3100
-Wire Wire Line
-	7000 3200 7400 3200
-Wire Wire Line
-	7400 3200 8450 3200
-Wire Wire Line
-	7000 3300 7250 3300
-Wire Wire Line
-	7250 3300 8450 3300
+	7000 2900 8450 2900
+Wire Wire Line
+	7000 3000 8450 3000
+Wire Wire Line
+	7000 3100 8450 3100
+Wire Wire Line
+	7000 3200 8450 3200
+Wire Wire Line
+	7000 3300 8450 3300
 Wire Wire Line
 	8150 3400 8150 2900
@@
 	7700 2250 7700 2500
 Wire Wire Line
-	7250 2250 7400 2250
-Wire Wire Line
-	7400 2250 7550 2250
-Wire Wire Line
-	7550 2250 7700 2250
-Wire Wire Line
-	7250 2150 7250 2250
-Wire Wire Line
-	7250 2250 7250 2500
+	7250 2250 7700 2250
+Wire Wire Line
+	7250 2150 7250 2500
 Connection ~ 7250 2250
 Wire Wire Line
@@
 	9900 2600 10100 2600
 Wire Wire Line
-	4200 2100 4400 2100
-Wire Wire Line
-	4400 2100 4550 2100
+	4200 2100 4550 2100
 Wire Wire Line
 	4400 2100 4400 1250
 Wire Wire Line
-	3000 1100 3000 1250
-Wire Wire Line
-	3000 1250 3000 1450
-Wire Wire Line
-	3000 1450 3000 2200
-Wire Wire Line
-	2600 2200 3000 2200
-Wire Wire Line
-	3000 2200 3200 2200
+	3000 1100 3000 2200
+Wire Wire Line
+	2600 2200 3200 2200
 Wire Wire Line
 	3200 2300 3050 2300
 Wire Wire Line
-	3050 2300 3050 2650
-Wire Wire Line
-	3050 2650 3050 2750
-Wire Wire Line
-	3050 2750 3050 2800
+	3050 2300 3050 2800
 Wire Wire Line
 	4300 2000 4200 2000
 Wire Wire Line
-	2600 2000 2900 2000
-Wire Wire Line
-	2900 2000 3150 2000
-Wire Wire Line
-	3150 2000 3200 2000
+	2600 2000 3200 2000
 Wire Wire Line
 	3200 2100 2600 2100
 Wire Wire Line
-	4200 2200 4250 2200
-Wire Wire Line
-	4250 2200 4550 2200
+	4200 2200 4550 2200
 Wire Wire Line
 	4200 2300 4550 2300
 Wire Wire Line
-	3600 1100 3750 1100
-Wire Wire Line
-	3750 1100 4300 1100
-Wire Wire Line
-	4300 1100 4400 1100
+	3600 1100 4400 1100
 Wire Wire Line
 	4400 1250 3000 1250
@@
 	4300 1100 4300 2000
 Wire Wire Line
-	2850 1100 3000 1100
-Wire Wire Line
-	3000 1100 3300 1100
+	2850 1100 3300 1100
 Connection ~ 3000 1250
 Connection ~ 4300 1100
@@
 	3600 1450 3750 1450
 Wire Wire Line
-	3750 1100 3750 1450
-Wire Wire Line
-	3750 1450 3750 1600
+	3750 1100 3750 1600
 Connection ~ 3750 1100
 Wire Wire Line

Commit message: , diff pair, memory and power component grouping
Parts:
- added C75, C76: 0.1uF, Capacitor_SMD:C_0402_1005Metric, symbol C
- added R155: 10K, Resistor_SMD:R_0402_1005Metric, symbol R
- R103: value 10K -> DNP
Connections:
- net +3V3: now also C21.1, C75.1, C76.1, R155.2
- net FLASH_~HOLD: now also R155.1; no longer C21.1, R101.2, R102.2, U3.3 (~WP)
- net GND: now also C75.2, C76.2
- new net FLASH_~WP: R101.2, R102.2, U3.3 (~WP)
Other:
- moved on the sheet: C21, R101
