File: ice40_FPGA_Breakout/SO-DIMM_200_Connector.sch (KiCad schematic (older format))
At the start: 21 parts, among them J9 SO-DIMM

Commit message: update differential pair connection in schematic and updating layout placement for diff pair
Connections:
- net DP1+: now also J9.9 (DATA_MOSI_1_LVDS+)
- net DP10+: now also J9.71 (DATA_MISO_5_LVDS-)
- net DP10-: now also J9.69 (DATA_MISO_5_LVDS+)
- net DP11+: now also J9.77 (DATA_MOSI_6_LVDS-)
- net DP11-: now also J9.75 (DATA_MOSI_6_LVDS+)
- net DP12+: now also J9.83 (DATA_MISO_6_LVDS-)
- net DP12-: now also J9.81 (DATA_MISO_6_LVDS+)
- net DP13+: now also J9.89 (DATA_MOSI_7_LVDS-)
- net DP13-: now also J9.87 (DATA_MOSI_7_LVDS+)
- net DP14+: now also J9.95 (DATA_MISO_7_LVDS-)
- net DP14-: now also J9.93 (DATA_MISO_7_LVDS+)
- net DP15+: now also J9.101 (DATA_MOSI_8_LVDS-)
- net DP15-: now also J9.99 (DATA_MOSI_8_LVDS+)
- net DP16+: now also J9.107 (DATA_MISO_8_LVDS-)
- net DP16-: now also J9.105 (DATA_MISO_8_LVDS+)
- net DP2+: now also J9.15 (DATA_MISO_1_LVD+)
- net DP2-: now also J9.17 (DATA_MISO_1_LVDS-)
- net DP3+: now also J9.21 (DATA_MOSI_2_LVDS+)
- net DP3-: now also J9.23 (DATA_MOSI_2_LVDS-)
- net DP4+: now also J9.27 (DATA_MISO_2_LVDS+)
- net DP4-: now also J9.29 (DATA_MISO_2_LVDS-)
- net DP5+: now also J9.33 (DATA_MOSI_3_LVDS+)
- net DP5-: now also J9.35 (DATA_MOSI_3_LVDS-)
- net DP6+: now also J9.47 (DATA_MISO_3_LVDS-)
- net DP6-: now also J9.45 (DATA_MISO_3_LVDS+)
- net DP7+: now also J9.53 (DATA_MOSI_4_LVDS-)
- net DP7-: now also J9.51 (DATA_MOSI_4_LVDS+)
- net DP8+: now also J9.59 (DATA_MISO_4_LVDS-)
- net DP8-: now also J9.57 (DATA_MISO_4_LVDS+)
- net DP9+: now also J9.65 (DATA_MOSI_5_LVDS-)
- net DP9-: now also J9.63 (DATA_MOSI_5_LVDS+)
Changed lines of the file:
@@
 $Descr A4 11693 8268
 encoding utf-8
-Sheet 7 7
+Sheet 6 7
 Title ""
 Date ""
@@
 2V5_EXT_IN
 $Comp
-L GND #PWR47
+L GND #PWR038
 U 1 1 5A41B6AD
 P 2850 5800
-F 0 "#PWR47" H 2850 5550 50  0001 C CNN
+F 0 "#PWR038" H 2850 5550 50  0001 C CNN
 F 1 "GND" H 2950 5800 50  0000 C CNN
 F 2 "" H 2850 5800 50  0001 C CNN
@@
 $EndComp
 $Comp
-L GND #PWR48
+L GND #PWR039
 U 1 1 5A41B7D9
 P 2850 6350
-F 0 "#PWR48" H 2850 6100 50  0001 C CNN
+F 0 "#PWR039" H 2850 6100 50  0001 C CNN
 F 1 "GND" H 2950 6350 50  0000 C CNN
 F 2 "" H 2850 6350 50  0001 C CNN
@@
 $EndComp
 $Comp
-L GND #PWR50
+L GND #PWR040
 U 1 1 5A41B927
 P 2850 7500
-F 0 "#PWR50" H 2850 7250 50  0001 C CNN
+F 0 "#PWR040" H 2850 7250 50  0001 C CNN
 F 1 "GND" H 2950 7500 50  0000 C CNN
 F 2 "" H 2850 7500 50  0001 C CNN
@@
 $EndComp
 $Comp
-L GND #PWR49
+L GND #PWR041
 U 1 1 5A41B976
 P 2850 6900
-F 0 "#PWR49" H 2850 6650 50  0001 C CNN
+F 0 "#PWR041" H 2850 6650 50  0001 C CNN
 F 1 "GND" H 2950 6900 50  0000 C CNN
 F 2 "" H 2850 6900 50  0001 C CNN
@@
 $EndComp
 $Comp
-L GND #PWR51
+L GND #PWR042
 U 1 1 5A41CA24
 P 11050 4500
-F 0 "#PWR51" H 11050 4250 50  0001 C CNN
+F 0 "#PWR042" H 11050 4250 50  0001 C CNN
 F 1 "GND" H 11050 4350 50  0000 C CNN
 F 2 "" H 11050 4500 50  0001 C CNN
@@
 Connection ~ 10950 1500
 $Comp
-L GND #PWR52
+L GND #PWR043
 U 1 1 5A421824
 P 11100 1550
-F 0 "#PWR52" H 11100 1300 50  0001 C CNN
+F 0 "#PWR043" H 11100 1300 50  0001 C CNN
 F 1 "GND" H 11100 1400 50  0000 C CNN
 F 2 "" H 11100 1550 50  0001 C CNN
@@
 Text GLabel 800  1350 1    39   Input ~ 0
 3V3_EXT_IN
-Text HLabel 7050 5800 3    39   Input ~ 0
+Text HLabel 10450 1275 1    39   Input ~ 0
 DP1-
-Text HLabel 7100 5800 3    39   Input ~ 0
+Text HLabel 10550 1275 1    39   Input ~ 0
 DP1+
-Text HLabel 7250 5800 3    39   Input ~ 0
+Text HLabel 10150 1275 1    39   Input ~ 0
 DP2-
-Text HLabel 7450 5800 3    39   Input ~ 0
+Text HLabel 9850 1275 1    39   Input ~ 0
 DP3-
-Text HLabel 7650 5800 3    39   Input ~ 0
+Text HLabel 9550 1275 1    39   Input ~ 0
 DP4-
-Text HLabel 7850 5800 3    39   Input ~ 0
+Text HLabel 9250 1275 1    39   Input ~ 0
 DP5-
-Text HLabel 8050 5800 3    39   Input ~ 0
+Text HLabel 8500 1225 1    39   Input ~ 0
 DP6-
-Text HLabel 8250 5800 3    39   Input ~ 0
+Text HLabel 8200 1225 1    39   Input ~ 0
 DP7-
-Text HLabel 8450 5800 3    39   Input ~ 0
+Text HLabel 7900 1225 1    39   Input ~ 0
 DP8-
-Text HLabel 8650 5800 3    39   Input ~ 0
+Text HLabel 7600 1225 1    39   Input ~ 0
 DP9-
-Text HLabel 8850 5800 3    39   Input ~ 0
+Text HLabel 7300 1225 1    39   Input ~ 0
 DP10-
-Text HLabel 9050 5800 3    39   Input ~ 0
+Text HLabel 7000 1225 1    39   Input ~ 0
 DP11-
-Text HLabel 9250 5800 3    39   Input ~ 0
+Text HLabel 6700 1225 1    39   Input ~ 0
 DP12-
-Text HLabel 9450 5800 3    39   Input ~ 0
+Text HLabel 6400 1225 1    39   Input ~ 0
 DP13-
-Text HLabel 9650 5800 3    39   Input ~ 0
+Text HLabel 6100 1225 1    39   Input ~ 0
 DP14-
-Text HLabel 9850 5800 3    39   Input ~ 0
+Text HLabel 5800 1225 1    39   Input ~ 0
 DP15-
-Text HLabel 10050 5800 3    39   Input ~ 0
+Text HLabel 5500 1225 1    39   Input ~ 0
 DP16-
-Text HLabel 10250 5800 3    39   Input ~ 0
-DP17-
-Text HLabel 10450 5800 3    39   Input ~ 0
-DP18-
-Text HLabel 10650 5800 3    39   Input ~ 0
-DP19-
-Text HLabel 10850 5800 3    39   Input ~ 0
-DP20-
-Text HLabel 7300 5800 3    39   Input ~ 0
+Text HLabel 10250 1275 1    39   Input ~ 0
 DP2+
-Text HLabel 7500 5800 3    39   Input ~ 0
+Text HLabel 9950 1275 1    39   Input ~ 0
 DP3+
-Text HLabel 7700 5800 3    39   Input ~ 0
+Text HLabel 9650 1275 1    39   Input ~ 0
 DP4+
-Text HLabel 7900 5800 3    39   Input ~ 0
+Text HLabel 9350 1275 1    39   Input ~ 0
 DP5+
-Text HLabel 8100 5800 3    39   Input ~ 0
+Text HLabel 8400 1225 1    39   Input ~ 0
 DP6+
-Text HLabel 8300 5800 3    39   Input ~ 0
+Text HLabel 8100 1225 1    39   Input ~ 0
 DP7+
-Text HLabel 8500 5800 3    39   Input ~ 0
+Text HLabel 7800 1225 1    39   Input ~ 0
 DP8+
-Text HLabel 8700 5800 3    39   Input ~ 0
+Text HLabel 7500 1225 1    39   Input ~ 0
 DP9+
-Text HLabel 8900 5800 3    39   Input ~ 0
+Text HLabel 7200 1225 1    39   Input ~ 0
 DP10+
-Text HLabel 9100 5800 3    39   Input ~ 0
+Text HLabel 6900 1225 1    39   Input ~ 0
 DP11+
-Text HLabel 9300 5800 3    39   Input ~ 0
+Text HLabel 6600 1225 1    39   Input ~ 0
 DP12+
-Text HLabel 9500 5800 3    39   Input ~ 0
+Text HLabel 6300 1225 1    39   Input ~ 0
 DP13+
-Text HLabel 9700 5800 3    39   Input ~ 0
+Text HLabel 6000 1225 1    39   Input ~ 0
 DP14+
-Text HLabel 9900 5800 3    39   Input ~ 0
+Text HLabel 5700 1225 1    39   Input ~ 0
 DP15+
-Text HLabel 10100 5800 3    39   Input ~ 0
+Text HLabel 5400 1225 1    39   Input ~ 0
 DP16+
-Text HLabel 10300 5800 3    39   Input ~ 0
-DP17+
-Text HLabel 10500 5800 3    39   Input ~ 0
-DP18+
-Text HLabel 10700 5800 3    39   Input ~ 0
-DP19+
-Text HLabel 10900 5800 3    39   Input ~ 0
-DP20+
 Text HLabel 6450 5850 3    39   Input ~ 0
 ET_SPI_MISO
@@
 Text HLabel 6850 5850 3    39   Input ~ 0
 EXT_RESET
+Wire Wire Line
+	10550 1700 10550 1275
+Wire Wire Line
+	10450 1675 10450 1275
+Wire Wire Line
+	10250 1700 10250 1275
+Wire Wire Line
+	10150 1700 10150 1275
+Wire Wire Line
+	9950 1700 9950 1275
+Wire Wire Line
+	9850 1275 9850 1700
+Wire Wire Line
+	9650 1700 9650 1275
+Wire Wire Line
+	9550 1700 9550 1275
+Wire Wire Line
+	9350 1700 9350 1275
+Wire Wire Line
+	9250 1700 9250 1275
+Wire Wire Line
+	8500 1700 8500 1225
+Wire Wire Line
+	8400 1700 8400 1225
+Wire Wire Line
+	8200 1700 8200 1225
+Wire Wire Line
+	8100 1700 8100 1225
+Wire Wire Line
+	7900 1700 7900 1225
+Wire Wire Line
+	7800 1700 7800 1225
+Wire Wire Line
+	7600 1225 7600 1700
+Wire Wire Line
+	7500 1700 7500 1225
+Wire Wire Line
+	7300 1700 7300 1225
+Wire Wire Line
+	7200 1700 7200 1225
+Wire Wire Line
+	7000 1700 7000 1225
+Wire Wire Line
+	6900 1700 6900 1225
+Wire Wire Line
+	6700 1700 6700 1225
+Wire Wire Line
+	6600 1700 6600 1225
+Wire Wire Line
+	6400 1700 6400 1225
+Wire Wire Line
+	6300 1700 6300 1225
+Wire Wire Line
+	6100 1700 6100 1225
+Wire Wire Line
+	6000 1700 6000 1225
+Wire Wire Line
+	5800 1700 5800 1225
+Wire Wire Line
+	5700 1700 5700 1225
+Wire Wire Line
+	5500 1700 5500 1225
+Wire Wire Line
+	5400 1700 5400 1225
 $EndSCHEMATC

Commit message: Regrouping con't
Parts:
- added TP17, TP18, TP19, TP20, TP21, TP22, TP23, TP24, TP25, TP26, TP27, TP28, TP29, TP30, TP31, TP32, TP33, TP34, TP35, TP36, TP37, TP38, TP39, TP40, TP41, TP42, TP43, TP44, TP45, TP46, TP47, TP48, TP49, TP50: Test_Point, TestPoint:TestPoint_THTPad_D1.0mm_Drill0.5mm, symbol Test_Point
Connections:
- net DP1+: now also TP49.1
- net DP1-: now also TP48.1
- net DP10+: now also TP30.1
- net DP10-: now also TP31.1
- net DP11+: now also TP28.1
- net DP11-: now also TP29.1
- net DP12+: now also TP26.1
- net DP12-: now also TP27.1
- net DP13+: now also TP24.1
- net DP13-: now also TP25.1
- net DP14+: now also TP22.1
- net DP14-: now also TP23.1
- net DP15+: now also TP20.1
- net DP15-: now also TP21.1
- net DP16+: now also TP18.1
- net DP16-: now also TP19.1
- net DP2+: now also TP47.1
- net DP2-: now also TP46.1
- net DP3+: now also TP45.1
- net DP3-: now also TP44.1
- net DP4+: now also TP43.1
- net DP4-: now also TP42.1
- net DP5+: now also TP41.1
- net DP5-: now also TP40.1
- net DP6+: now also TP38.1
- net DP6-: now also TP39.1
- net DP7+: now also TP36.1
- net DP7-: now also TP37.1
- net DP8+: now also TP34.1
- net DP8-: now also TP35.1
- net DP9+: now also TP32.1
- net DP9-: now also TP33.1
- net LVPECLK+: now also TP17.1
- net LVPECLK-: now also TP50.1

Commit message: grouping complete ready to route
Parts:
- TP17, TP18, TP19, TP20, TP21, TP22, TP23, TP24, TP25, TP26, TP27, TP28, TP29, TP30, TP31, TP32, TP33, TP34, TP35, TP36, TP37, TP38, TP39, TP40, TP41, TP42, TP43, TP44, TP45, TP46, TP47, TP48, TP49, TP50: footprint TestPoint:TestPoint_THTPad_D1.0mm_Drill0.5mm -> TestPoint:TestPoint_Pad_D1.0mm
