File: ice40_FPGA_Breakout/SRAM_16bit.sch (KiCad schematic (older format))
At the start: 22 parts, among them U1 iCE40HX8_CT256, U2 AT25SF041-SSHD-T

Commit message: update differential pair connection in schematic and updating layout placement for diff pair
Parts:
- U1: footprint (none) -> GTI_Footprint_Lib:BGA-256_12mmx12mm_Layout_14mmx14mm_P0.8mm_R0.5mm
Changed lines of the file:
@@
 $Descr A4 11693 8268
 encoding utf-8
-Sheet 3 7
+Sheet 2 7
 Title ""
 Date ""
@@
 F 0 "U1" H 8250 3150 60  0000 C CNN
 F 1 "iCE40HX8_CT256" H 8850 3000 60  0000 C CNN
-F 2 "" H 8150 3050 60  0001 C CNN
+F 2 "GTI_Footprint_Lib:BGA-256_12mmx12mm_Layout_14mmx14mm_P0.8mm_R0.5mm" H 8150 3050 60  0001 C CNN
 F 3 "" H 8150 3050 60  0001 C CNN
 	6    8150 3050
@@
 $EndComp
 $Comp
-L GND #PWR17
+L GND #PWR02
 U 1 1 5A3F82B7
 P 9950 3750
-F 0 "#PWR17" H 9950 3500 50  0001 C CNN
+F 0 "#PWR02" H 9950 3500 50  0001 C CNN
 F 1 "GND" H 9950 3600 50  0000 C CNN
 F 2 "" H 9950 3750 50  0001 C CNN
@@
 $EndComp
 $Comp
-L GND #PWR15
+L GND #PWR03
 U 1 1 5A2D962F
 P 9150 2000
-F 0 "#PWR15" H 9150 1750 50  0001 C CNN
+F 0 "#PWR03" H 9150 1750 50  0001 C CNN
 F 1 "GND" H 9150 1850 50  0000 C CNN
 F 2 "" H 9150 2000 50  0001 C CNN
@@
 $EndComp
 $Comp
-L GND #PWR14
+L GND #PWR04
 U 1 1 5A2D9808
 P 8700 1250
-F 0 "#PWR14" H 8700 1000 50  0001 C CNN
+F 0 "#PWR04" H 8700 1000 50  0001 C CNN
 F 1 "GND" H 8700 1100 50  0000 C CNN
 F 2 "" H 8700 1250 50  0001 C CNN
@@
 $EndComp
 $Comp
-L GND #PWR11
+L GND #PWR05
 U 1 1 5A2DC454
 P 7700 3850
-F 0 "#PWR11" H 7700 3600 50  0001 C CNN
+F 0 "#PWR05" H 7700 3600 50  0001 C CNN
 F 1 "GND" H 7850 3800 50  0000 C CNN
 F 2 "" H 7700 3850 50  0001 C CNN
@@
 $EndComp
 $Comp
-L GND #PWR13
+L GND #PWR06
 U 1 1 5A2DC8C5
 P 8500 2200
-F 0 "#PWR13" H 8500 1950 50  0001 C CNN
+F 0 "#PWR06" H 8500 1950 50  0001 C CNN
 F 1 "GND" H 8500 2050 50  0000 C CNN
 F 2 "" H 8500 2200 50  0001 C CNN
@@
 	7450 3200 7950 3200
 $Comp
-L GND #PWR18
+L GND #PWR07
 U 1 1 5A2E5ABD
 P 10750 3000
-F 0 "#PWR18" H 10750 2750 50  0001 C CNN
+F 0 "#PWR07" H 10750 2750 50  0001 C CNN
 F 1 "GND" H 10750 2850 50  0000 C CNN
 F 2 "" H 10750 3000 50  0001 C CNN
@@
 $EndComp
 $Comp
-L GND #PWR16
+L GND #PWR08
 U 1 1 5A2FB32F
 P 9350 1200
-F 0 "#PWR16" H 9350 950 50  0001 C CNN
+F 0 "#PWR08" H 9350 950 50  0001 C CNN
 F 1 "GND" H 9250 1200 50  0000 C CNN
 F 2 "" H 9350 1200 50  0001 C CNN
@@
 LED0
 $Comp
-L GND #PWR12
+L GND #PWR09
 U 1 1 5A4230FF
 P 7850 950
-F 0 "#PWR12" H 7850 700 50  0001 C CNN
+F 0 "#PWR09" H 7850 700 50  0001 C CNN
 F 1 "GND" H 7800 800 50  0000 C CNN
 F 2 "" H 7850 950 50  0001 C CNN

Commit message: Regrouping con't
Parts:
- TP10: footprint TestPoint:TestPoint_Pad_D2.0mm -> TestPoint:TestPoint_THTPad_D1.0mm_Drill0.5mm
Changed lines of the file:
@@
 $EndComp
 $Comp
-L GND #PWR02
+L GND #PWR8
 U 1 1 5A3F82B7
 P 9950 3750
-F 0 "#PWR02" H 9950 3500 50  0001 C CNN
+F 0 "#PWR8" H 9950 3500 50  0001 C CNN
 F 1 "GND" H 9950 3600 50  0000 C CNN
 F 2 "" H 9950 3750 50  0001 C CNN
@@
 $EndComp
 $Comp
-L GND #PWR03
+L GND #PWR6
 U 1 1 5A2D962F
 P 9150 2000
-F 0 "#PWR03" H 9150 1750 50  0001 C CNN
+F 0 "#PWR6" H 9150 1750 50  0001 C CNN
 F 1 "GND" H 9150 1850 50  0000 C CNN
 F 2 "" H 9150 2000 50  0001 C CNN
@@
 $EndComp
 $Comp
-L GND #PWR04
+L GND #PWR5
 U 1 1 5A2D9808
 P 8700 1250
-F 0 "#PWR04" H 8700 1000 50  0001 C CNN
+F 0 "#PWR5" H 8700 1000 50  0001 C CNN
 F 1 "GND" H 8700 1100 50  0000 C CNN
 F 2 "" H 8700 1250 50  0001 C CNN
@@
 $EndComp
 $Comp
-L GND #PWR05
+L GND #PWR2
 U 1 1 5A2DC454
 P 7700 3850
-F 0 "#PWR05" H 7700 3600 50  0001 C CNN
+F 0 "#PWR2" H 7700 3600 50  0001 C CNN
 F 1 "GND" H 7850 3800 50  0000 C CNN
 F 2 "" H 7700 3850 50  0001 C CNN
@@
 $EndComp
 $Comp
-L GND #PWR06
+L GND #PWR4
 U 1 1 5A2DC8C5
 P 8500 2200
-F 0 "#PWR06" H 8500 1950 50  0001 C CNN
+F 0 "#PWR4" H 8500 1950 50  0001 C CNN
 F 1 "GND" H 8500 2050 50  0000 C CNN
 F 2 "" H 8500 2200 50  0001 C CNN
@@
 	7450 3200 7950 3200
 $Comp
-L GND #PWR07
+L GND #PWR9
 U 1 1 5A2E5ABD
 P 10750 3000
-F 0 "#PWR07" H 10750 2750 50  0001 C CNN
+F 0 "#PWR9" H 10750 2750 50  0001 C CNN
 F 1 "GND" H 10750 2850 50  0000 C CNN
 F 2 "" H 10750 3000 50  0001 C CNN
@@
 F 0 "TP10" V 1850 7750 50  0000 C CNN
 F 1 "PLL CLK2 OUT" V 1850 8250 50  0000 C CNN
-F 2 "TestPoint:TestPoint_Pad_D2.0mm" H 2050 7450 50  0001 C CNN
+F 2 "TestPoint:TestPoint_THTPad_D1.0mm_Drill0.5mm" H 2050 7450 50  0001 C CNN
 F 3 "" H 2050 7450 50  0001 C CNN
 	1    1850 7450
@@
 $EndComp
 $Comp
-L GND #PWR08
+L GND #PWR7
 U 1 1 5A2FB32F
 P 9350 1200
-F 0 "#PWR08" H 9350 950 50  0001 C CNN
+F 0 "#PWR7" H 9350 950 50  0001 C CNN
 F 1 "GND" H 9250 1200 50  0000 C CNN
 F 2 "" H 9350 1200 50  0001 C CNN
@@
 LED0
 $Comp
-L GND #PWR09
+L GND #PWR3
 U 1 1 5A4230FF
 P 7850 950
-F 0 "#PWR09" H 7850 700 50  0001 C CNN
+F 0 "#PWR3" H 7850 700 50  0001 C CNN
 F 1 "GND" H 7800 800 50  0000 C CNN
 F 2 "" H 7850 950 50  0001 C CNN

Commit message: grouping complete ready to route
Parts:
- TP9: footprint TestPoint:TestPoint_Pad_D2.0mm -> TestPoint:TestPoint_Pad_D1.0mm
Changed lines of the file:
@@
 $EndComp
 $Comp
-L GND #PWR8
+L GND #PWR02
 U 1 1 5A3F82B7
 P 9950 3750
-F 0 "#PWR8" H 9950 3500 50  0001 C CNN
+F 0 "#PWR02" H 9950 3500 50  0001 C CNN
 F 1 "GND" H 9950 3600 50  0000 C CNN
 F 2 "" H 9950 3750 50  0001 C CNN
@@
 $EndComp
 $Comp
-L GND #PWR6
+L GND #PWR03
 U 1 1 5A2D962F
 P 9150 2000
-F 0 "#PWR6" H 9150 1750 50  0001 C CNN
+F 0 "#PWR03" H 9150 1750 50  0001 C CNN
 F 1 "GND" H 9150 1850 50  0000 C CNN
 F 2 "" H 9150 2000 50  0001 C CNN
@@
 $EndComp
 $Comp
-L GND #PWR5
+L GND #PWR04
 U 1 1 5A2D9808
 P 8700 1250
-F 0 "#PWR5" H 8700 1000 50  0001 C CNN
+F 0 "#PWR04" H 8700 1000 50  0001 C CNN
 F 1 "GND" H 8700 1100 50  0000 C CNN
 F 2 "" H 8700 1250 50  0001 C CNN
@@
 $EndComp
 $Comp
-L GND #PWR2
+L GND #PWR05
 U 1 1 5A2DC454
 P 7700 3850
-F 0 "#PWR2" H 7700 3600 50  0001 C CNN
+F 0 "#PWR05" H 7700 3600 50  0001 C CNN
 F 1 "GND" H 7850 3800 50  0000 C CNN
 F 2 "" H 7700 3850 50  0001 C CNN
@@
 $EndComp
 $Comp
-L GND #PWR4
+L GND #PWR06
 U 1 1 5A2DC8C5
 P 8500 2200
-F 0 "#PWR4" H 8500 1950 50  0001 C CNN
+F 0 "#PWR06" H 8500 1950 50  0001 C CNN
 F 1 "GND" H 8500 2050 50  0000 C CNN
 F 2 "" H 8500 2200 50  0001 C CNN
@@
 	7450 3200 7950 3200
 $Comp
-L GND #PWR9
+L GND #PWR07
 U 1 1 5A2E5ABD
 P 10750 3000
-F 0 "#PWR9" H 10750 2750 50  0001 C CNN
+F 0 "#PWR07" H 10750 2750 50  0001 C CNN
 F 1 "GND" H 10750 2850 50  0000 C CNN
 F 2 "" H 10750 3000 50  0001 C CNN
@@
 F 0 "TP9" V 1850 4000 50  0000 C CNN
 F 1 "PLL CLK1 OUT" V 1850 4500 50  0000 C CNN
-F 2 "TestPoint:TestPoint_Pad_D2.0mm" H 2050 3700 50  0001 C CNN
+F 2 "TestPoint:TestPoint_Pad_D1.0mm" H 2050 3700 50  0001 C CNN
 F 3 "" H 2050 3700 50  0001 C CNN
 	1    1850 3700
@@
 $EndComp
 $Comp
-L GND #PWR7
+L GND #PWR08
 U 1 1 5A2FB32F
 P 9350 1200
-F 0 "#PWR7" H 9350 950 50  0001 C CNN
+F 0 "#PWR08" H 9350 950 50  0001 C CNN
 F 1 "GND" H 9250 1200 50  0000 C CNN
 F 2 "" H 9350 1200 50  0001 C CNN
@@
 LED0
 $Comp
-L GND #PWR3
+L GND #PWR09
 U 1 1 5A4230FF
 P 7850 950
-F 0 "#PWR3" H 7850 700 50  0001 C CNN
+F 0 "#PWR09" H 7850 700 50  0001 C CNN
 F 1 "GND" H 7800 800 50  0000 C CNN
 F 2 "" H 7850 950 50  0001 C CNN
