File: ice40_FPGA_Breakout/USB_FTDI.sch (KiCad schematic (older format))
At the start: 52 parts, among them J1 USB_B_Micro, J2 3pos_Jumper, J3 3pos_Jumper, U5 93LCxxC, U6 FT2232H, Y1 ABM10AIG-12.000MHZ-4Z-T3

Commit message: grouping complete ready to route
Parts:
- TP11: footprint TestPoint:TestPoint_Pad_D2.0mm -> TestPoint:TestPoint_Pad_D1.0mm
Changed lines of the file:
@@
 $EndComp
 $Comp
-L GND #PWR27
+L GND #PWR014
 U 1 1 5A0D11EC
 P 7550 6150
-F 0 "#PWR27" H 7550 5900 50  0001 C CNN
+F 0 "#PWR014" H 7550 5900 50  0001 C CNN
 F 1 "GND" H 7550 6000 50  0000 C CNN
 F 2 "" H 7550 6150 50  0001 C CNN
@@
 $EndComp
 $Comp
-L GND #PWR23
+L GND #PWR015
 U 1 1 5A0D12CE
 P 5500 6100
-F 0 "#PWR23" H 5500 5850 50  0001 C CNN
+F 0 "#PWR015" H 5500 5850 50  0001 C CNN
 F 1 "GND" H 5500 5950 50  0000 C CNN
 F 2 "" H 5500 6100 50  0001 C CNN
@@
 $EndComp
 $Comp
-L GND #PWR20
+L GND #PWR016
 U 1 1 5A0D137A
 P 4950 6100
-F 0 "#PWR20" H 4950 5850 50  0001 C CNN
+F 0 "#PWR016" H 4950 5850 50  0001 C CNN
 F 1 "GND" H 4950 5950 50  0000 C CNN
 F 2 "" H 4950 6100 50  0001 C CNN
@@
 $EndComp
 $Comp
-L GND #PWR26
+L GND #PWR017
 U 1 1 5A0D14C2
 P 5750 2550
-F 0 "#PWR26" H 5750 2300 50  0001 C CNN
+F 0 "#PWR017" H 5750 2300 50  0001 C CNN
 F 1 "GND" H 5750 2400 50  0000 C CNN
 F 2 "" H 5750 2550 50  0001 C CNN
@@
 $EndComp
 $Comp
-L GND #PWR22
+L GND #PWR018
 U 1 1 5A0D1506
 P 5500 2550
-F 0 "#PWR22" H 5500 2300 50  0001 C CNN
+F 0 "#PWR018" H 5500 2300 50  0001 C CNN
 F 1 "GND" H 5500 2400 50  0000 C CNN
 F 2 "" H 5500 2550 50  0001 C CNN
@@
 $EndComp
 $Comp
-L GND #PWR16
+L GND #PWR019
 U 1 1 5A0D154A
 P 3150 5000
-F 0 "#PWR16" H 3150 4750 50  0001 C CNN
+F 0 "#PWR019" H 3150 4750 50  0001 C CNN
 F 1 "GND" H 3150 4850 50  0000 C CNN
 F 2 "" H 3150 5000 50  0001 C CNN
@@
 $EndComp
 $Comp
-L GND #PWR15
+L GND #PWR020
 U 1 1 5A0D172E
 P 2500 1600
-F 0 "#PWR15" H 2500 1350 50  0001 C CNN
+F 0 "#PWR020" H 2500 1350 50  0001 C CNN
 F 1 "GND" H 2500 1450 50  0000 C CNN
 F 2 "" H 2500 1600 50  0001 C CNN
@@
 $EndComp
 $Comp
-L GND #PWR18
+L GND #PWR021
 U 1 1 5A0D17DA
 P 4500 3450
-F 0 "#PWR18" H 4500 3200 50  0001 C CNN
+F 0 "#PWR021" H 4500 3200 50  0001 C CNN
 F 1 "GND" H 4500 3300 50  0000 C CNN
 F 2 "" H 4500 3450 50  0001 C CNN
@@
 $EndComp
 $Comp
-L GND #PWR14
+L GND #PWR022
 U 1 1 5A0D263E
 P 1550 3300
-F 0 "#PWR14" H 1550 3050 50  0001 C CNN
+F 0 "#PWR022" H 1550 3050 50  0001 C CNN
 F 1 "GND" H 1550 3150 50  0000 C CNN
 F 2 "" H 1550 3300 50  0001 C CNN
@@
 $EndComp
 $Comp
-L GND #PWR17
+L GND #PWR023
 U 1 1 5A0E190F
 P 3400 5000
-F 0 "#PWR17" H 3400 4750 50  0001 C CNN
+F 0 "#PWR023" H 3400 4750 50  0001 C CNN
 F 1 "GND" H 3400 4850 50  0000 C CNN
 F 2 "" H 3400 5000 50  0001 C CNN
@@
 $EndComp
 $Comp
-L GND #PWR25
+L GND #PWR024
 U 1 1 5A0E83DE
 P 5550 3950
-F 0 "#PWR25" H 5550 3700 50  0001 C CNN
+F 0 "#PWR024" H 5550 3700 50  0001 C CNN
 F 1 "GND" H 5550 3800 50  0000 C CNN
 F 2 "" H 5550 3950 50  0001 C CNN
@@
 4.7V from USB
 $Comp
-L GND #PWR24
+L GND #PWR025
 U 1 1 5A0F5EF9
 P 5550 1600
-F 0 "#PWR24" H 5550 1350 50  0001 C CNN
+F 0 "#PWR025" H 5550 1350 50  0001 C CNN
 F 1 "GND" H 5550 1450 50  0000 C CNN
 F 2 "" H 5550 1600 50  0001 C CNN
@@
 $EndComp
 $Comp
-L GND #PWR21
+L GND #PWR026
 U 1 1 5A2C2E4B
 P 5250 5650
-F 0 "#PWR21" H 5250 5400 50  0001 C CNN
+F 0 "#PWR026" H 5250 5400 50  0001 C CNN
 F 1 "GND" H 5250 5500 50  0000 C CNN
 F 2 "" H 5250 5650 50  0001 C CNN
@@
 F 0 "TP11" H 2000 1620 50  0000 C CNN
 F 1 "Test_Point" H 2000 1550 50  0000 C CNN
-F 2 "TestPoint:TestPoint_Pad_D2.0mm" H 2200 1350 50  0001 C CNN
+F 2 "TestPoint:TestPoint_Pad_D1.0mm" H 2200 1350 50  0001 C CNN
 F 3 "" H 2200 1350 50  0001 C CNN
 	1    2000 1350
@@
 1V8_REG
 $Comp
-L GND #PWR19
+L GND #PWR027
 U 1 1 5A40997E
 P 4750 1150
-F 0 "#PWR19" H 4750 900 50  0001 C CNN
+F 0 "#PWR027" H 4750 900 50  0001 C CNN
 F 1 "GND" H 4750 1000 50  0000 C CNN
 F 2 "" H 4750 1150 50  0001 C CNN
@@
 Connection ~ 4750 3350
 $Comp
-L GND #PWR28
+L GND #PWR028
 U 1 1 5ACC1320
 P 9750 1575
-F 0 "#PWR28" H 9750 1325 50  0001 C CNN
+F 0 "#PWR028" H 9750 1325 50  0001 C CNN
 F 1 "GND" H 9750 1425 50  0000 C CNN
 F 2 "" H 9750 1575 50  0001 C CNN
