File: ice40_FPGA_Breakout/Xtal_Bias_Test.sch (KiCad schematic (older format))
At the start: 61 parts, among them J4 4POS_JUMPER, J5 4POS_JUMPER, J6 4POS_JUMPER, J7 4POS_JUMPER, J8 4POS_JUMPER, U7 MIC53x4, X1 OSC_4-SMD, X2 OSC_6-SMD

Commit message: Regrouping con't
Parts:
- TP12: footprint TestPoint:TestPoint_Pad_D2.0mm -> TestPoint:TestPoint_THTPad_D1.0mm_Drill0.5mm
Changed lines of the file:
@@
 $EndComp
 $Comp
-L GND #PWR029
+L GND #PWR35
 U 1 1 5A30306B
 P 6900 3200
-F 0 "#PWR029" H 6900 2950 50  0001 C CNN
+F 0 "#PWR35" H 6900 2950 50  0001 C CNN
 F 1 "GND" H 7050 3150 50  0000 C CNN
 F 2 "" H 6900 3200 50  0001 C CNN
@@
 $EndComp
 $Comp
-L GND #PWR030
+L GND #PWR37
 U 1 1 5A303071
 P 7750 3150
-F 0 "#PWR030" H 7750 2900 50  0001 C CNN
+F 0 "#PWR37" H 7750 2900 50  0001 C CNN
 F 1 "GND" H 7900 3100 50  0000 C CNN
 F 2 "" H 7750 3150 50  0001 C CNN
@@
 $EndComp
 $Comp
-L GND #PWR031
+L GND #PWR34
 U 1 1 5A3030AF
 P 6900 2050
-F 0 "#PWR031" H 6900 1800 50  0001 C CNN
+F 0 "#PWR34" H 6900 1800 50  0001 C CNN
 F 1 "GND" H 7050 2000 50  0000 C CNN
 F 2 "" H 6900 2050 50  0001 C CNN
@@
 $EndComp
 $Comp
-L GND #PWR032
+L GND #PWR36
 U 1 1 5A3030B5
 P 7750 2000
-F 0 "#PWR032" H 7750 1750 50  0001 C CNN
+F 0 "#PWR36" H 7750 1750 50  0001 C CNN
 F 1 "GND" H 7900 1950 50  0000 C CNN
 F 2 "" H 7750 2000 50  0001 C CNN
@@
 GND
 $Comp
-L GND #PWR033
+L GND #PWR33
 U 1 1 5A406131
 P 6400 1350
-F 0 "#PWR033" H 6400 1100 50  0001 C CNN
+F 0 "#PWR33" H 6400 1100 50  0001 C CNN
 F 1 "GND" H 6550 1300 50  0000 C CNN
 F 2 "" H 6400 1350 50  0001 C CNN
@@
 $EndComp
 $Comp
-L GND #PWR034
+L GND #PWR29
 U 1 1 5A4CCE3C
 P 1300 2950
-F 0 "#PWR034" H 1300 2700 50  0001 C CNN
+F 0 "#PWR29" H 1300 2700 50  0001 C CNN
 F 1 "GND" H 1300 2800 50  0000 C CNN
 F 2 "" H 1300 2950 50  0001 C CNN
@@
 $EndComp
 $Comp
-L GND #PWR035
+L GND #PWR32
 U 1 1 5A4CCE5E
 P 4850 2850
-F 0 "#PWR035" H 4850 2600 50  0001 C CNN
+F 0 "#PWR32" H 4850 2600 50  0001 C CNN
 F 1 "GND" H 4850 2700 50  0000 C CNN
 F 2 "" H 4850 2850 50  0001 C CNN
@@
 $EndComp
 $Comp
-L GND #PWR036
+L GND #PWR31
 U 1 1 5A4CCE8E
 P 3900 4200
-F 0 "#PWR036" H 3900 3950 50  0001 C CNN
+F 0 "#PWR31" H 3900 3950 50  0001 C CNN
 F 1 "GND" H 3900 4050 50  0000 C CNN
 F 2 "" H 3900 4200 50  0001 C CNN
@@
 $EndComp
 $Comp
-L GND #PWR037
+L GND #PWR30
 U 1 1 5A4CCE94
 P 2500 4200
-F 0 "#PWR037" H 2500 3950 50  0001 C CNN
+F 0 "#PWR30" H 2500 3950 50  0001 C CNN
 F 1 "GND" H 2500 4050 50  0000 C CNN
 F 2 "" H 2500 4200 50  0001 C CNN
@@
 F 0 "TP12" V 5200 3500 50  0000 C CNN
 F 1 "Test_Point" V 5100 3450 50  0000 C CNN
-F 2 "TestPoint:TestPoint_Pad_D2.0mm" H 5400 3200 50  0001 C CNN
+F 2 "TestPoint:TestPoint_THTPad_D1.0mm_Drill0.5mm" H 5400 3200 50  0001 C CNN
 F 3 "" H 5400 3200 50  0001 C CNN
 	1    5200 3200
