File: ice40_FPGA_Breakout/hiltop_backplane_brd.sch (KiCad schematic (older format))
At the start: 0 parts

Commit message: mother board to backplane connector added, power connector added
Changed lines of the file:
@@
 $Descr A4 11693 8268
 encoding utf-8
-Sheet 1 5
+Sheet 1 6
 Title "Project X"
 Date ""
@@
 Wire Wire Line
 	9125 975  9125 1000
+$Sheet
+S 1700 3100 2000 2050
+U 5C074E5E
+F0 "MotherBoard_Connector" 60
+F1 "MotherBoard_Connector.sch" 60
+$EndSheet
 $EndSCHEMATC
