File: kicad_hiltop_63hp_backplane/_autosave-hiltop_backplane_brd.kicad_pcb (KiCad board)
At the start: 6 copper layers, 200 x 129 mm, 232 parts, among them J1 USB_B_Micro, J10 Conn_01x02, J11 SO-DIMM, J12 4POS_JUMPER, J13 4POS_JUMPER, J14 4POS_JUMPER, J2 3pos_Jumper, J3 3pos_Jumper, J4 4POS_JUMPER, J5 4POS_JUMPER, J6 CONN_DIN_HDR_96POS, J7 HILTOP_PCIE-64_CONN, J8 Conn_02x04_Odd_Even, J9 Conn_02x02_Counter_Clockwise, U1 93LCxxC, U2 FT2232H, U3 LTC4311, U4 LTC4311, U5 USB2517, Y1 ABM10AIG-12.000MHZ-4Z-T3, Y2 24Mhz Xtal

Commit message: schematic error reduced and footprint mapped
Parts:
- added J15: 4POS_JUMPER, Connector_PinHeader_2.00mm:PinHeader_2x02_P2.00mm_Vertical, F.Cu at (127.3, -52.8)
- added J16: 4POS_JUMPER, Connector_PinHeader_2.00mm:PinHeader_2x02_P2.00mm_Vertical, F.Cu at (132.3, -52.8)
- J4, J5: value 4POS_JUMPER -> CONN_DIN_HDR_96POS
- moved J7 228.7 mm to (-62.5, -77.2)
Connections:
- J4 pad 1: /USB_HUB_LED_JUMPERS/FTDI_AD3_SS -> (no net)
- J4 pad 10a: (no net) -> GND
- J4 pad 10b: (no net) -> /SPI0_SCK
- J4 pad 10c: (no net) -> Net-(F5-Pad1)
- J4 pad 11a: (no net) -> /backplane_connector/FPGA_GPIO1
- J4 pad 11b: (no net) -> /SPI0_CS0
- J4 pad 11c: (no net) -> GND
- J4 pad 12a: (no net) -> /backplane_connector/FPGA_GPIO2
- J4 pad 12b: (no net) -> /SPI0_CS1
- J4 pad 12c: (no net) -> /I2C0_SDA
- J4 pad 13a: (no net) -> /backplane_connector/FPGA_GPIO3
- J4 pad 13b: (no net) -> GND
- J4 pad 13c: (no net) -> /I2C0_SCL
- J4 pad 14a: (no net) -> /backplane_connector/FPGA_GPIO4
- J4 pad 14b: (no net) -> /SPI1_MOSI
- J4 pad 14c: (no net) -> GND
- J4 pad 15a: (no net) -> /backplane_connector/FPGA_GPIO5
- J4 pad 15b: (no net) -> /SPI1_MISO
- J4 pad 15c: (no net) -> /I2C1_SDA
- J4 pad 16a: (no net) -> /backplane_connector/FPGA_GPIO6
- J4 pad 16b: (no net) -> /SPI1_SCK
- J4 pad 16c: (no net) -> /I2C1_SCL
- J4 pad 17a: (no net) -> /backplane_connector/FPGA_GPIO7
- J4 pad 17b: (no net) -> /SPI1_CS0
- J4 pad 17c: (no net) -> GND
- J4 pad 18a: (no net) -> /backplane_connector/FPGA_GPIO8
- J4 pad 18b: (no net) -> /SPI1_CS1
- J4 pad 18c: (no net) -> /ice40_breakout_brd/GPIO_34
- J4 pad 19a: (no net) -> /backplane_connector/FPGA_GPIO9
- J4 pad 19b: (no net) -> /SPI1_CS2
- J4 pad 19c: (no net) -> /ice40_breakout_brd/GPIO_35
- J4 pad 1a: (no net) -> GND
- J4 pad 1b: (no net) -> GND
- J4 pad 1c: (no net) -> Net-(F1-Pad1)
- J4 pad 20a: (no net) -> /backplane_connector/FPGA_GPIO10
- J4 pad 20b: (no net) -> /ice40_breakout_brd/GPIO_31
- J4 pad 20c: (no net) -> /ice40_breakout_brd/GPIO_36
- J4 pad 21a: (no net) -> GND
- J4 pad 21b: (no net) -> /ice40_breakout_brd/GPIO_32
- J4 pad 21c: (no net) -> /ice40_breakout_brd/GPIO_37
- J4 pad 22a: (no net) -> /ice40_breakout_brd/GPIO_38
- J4 pad 22b: (no net) -> /ice40_breakout_brd/GPIO_33
- J4 pad 22c: (no net) -> /PWM0
- J4 pad 23a: (no net) -> /ice40_breakout_brd/GPIO_39
- J4 pad 23b: (no net) -> GND
- J4 pad 23c: (no net) -> /PWM1
- J4 pad 24a: (no net) -> /ice40_breakout_brd/GPIO_40
- J4 pad 24b: (no net) -> /CLK
- J4 pad 24c: (no net) -> GND
- J4 pad 25a: (no net) -> /backplane_connector/LCOM1
- J4 pad 25b: (no net) -> /TRIG
- J4 pad 25c: (no net) -> /backplane_connector/RCOM1A
- J4 pad 26a: (no net) -> /backplane_connector/LCOM2
- J4 pad 26b: (no net) -> /PSEL0
- J4 pad 26c: (no net) -> /backplane_connector/RCOM2A
- J4 pad 27a: (no net) -> /backplane_connector/LCOM3
- J4 pad 27b: (no net) -> /SHUTDOWN
- J4 pad 27c: (no net) -> /backplane_connector/RCOM3A
- J4 pad 28a: (no net) -> /backplane_connector/LCOM4
- J4 pad 28b: (no net) -> /RST
- J4 pad 28c: (no net) -> /backplane_connector/RCOM4A
- J4 pad 29a: (no net) -> /backplane_connector/LCOM5
- J4 pad 29b: (no net) -> GND
- J4 pad 29c: (no net) -> /backplane_connector/RCOM5A
- J4 pad 2a: (no net) -> Net-(J4-Pad2a)
- J4 pad 2b: (no net) -> GND
- J4 pad 2c: (no net) -> Net-(F1-Pad1)
- J4 pad 30a: (no net) -> /backplane_connector/LCOM6
- J4 pad 30b: (no net) -> /USB1_N
- J4 pad 30c: (no net) -> /backplane_connector/RCOM6A
- J4 pad 31a: (no net) -> /backplane_connector/LCOM7
- J4 pad 31b: (no net) -> /USB1_P
- J4 pad 31c: (no net) -> /backplane_connector/RCOM7A
- J4 pad 32a: (no net) -> /backplane_connector/LCOM8
- J4 pad 32b: (no net) -> GND
- J4 pad 32c: (no net) -> /backplane_connector/RCOM8A
- J4 pad 3a: (no net) -> Net-(J4-Pad3a)
- J4 pad 3b: (no net) -> GND
- J4 pad 3c: (no net) -> Net-(F2-Pad1)
- J4 pad 4a: (no net) -> GND
- J4 pad 4b: (no net) -> GND
- J4 pad 4c: (no net) -> Net-(F2-Pad1)
- J4 pad 5a: (no net) -> Net-(J4-Pad5a)
- J4 pad 5b: (no net) -> GND
- J4 pad 5c: (no net) -> Net-(F3-Pad1)
- J4 pad 6a: (no net) -> Net-(J4-Pad6a)
- J4 pad 6b: (no net) -> GND
- J4 pad 6c: (no net) -> Net-(F3-Pad1)
- J4 pad 7a: (no net) -> GND
- J4 pad 7b: (no net) -> GND
- J4 pad 7c: (no net) -> Net-(F4-Pad1)
- J4 pad 8a: (no net) -> Net-(J4-Pad8a)
- J4 pad 8b: (no net) -> /SPI0_MOSI
- J4 pad 8c: (no net) -> Net-(F4-Pad1)
- J4 pad 9a: (no net) -> Net-(J4-Pad9a)
- J4 pad 9b: (no net) -> /SPI0_MISO
- J4 pad 9c: (no net) -> Net-(F5-Pad1)
- J5 pad 1: /USB_HUB_LED_JUMPERS/FPGA_SPI_SDO -> (no net)
- J5 pad 10a: (no net) -> GND
- J5 pad 10b: (no net) -> /SPI0_SCK
- J5 pad 10c: (no net) -> Net-(F10-Pad1)
- J5 pad 11a: (no net) -> /backplane_connector/FPGA_GPIO11
- J5 pad 11b: (no net) -> /SPI0_CS0
- J5 pad 11c: (no net) -> GND
- J5 pad 12a: (no net) -> /backplane_connector/FPGA_GPIO12
- J5 pad 12b: (no net) -> /SPI0_CS1
- J5 pad 12c: (no net) -> /I2C0_SDA
- J5 pad 13a: (no net) -> /backplane_connector/FPGA_GPIO13
- J5 pad 13b: (no net) -> GND
- J5 pad 13c: (no net) -> /I2C0_SCL
- J5 pad 14a: (no net) -> /backplane_connector/FPGA_GPIO14
- J5 pad 14b: (no net) -> /SPI1_MOSI
- J5 pad 14c: (no net) -> GND
- J5 pad 15a: (no net) -> /backplane_connector/FPGA_GPIO15
- J5 pad 15b: (no net) -> /SPI1_MISO
- J5 pad 15c: (no net) -> /I2C1_SDA
- J5 pad 16a: (no net) -> /backplane_connector/FPGA_GPIO16
- J5 pad 16b: (no net) -> /SPI1_SCK
- J5 pad 16c: (no net) -> /I2C1_SCL
- J5 pad 17a: (no net) -> /backplane_connector/FPGA_GPIO17
- J5 pad 17b: (no net) -> /SPI1_CS0
- J5 pad 17c: (no net) -> GND
- J5 pad 18a: (no net) -> /backplane_connector/FPGA_GPIO18
- J5 pad 18b: (no net) -> /SPI1_CS1
- J5 pad 18c: (no net) -> /ice40_breakout_brd/GPIO_34
- J5 pad 19a: (no net) -> /backplane_connector/FPGA_GPIO19
- J5 pad 19b: (no net) -> /SPI1_CS2
- J5 pad 19c: (no net) -> /ice40_breakout_brd/GPIO_35
- J5 pad 1a: (no net) -> GND
- J5 pad 1b: (no net) -> GND
- J5 pad 1c: (no net) -> Net-(F6-Pad1)
- J5 pad 20a: (no net) -> /backplane_connector/FPGA_GPIO20
- J5 pad 20b: (no net) -> /ice40_breakout_brd/GPIO_31
- J5 pad 20c: (no net) -> /ice40_breakout_brd/GPIO_36
- J5 pad 21a: (no net) -> GND
- J5 pad 21b: (no net) -> /ice40_breakout_brd/GPIO_32
- J5 pad 21c: (no net) -> /ice40_breakout_brd/GPIO_37
- J5 pad 22a: (no net) -> /ice40_breakout_brd/GPIO_38
- J5 pad 22b: (no net) -> /ice40_breakout_brd/GPIO_33
- J5 pad 22c: (no net) -> /PWM0
- J5 pad 23a: (no net) -> /ice40_breakout_brd/GPIO_39
- J5 pad 23b: (no net) -> GND
- J5 pad 23c: (no net) -> /PWM1
- J5 pad 24a: (no net) -> /ice40_breakout_brd/GPIO_40
- J5 pad 24b: (no net) -> /CLK
- J5 pad 24c: (no net) -> GND
- J5 pad 25a: (no net) -> /backplane_connector/RCOM1A
- J5 pad 25b: (no net) -> /TRIG
- J5 pad 25c: (no net) -> /backplane_connector/RCOM1B
- J5 pad 26a: (no net) -> /backplane_connector/RCOM2A
- J5 pad 26b: (no net) -> /PSEL1
- J5 pad 26c: (no net) -> /backplane_connector/RCOM2B
- J5 pad 27a: (no net) -> /backplane_connector/RCOM3A
- J5 pad 27b: (no net) -> /SHUTDOWN
- J5 pad 27c: (no net) -> /backplane_connector/RCOM3B
- J5 pad 28a: (no net) -> /backplane_connector/RCOM4A
- J5 pad 28b: (no net) -> /RST
- J5 pad 28c: (no net) -> /backplane_connector/RCOM4B
- J5 pad 29a: (no net) -> /backplane_connector/RCOM5A
- J5 pad 29b: (no net) -> GND
- J5 pad 29c: (no net) -> /backplane_connector/RCOM5B
- J5 pad 2a: (no net) -> Net-(J5-Pad2a)
- J5 pad 2b: (no net) -> GND
- J5 pad 2c: (no net) -> Net-(F6-Pad1)
- J5 pad 30a: (no net) -> /backplane_connector/RCOM6A
- J5 pad 30b: (no net) -> /USB2_P
- J5 pad 30c: (no net) -> /backplane_connector/RCOM6B
- J5 pad 31a: (no net) -> /backplane_connector/RCOM7A
- J5 pad 31b: (no net) -> /USB2_N
- J5 pad 31c: (no net) -> /backplane_connector/RCOM7B
- J5 pad 32a: (no net) -> /backplane_connector/RCOM8A
- J5 pad 32b: (no net) -> GND
- J5 pad 32c: (no net) -> /backplane_connector/RCOM8B
- J5 pad 3a: (no net) -> Net-(J5-Pad3a)
- J5 pad 3b: (no net) -> GND
- J5 pad 3c: (no net) -> Net-(F7-Pad1)
- J5 pad 4a: (no net) -> GND
- J5 pad 4b: (no net) -> GND
- J5 pad 4c: (no net) -> Net-(F7-Pad1)
- J5 pad 5a: (no net) -> Net-(J5-Pad5a)
- J5 pad 5b: (no net) -> GND
- J5 pad 5c: (no net) -> Net-(F8-Pad1)
- J5 pad 6a: (no net) -> Net-(J5-Pad6a)
- J5 pad 6b: (no net) -> GND
- J5 pad 6c: (no net) -> Net-(F8-Pad1)
- J5 pad 7a: (no net) -> GND
- J5 pad 7b: (no net) -> GND
- J5 pad 7c: (no net) -> Net-(F9-Pad1)
- J5 pad 8a: (no net) -> Net-(J5-Pad8a)
- J5 pad 8b: (no net) -> /SPI0_MOSI
- J5 pad 8c: (no net) -> Net-(F9-Pad1)
- J5 pad 9a: (no net) -> Net-(J5-Pad9a)
- J5 pad 9b: (no net) -> /SPI0_MISO
- J5 pad 9c: (no net) -> Net-(F10-Pad1)
- J6 pad 1: GND -> (no net)
- J6 pad 10a: (no net) -> GND
- J6 pad 10b: (no net) -> /SPI0_SCK
- J6 pad 10c: (no net) -> Net-(F15-Pad1)
- J6 pad 11a: (no net) -> /backplane_connector/FPGA_GPIO21
- J6 pad 11b: (no net) -> /SPI0_CS0
- J6 pad 11c: (no net) -> GND
- J6 pad 12a: (no net) -> /backplane_connector/FPGA_GPIO22
- J6 pad 12b: (no net) -> /SPI0_CS1
- J6 pad 12c: (no net) -> /I2C0_SDA
- J6 pad 13a: (no net) -> /backplane_connector/FPGA_GPIO23
- J6 pad 13b: (no net) -> GND
- J6 pad 13c: (no net) -> /I2C0_SCL
- J6 pad 14a: (no net) -> /backplane_connector/FPGA_GPIO24
- J6 pad 14b: (no net) -> /SPI1_MOSI
- J6 pad 14c: (no net) -> GND
- J6 pad 15a: (no net) -> /backplane_connector/FPGA_GPIO25
- J6 pad 15b: (no net) -> /SPI1_MISO
- J6 pad 15c: (no net) -> /I2C1_SDA
- J6 pad 16a: (no net) -> /backplane_connector/FPGA_GPIO26
- J6 pad 16b: (no net) -> /SPI1_SCK
- J6 pad 16c: (no net) -> /I2C1_SCL
- J6 pad 17a: (no net) -> /backplane_connector/FPGA_GPIO27
- J6 pad 17b: (no net) -> /SPI1_CS0
- J6 pad 17c: (no net) -> GND
- J6 pad 18a: (no net) -> /backplane_connector/FPGA_GPIO28
- J6 pad 18b: (no net) -> /SPI1_CS1
- J6 pad 18c: (no net) -> /ice40_breakout_brd/GPIO_34
- J6 pad 19a: (no net) -> /backplane_connector/FPGA_GPIO29
- J6 pad 19b: (no net) -> /SPI1_CS2
- J6 pad 19c: (no net) -> /ice40_breakout_brd/GPIO_35
- J6 pad 1a: (no net) -> GND
- J6 pad 1b: (no net) -> GND
- J6 pad 1c: (no net) -> Net-(F11-Pad1)
- J6 pad 20a: (no net) -> /backplane_connector/FPGA_GPIO30
- J6 pad 20b: (no net) -> /ice40_breakout_brd/GPIO_31
- J6 pad 20c: (no net) -> /ice40_breakout_brd/GPIO_36
- J6 pad 21a: (no net) -> GND
- J6 pad 21b: (no net) -> /ice40_breakout_brd/GPIO_32
- J6 pad 21c: (no net) -> /ice40_breakout_brd/GPIO_37
- J6 pad 22a: (no net) -> /ice40_breakout_brd/GPIO_38
- J6 pad 22b: (no net) -> /ice40_breakout_brd/GPIO_33
- J6 pad 22c: (no net) -> /PWM0
- J6 pad 23a: (no net) -> /ice40_breakout_brd/GPIO_39
- J6 pad 23b: (no net) -> GND
- J6 pad 23c: (no net) -> /PWM1
- J6 pad 24a: (no net) -> /ice40_breakout_brd/GPIO_40
- J6 pad 24b: (no net) -> /CLK
- J6 pad 24c: (no net) -> GND
- J6 pad 25a: (no net) -> /backplane_connector/RCOM1B
- J6 pad 25b: (no net) -> /TRIG
- J6 pad 25c: (no net) -> /backplane_connector/RCOM1
- J6 pad 26a: (no net) -> /backplane_connector/RCOM2B
- J6 pad 26b: (no net) -> /PSEL2
- J6 pad 26c: (no net) -> /backplane_connector/RCOM2
- J6 pad 27a: (no net) -> /backplane_connector/RCOM3B
- J6 pad 27b: (no net) -> /SHUTDOWN
- J6 pad 27c: (no net) -> /backplane_connector/RCOM3
- J6 pad 28a: (no net) -> /backplane_connector/RCOM4B
- J6 pad 28b: (no net) -> /RST
- J6 pad 28c: (no net) -> /backplane_connector/RCOM4
- J6 pad 29a: (no net) -> /backplane_connector/RCOM5B
- J6 pad 29b: (no net) -> GND
- J6 pad 29c: (no net) -> /backplane_connector/RCOM5
- J6 pad 2a: (no net) -> Net-(J6-Pad2a)
- J6 pad 2b: (no net) -> GND
- J6 pad 2c: (no net) -> Net-(F11-Pad1)
- J6 pad 30a: (no net) -> /backplane_connector/RCOM6B
- J6 pad 30b: (no net) -> /USB3_N
- J6 pad 30c: (no net) -> /backplane_connector/RCOM6
- J6 pad 31a: (no net) -> /backplane_connector/RCOM7B
- J6 pad 31b: (no net) -> /USB3_P
- J6 pad 31c: (no net) -> /backplane_connector/RCOM7
- J6 pad 32a: (no net) -> /backplane_connector/RCOM8B
- J6 pad 32b: (no net) -> GND
- J6 pad 32c: (no net) -> /backplane_connector/RCOM8
- J6 pad 3a: (no net) -> Net-(J6-Pad3a)
- J6 pad 3b: (no net) -> GND
- J6 pad 3c: (no net) -> Net-(F12-Pad1)
- J6 pad 4a: (no net) -> GND
- J6 pad 4b: (no net) -> GND
- J6 pad 4c: (no net) -> Net-(F12-Pad1)
- J6 pad 5a: (no net) -> Net-(J6-Pad5a)
- J6 pad 5b: (no net) -> GND
- J6 pad 5c: (no net) -> Net-(F13-Pad1)
- J6 pad 6a: (no net) -> Net-(J6-Pad6a)
- J6 pad 6b: (no net) -> GND
- J6 pad 6c: (no net) -> Net-(F13-Pad1)
- J6 pad 7a: (no net) -> GND
- J6 pad 7b: (no net) -> GND
- J6 pad 7c: (no net) -> Net-(F14-Pad1)
- J6 pad 8a: (no net) -> Net-(J6-Pad8a)
- J6 pad 8b: (no net) -> /SPI0_MOSI
- J6 pad 8c: (no net) -> Net-(F14-Pad1)
- J6 pad 9a: (no net) -> Net-(J6-Pad9a)
- J6 pad 9b: (no net) -> /SPI0_MISO
- J6 pad 9c: (no net) -> Net-(F15-Pad1)
- R18 pad 1: Net-(J4-Pad66) -> Net-(J4-Pad2a)
- R20 pad 1: Net-(J4-Pad67) -> Net-(J4-Pad3a)
- R21 pad 1: Net-(J4-Pad69) -> Net-(J4-Pad5a)
- R23 pad 1: Net-(J4-Pad70) -> Net-(J4-Pad6a)
- R24 pad 1: Net-(J4-Pad72) -> Net-(J4-Pad8a)
- R26 pad 1: Net-(J4-Pad73) -> Net-(J4-Pad9a)
- R27 pad 1: Net-(J5-Pad66) -> Net-(J5-Pad2a)
- R29 pad 1: Net-(J5-Pad67) -> Net-(J5-Pad3a)
- R30 pad 1: Net-(J5-Pad69) -> Net-(J5-Pad5a)
- R32 pad 1: Net-(J5-Pad70) -> Net-(J5-Pad6a)
- R33 pad 1: Net-(J5-Pad72) -> Net-(J5-Pad8a)
- R35 pad 1: Net-(J5-Pad73) -> Net-(J5-Pad9a)
- R36 pad 1: Net-(J6-Pad66) -> Net-(J6-Pad2a)
- R38 pad 1: Net-(J6-Pad67) -> Net-(J6-Pad3a)
- R39 pad 1: Net-(J6-Pad69) -> Net-(J6-Pad5a)
- R41 pad 1: Net-(J6-Pad70) -> Net-(J6-Pad6a)
- R42 pad 1: Net-(J6-Pad72) -> Net-(J6-Pad8a)
- R44 pad 1: Net-(J6-Pad73) -> Net-(J6-Pad9a)
