File: kicad_hiltop_63hp_backplane/backplane_connector.sch (KiCad schematic (older format))
At the start: 66 parts

Commit message: PCI EXPRESS 96
Parts:
- removed C? (x3): 10nF, Capacitor_SMD:C_0402_1005Metric, symbol device:C
- removed R24, R25, R26, R27, R28, R29, R31, R80, R81, R82: 100, Resistor_SMD:R_0402_1005Metric, symbol device:R
- removed R44, R45, R46, R47, R48, R49, R50, R51, R52, R53, R54, R55, R58, R59, R66, R67, R68, R69, R70, R71: 150, Resistor_SMD:R_0402_1005Metric, symbol device:R
- removed U? (x3): LTC4311, Package_DFN_QFN:DFN-6-1EP_2x2mm_P0.5mm_EP0.61x1.42mm, symbol gti_Lattice:LTC4311
- added C? (x2): 10nF, Capacitor_SMD:C_0402_1005Metric, symbol device:C
- added R? (x4): 150, Resistor_SMD:R_0402_1005Metric, symbol device:R
- added R? (x2): 100, Resistor_SMD:R_0402_1005Metric, symbol device:R
- added U? (x2): LTC4311, Package_DFN_QFN:DFN-6-1EP_2x2mm_P0.5mm_EP0.61x1.42mm, symbol gti_Lattice:LTC4311
- gave numbers to parts that had none: 3
Connections:
- net labels added: +12V0, +3V3, +3V3V, +5V0, -5V0, FPGA_GPIO1, FPGA_GPIO10, FPGA_GPIO11, FPGA_GPIO12, FPGA_GPIO13, FPGA_GPIO14, FPGA_GPIO15, FPGA_GPIO16, FPGA_GPIO17, FPGA_GPIO18, FPGA_GPIO19, FPGA_GPIO2, FPGA_GPIO20, FPGA_GPIO21, FPGA_GPIO22, FPGA_GPIO23, FPGA_GPIO24, FPGA_GPIO25, FPGA_GPIO26, FPGA_GPIO27, FPGA_GPIO28, FPGA_GPIO29, FPGA_GPIO3, FPGA_GPIO30, FPGA_GPIO4, FPGA_GPIO5, FPGA_GPIO6, FPGA_GPIO7, FPGA_GPIO8, FPGA_GPIO9, I2C0_SCL, I2C0_SDA, I2C1_SCL, I2C1_SDA, LCOM1, LCOM2, LCOM3, LCOM4, LCOM5, LCOM6, LCOM7, LCOM8, MBRD_GPIO1, MBRD_GPIO10, MBRD_GPIO11, MBRD_GPIO12, MBRD_GPIO13, MBRD_GPIO14, MBRD_GPIO15, MBRD_GPIO16, MBRD_GPIO17, MBRD_GPIO18, MBRD_GPIO19, MBRD_GPIO2, MBRD_GPIO20, MBRD_GPIO21, MBRD_GPIO22, MBRD_GPIO23, MBRD_GPIO24, MBRD_GPIO25, MBRD_GPIO26, MBRD_GPIO27, MBRD_GPIO28, MBRD_GPIO29, MBRD_GPIO3, MBRD_GPIO30, MBRD_GPIO4, MBRD_GPIO5, MBRD_GPIO6, MBRD_GPIO7, MBRD_GPIO8, MBRD_GPIO9, PSEL_0, PSEL_1, PSEL_2, PWM0, PWM1, PWM2, PWM3, PWM5, PWM6, RCOM1, RCOM1A, RCOM1B, RCOM2, RCOM2A, RCOM2B, RCOM3, RCOM3A, RCOM3B, RCOM4, RCOM4A, RCOM4B, RCOM5, RCOM5A, RCOM5B, RCOM6, RCOM6A, RCOM6B, RCOM7, RCOM7A, RCOM7B, RCOM8, RCOM8A, RCOM8B, RESERVED_1, RESERVED_2, RESERVED_3, RESET, SHUTDOWN, SPI0_CS0, SPI0_CS1, SPI0_MISO, SPI0_MOSI, SPI0_SCK, SPI1_CS0, SPI1_CS1, SPI1_MISO, SPI1_MOSI, SPI1_SCK, SYS_CLK_0, SYS_CLK_1, SYS_CLK_2, SYS_TRIG_0, SYS_TRIG_1, SYS_TRIG_2, USB_N, USB_P, V_ADJ
- net labels removed: +3V3_IN, CON_SCL1, CON_SCL2, CON_SCL3, CON_SDA1, CON_SDA2, CON_SDA3, D1+, D1-, D10+, D10-, D11+, D11-, D12+, D12-, D13+, D13-, D14+, D14-, D15+, D15-, D16+, D16-, D2+, D2-, D3+, D3-, D4+, D4-, D5+, D5-, D6+, D6-, D7+, D7-, D8+, D8-, D9+, D9-, DCK+, DCK-, LVDS_D10+, LVDS_D10-, LVDS_D11+, LVDS_D11-, LVDS_D12+, LVDS_D12-, LVDS_D13+, LVDS_D13-, LVDS_D14+, LVDS_D14-, LVDS_D15+, LVDS_D15-, LVDS_D16+, LVDS_D16-, LVDS_D7+, LVDS_D7-, LVDS_D8+, LVDS_D8-, LVDS_D9+, LVDS_D9-
- wire segments 329 -> 476
Other:
- note removed: "Differential Signals/Clock\n"
- moved on the sheet: J15B, J16B, J17B, R18, R19, R20, R21, R22, R23, R30, R32, R33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

Commit message: back plane connector update
Parts:
- added F? (x15): Polyfuse, symbol device:Polyfuse
Connections:
- net PWM2 is gone; now on net PWM0: J16.22c (86)
- net PWM3 is gone; now on net PWM1: J16.23c (87)
- net PWM5 is gone; now on net PWM0: J17.22c (86)
- net PWM6 is gone; now on net PWM1: J17.23c (87)
- net +12V0: now also F?.2, F?.2, F?.2; no longer J15.1c (65), J15.2c (66), J16.1c (65), J16.2c (66), J17.1c (65), J17.2c (66)
- net +3V3V: now also F?.2, F?.2, F?.2; no longer J15.7c (71), J15.8c (72), J16.7c (71), J16.8c (72), J17.7c (71), J17.8c (72)
- net +5V0: now also F?.2, F?.2, F?.2; no longer J15.3c (67), J15.4c (68), J16.3c (67), J16.4c (68), J17.3c (67), J17.4c (68)
- net -5V0: now also F?.2, F?.2, F?.2; no longer J15.5c (69), J15.6c (70), J16.5c (69), J16.6c (70), J17.5c (69), J17.6c (70)
- net V_ADJ: now also F?.2, F?.2, F?.2; no longer J15.10c (74), J15.9c (73), J16.10c (74), J16.9c (73), J17.10c (74), J17.9c (73)
- new net: F?.1, J17.10c (74), J17.9c (73)
- new net: F?.1, J17.1c (65), J17.2c (66)
- new net: F?.1, J17.3c (67), J17.4c (68)
- new net: F?.1, J17.5c (69), J17.6c (70)
- new net: F?.1, J17.7c (71), J17.8c (72)
- new net: F?.1, J16.10c (74), J16.9c (73)
- new net: F?.1, J16.1c (65), J16.2c (66)
- new net: F?.1, J16.3c (67), J16.4c (68)
- new net: F?.1, J16.5c (69), J16.6c (70)
- new net: F?.1, J16.7c (71), J16.8c (72)
- new net: F?.1, J15.10c (74), J15.9c (73)
- new net: F?.1, J15.1c (65), J15.2c (66)
- new net: F?.1, J15.3c (67), J15.4c (68)
- new net: F?.1, J15.5c (69), J15.6c (70)
- new net: F?.1, J15.7c (71), J15.8c (72)
Changed lines of the file:
@@
 Wire Wire Line
 	1575 1325 1575 1475
-Text HLabel 775  1475 3    60   Input ~ 0
+Text HLabel 775  1925 3    60   Input ~ 0
 +12V0
-Text HLabel 975  1475 3    60   Input ~ 0
+Text HLabel 975  1925 3    60   Input ~ 0
 +5V0
-Text HLabel 1375 1475 3    60   Input ~ 0
+Text HLabel 1375 1925 3    60   Input ~ 0
 +3V3V
-Text HLabel 1175 1475 3    60   Input ~ 0
+Text HLabel 1175 1925 3    60   Input ~ 0
 -5V0
-Text HLabel 1575 1475 3    60   Input ~ 0
+Text HLabel 1575 1925 3    60   Input ~ 0
 V_ADJ
 Wire Wire Line
@@
 Wire Wire Line
 	5100 1325 5100 1475
-Text HLabel 4300 1475 3    60   Input ~ 0
-+12V0
-Text HLabel 4500 1475 3    60   Input ~ 0
-+5V0
-Text HLabel 4900 1475 3    60   Input ~ 0
-+3V3V
-Text HLabel 4700 1475 3    60   Input ~ 0
--5V0
-Text HLabel 5100 1475 3    60   Input ~ 0
-V_ADJ
 Wire Wire Line
 	7825 1175 7825 1325
@@
 Wire Wire Line
 	8625 1325 8625 1475
-Text HLabel 7825 1475 3    60   Input ~ 0
-+12V0
-Text HLabel 8025 1475 3    60   Input ~ 0
-+5V0
-Text HLabel 8425 1475 3    60   Input ~ 0
-+3V3V
-Text HLabel 8225 1475 3    60   Input ~ 0
--5V0
-Text HLabel 8625 1475 3    60   Input ~ 0
-V_ADJ
 Wire Wire Line
 	1875 1175 1875 1475
@@
 Text HLabel 9650 3325 3    60   Input ~ 0
 RESERVED_3
-Text HLabel 6125 3325 3    60   Input ~ 0
-RESERVED_2
 Text HLabel 2600 3325 3    60   Input ~ 0
 RESERVED_1
@@
 PWM1
 Text HLabel 6400 1500 3    60   Input ~ 0
-PWM2
+PWM0
 Text HLabel 6500 1500 3    60   Input ~ 0
-PWM3
+PWM1
 Text HLabel 9925 1500 3    60   Input ~ 0
-PWM5
+PWM0
 Text HLabel 10025 1500 3    60   Input ~ 0
-PWM6
+PWM1
 $Comp
 L gti_Lattice:LTC4311 U?
@@
 Wire Wire Line
 	7950 5550 7950 5450
+$Comp
+L device:Polyfuse F?
+U 1 1 60455C00
+P 775 1625
+F 0 "F?" V 725 1750 50  0000 L CNN
+F 1 "Polyfuse" V 863 1580 50  0000 L CNN
+F 2 "" H 825 1425 50  0001 L CNN
+F 3 "" H 775 1625 50  0001 C CNN
+	1    775  1625
+	1    0    0    -1
+$EndComp
+Wire Wire Line
+	775  1925 775  1775
+$Comp
+L device:Polyfuse F?
+U 1 1 604A6423
+P 975 1625
+F 0 "F?" V 925 1750 50  0000 L CNN
+F 1 "Polyfuse" V 1063 1580 50  0000 L CNN
+F 2 "" H 1025 1425 50  0001 L CNN
+F 3 "" H 975 1625 50  0001 C CNN
+	1    975  1625
+	1    0    0    -1
+$EndComp
+$Comp
+L device:Polyfuse F?
+U 1 1 604A6497
+P 1175 1625
+F 0 "F?" V 1125 1750 50  0000 L CNN
+F 1 "Polyfuse" V 1263 1580 50  0000 L CNN
+F 2 "" H 1225 1425 50  0001 L CNN
+F 3 "" H 1175 1625 50  0001 C CNN
+	1    1175 1625
+	1    0    0    -1
+$EndComp
+$Comp
+L device:Polyfuse F?
+U 1 1 604A664B
+P 1375 1625
+F 0 "F?" V 1325 1750 50  0000 L CNN
+F 1 "Polyfuse" V 1463 1580 50  0000 L CNN
+F 2 "" H 1425 1425 50  0001 L CNN
+F 3 "" H 1375 1625 50  0001 C CNN
+	1    1375 1625
+	1    0    0    -1
+$EndComp
+$Comp
+L device:Polyfuse F?
+U 1 1 604A66C3
+P 1575 1625
+F 0 "F?" V 1525 1750 50  0000 L CNN
+F 1 "Polyfuse" V 1663 1580 50  0000 L CNN
+F 2 "" H 1625 1425 50  0001 L CNN
+F 3 "" H 1575 1625 50  0001 C CNN
+	1    1575 1625
+	1    0    0    -1
+$EndComp
+Wire Wire Line
+	975  1775 975  1925
+Wire Wire Line
+	1175 1775 1175 1925
+Wire Wire Line
+	1375 1775 1375 1925
+Wire Wire Line
+	1575 1775 1575 1925
+Text HLabel 4300 1925 3    60   Input ~ 0
++12V0
+Text HLabel 4500 1925 3    60   Input ~ 0
++5V0
+Text HLabel 4900 1925 3    60   Input ~ 0
++3V3V
+Text HLabel 4700 1925 3    60   Input ~ 0
+-5V0
+Text HLabel 5100 1925 3    60   Input ~ 0
+V_ADJ
+$Comp
+L device:Polyfuse F?
+U 1 1 6073C287
+P 4300 1625
+F 0 "F?" V 4250 1750 50  0000 L CNN
+F 1 "Polyfuse" V 4388 1580 50  0000 L CNN
+F 2 "" H 4350 1425 50  0001 L CNN
+F 3 "" H 4300 1625 50  0001 C CNN
+	1    4300 1625
+	1    0    0    -1
+$EndComp
+Wire Wire Line
+	4300 1925 4300 1775
+$Comp
+L device:Polyfuse F?
+U 1 1 6073C28F
+P 4500 1625
+F 0 "F?" V 4450 1750 50  0000 L CNN
+F 1 "Polyfuse" V 4588 1580 50  0000 L CNN
+F 2 "" H 4550 1425 50  0001 L CNN
+F 3 "" H 4500 1625 50  0001 C CNN
+	1    4500 1625
+	1    0    0    -1
+$EndComp
+$Comp
+L device:Polyfuse F?
+U 1 1 6073C296
+P 4700 1625
+F 0 "F?" V 4650 1750 50  0000 L CNN
+F 1 "Polyfuse" V 4788 1580 50  0000 L CNN
+F 2 "" H 4750 1425 50  0001 L CNN
+F 3 "" H 4700 1625 50  0001 C CNN
+	1    4700 1625
+	1    0    0    -1
+$EndComp
+$Comp
+L device:Polyfuse F?
+U 1 1 6073C29D
+P 4900 1625
+F 0 "F?" V 4850 1750 50  0000 L CNN
+F 1 "Polyfuse" V 4988 1580 50  0000 L CNN
+F 2 "" H 4950 1425 50  0001 L CNN
+F 3 "" H 4900 1625 50  0001 C CNN
+	1    4900 1625
+	1    0    0    -1
+$EndComp
+$Comp
+L device:Polyfuse F?
+U 1 1 6073C2A4
+P 5100 1625
+F 0 "F?" V 5050 1750 50  0000 L CNN
+F 1 "Polyfuse" V 5188 1580 50  0000 L CNN
+F 2 "" H 5150 1425 50  0001 L CNN
+F 3 "" H 5100 1625 50  0001 C CNN
+	1    5100 1625
+	1    0    0    -1
+$EndComp
+Wire Wire Line
+	4500 1775 4500 1925
+Wire Wire Line
+	4700 1775 4700 1925
+Wire Wire Line
+	4900 1775 4900 1925
+Wire Wire Line
+	5100 1775 5100 1925
+Text HLabel 7825 1925 3    60   Input ~ 0
++12V0
+Text HLabel 8025 1925 3    60   Input ~ 0
++5V0
+Text HLabel 8425 1925 3    60   Input ~ 0
++3V3V
+Text HLabel 8225 1925 3    60   Input ~ 0
+-5V0
+Text HLabel 8625 1925 3    60   Input ~ 0
+V_ADJ
+$Comp
+L device:Polyfuse F?
+U 1 1 60790ED9
+P 7825 1625
+F 0 "F?" V 7775 1750 50  0000 L CNN
+F 1 "Polyfuse" V 7913 1580 50  0000 L CNN
+F 2 "" H 7875 1425 50  0001 L CNN
+F 3 "" H 7825 1625 50  0001 C CNN
+	1    7825 1625
+	1    0    0    -1
+$EndComp
+Wire Wire Line
+	7825 1925 7825 1775
+$Comp
+L device:Polyfuse F?
+U 1 1 60790EE1
+P 8025 1625
+F 0 "F?" V 7975 1750 50  0000 L CNN
+F 1 "Polyfuse" V 8113 1580 50  0000 L CNN
+F 2 "" H 8075 1425 50  0001 L CNN
+F 3 "" H 8025 1625 50  0001 C CNN
+	1    8025 1625
+	1    0    0    -1
+$EndComp
+$Comp
+L device:Polyfuse F?
+U 1 1 60790EE8
+P 8225 1625
+F 0 "F?" V 8175 1750 50  0000 L CNN
+F 1 "Polyfuse" V 8313 1580 50  0000 L CNN
+F 2 "" H 8275 1425 50  0001 L CNN
+F 3 "" H 8225 1625 50  0001 C CNN
+	1    8225 1625
+	1    0    0    -1
+$EndComp
+$Comp
+L device:Polyfuse F?
+U 1 1 60790EEF
+P 8425 1625
+F 0 "F?" V 8375 1750 50  0000 L CNN
+F 1 "Polyfuse" V 8513 1580 50  0000 L CNN
+F 2 "" H 8475 1425 50  0001 L CNN
+F 3 "" H 8425 1625 50  0001 C CNN
+	1    8425 1625
+	1    0    0    -1
+$EndComp
+$Comp
+L device:Polyfuse F?
+U 1 1 60790EF6
+P 8625 1625
+F 0 "F?" V 8575 1750 50  0000 L CNN
+F 1 "Polyfuse" V 8713 1580 50  0000 L CNN
+F 2 "" H 8675 1425 50  0001 L CNN
+F 3 "" H 8625 1625 50  0001 C CNN
+	1    8625 1625
+	1    0    0    -1
+$EndComp
+Wire Wire Line
+	8025 1775 8025 1925
+Wire Wire Line
+	8225 1775 8225 1925
+Wire Wire Line
+	8425 1775 8425 1925
+Wire Wire Line
+	8625 1775 8625 1925
+Text HLabel 6125 3325 3    60   Input ~ 0
+RESERVED_2
 $EndSCHEMATC

Commit message: Added new PCB outline for the backplane
Parts:
- C19, C20: renamed from C?; symbol device:C -> hiltop_backplane_brd-rescue:C-device
- F1, F12, F13, F14, F15, F16, F17, F18, F2, F3, F4, F5, F6, F7, F8: renamed from F?; symbol device:Polyfuse -> hiltop_backplane_brd-rescue:Polyfuse-device
- J15, J16, J17: footprint (none) -> Connectors_IEC_DIN:Socket_DIN41612-CaseC1-full-Female-96Pin-3rows; symbol gti_Lattice:CONN_DIN_HDR_96POS -> hiltop_backplane_brd-rescue:CONN_DIN_HDR_96POS-gti_Lattice
- R18, R19, R20, R21, R22, R23, R30, R32, R33, R34, R35, R36, R37, R38, R39, R40, R41, R42, R43, R56, R57: symbol device:R -> hiltop_backplane_brd-rescue:R-device
- R24, R25, R26, R27, R28, R29: renamed from R?; symbol device:R -> hiltop_backplane_brd-rescue:R-device
- U2, U3: renamed from U?; symbol gti_Lattice:LTC4311 -> hiltop_backplane_brd-rescue:LTC4311-gti_Lattice

Commit message: first pass draft for review
Parts:
- removed unit 3 of J15
- removed unit 2 of J15
- removed unit 3 of J16
- removed unit 2 of J16
- removed unit 3 of J17
- removed unit 2 of J17
- added unit 2 of J15
- added unit 3 of J15
- added unit 2 of J16
- added unit 3 of J16
- added unit 2 of J17
- added unit 3 of J17
- C19, C20: symbol hiltop_backplane_brd-rescue:C-device -> device:C
- F1, F12, F13, F14, F15, F16, F17, F18, F2, F3, F4, F5, F6, F7, F8: symbol hiltop_backplane_brd-rescue:Polyfuse-device -> device:Polyfuse
- J15, J16, J17: footprint Connectors_IEC_DIN:Socket_DIN41612-CaseC1-full-Female-96Pin-3rows -> (none); symbol hiltop_backplane_brd-rescue:CONN_DIN_HDR_96POS-gti_Lattice -> gti_Lattice:CONN_DIN_HDR_96POS
- R18, R19, R20, R21, R22, R23, R24, R25, R26, R27, R28, R29, R30, R32, R33, R34, R35, R36, R37, R38, R39, R40, R41, R42, R43, R56, R57: symbol hiltop_backplane_brd-rescue:R-device -> device:R
- U2, U3: symbol hiltop_backplane_brd-rescue:LTC4311-gti_Lattice -> gti_Lattice:LTC4311
Connections:
- net labels added: SPI1_CS2, SYS_CLK, SYS_TRIG, USB1_N, USB1_P, USB2_N, USB2_P, USB3_N, USB3_P
- net labels removed: MBRD_GPIO11, MBRD_GPIO12, MBRD_GPIO13, MBRD_GPIO14, MBRD_GPIO15, MBRD_GPIO16, MBRD_GPIO17, MBRD_GPIO18, MBRD_GPIO19, MBRD_GPIO20, MBRD_GPIO21, MBRD_GPIO22, MBRD_GPIO23, MBRD_GPIO24, MBRD_GPIO25, MBRD_GPIO26, MBRD_GPIO27, MBRD_GPIO28, MBRD_GPIO29, MBRD_GPIO30, RESERVED_1, RESERVED_2, RESERVED_3, SYS_CLK_0, SYS_CLK_1, SYS_CLK_2, SYS_TRIG_0, SYS_TRIG_1, SYS_TRIG_2, USB_N, USB_P
