File: kicad_hiltop_63hp_backplane/MotherBoard_Connector.sch (KiCad schematic (older format))
At the start: 12 parts

Commit message: PCI EXPRESS 96
Parts:
- added C?: 10nF, Capacitor_SMD:C_0402_1005Metric, symbol device:C
- added R? (x20): 150, Resistor_SMD:R_0402_1005Metric, symbol device:R
- added R? (x10): 100, Resistor_SMD:R_0402_1005Metric, symbol device:R
- added U?: LTC4311, Package_DFN_QFN:DFN-6-1EP_2x2mm_P0.5mm_EP0.61x1.42mm, symbol gti_Lattice:LTC4311
- gave numbers to parts that had none: 12
Connections:
- net labels added: +3V3_IN, CON_SCL3, CON_SDA3, D13+, D13-, D14+, D14-, D15+, D15-, D16+, D16-, LVDS_D10+, LVDS_D10-, LVDS_D11+, LVDS_D11-, LVDS_D12+, LVDS_D12-, LVDS_D13+, LVDS_D13-, LVDS_D14+, LVDS_D14-, LVDS_D15+, LVDS_D15-, LVDS_D16+, LVDS_D16-, LVDS_D7+, LVDS_D7-, LVDS_D8+, LVDS_D8-, LVDS_D9+, LVDS_D9-
- wire segments 106 -> 207

Commit message: back plane connector update
Parts:
- removed C?: 10nF, Capacitor_SMD:C_0402_1005Metric, symbol device:C
- removed F1, F2, F3, F4, F5, F6, F7, F8: Polyfuse, symbol device:Polyfuse
- removed U?: LTC4311, Package_DFN_QFN:DFN-6-1EP_2x2mm_P0.5mm_EP0.61x1.42mm, symbol gti_Lattice:LTC4311
Connections:
- net labels removed: +3V3_IN, CON_SCL3, CON_SDA3
- wire segments 207 -> 187

Commit message: Added new PCB outline for the backplane
Parts:
- J11: symbol hiltop_pcie-64_conn:HILTOP_PCIE-64_CONN -> hiltop_backplane_brd-rescue:HILTOP_PCIE-64_CONN-hiltop_pcie-64_conn
- J12: symbol Connector1:Conn_02x04_Odd_Even -> hiltop_backplane_brd-rescue:Conn_02x04_Odd_Even-Connector1
- J13: symbol Connector1:Conn_02x02_Counter_Clockwise -> hiltop_backplane_brd-rescue:Conn_02x02_Counter_Clockwise-Connector1
- J14: symbol Connector1:Conn_01x02 -> hiltop_backplane_brd-rescue:Conn_01x02-Connector1
- R31, R44, R45, R46, R47, R48, R49, R50, R51, R52, R53, R54, R55, R58, R59, R66, R67, R68, R69, R70, R71, R75, R76, R77, R78, R79, R80, R81, R82, R83: renamed from R?; symbol device:R -> hiltop_backplane_brd-rescue:R-device

Commit message: first pass draft for review
Parts:
- added F? (x3): Polyfuse, symbol device:Polyfuse
- J11: symbol hiltop_backplane_brd-rescue:HILTOP_PCIE-64_CONN-hiltop_pcie-64_conn -> gti_Lattice:HILTOP_PCIE-64_CONN
- J12: symbol hiltop_backplane_brd-rescue:Conn_02x04_Odd_Even-Connector1 -> Connector1:Conn_02x04_Odd_Even
- J13: symbol hiltop_backplane_brd-rescue:Conn_02x02_Counter_Clockwise-Connector1 -> Connector1:Conn_02x02_Counter_Clockwise
- J14: symbol hiltop_backplane_brd-rescue:Conn_01x02-Connector1 -> Connector1:Conn_01x02
- R31, R44, R45, R46, R47, R48, R49, R50, R51, R52, R53, R54, R55, R58, R59, R66, R67, R68, R69, R70, R71, R75, R76, R77, R78, R79, R80, R81, R82, R83: symbol hiltop_backplane_brd-rescue:R-device -> device:R
Connections:
- net MBRD_GPIO16 is gone; now on net MBRD_GPIO15: J11.A31 (GPIO16)
- net +1V2: now also F?.1
- net +1V8: now also F?.2; no longer J13.2 (Pin_2)
- net +2V5: now also F?.2; no longer J13.1 (Pin_1)
- net GND: now also J11.B15 (GND), J11.B19 (GND); no longer J11.B16 (GPIO6/BCM27)
- net MBRD_GPIO14: now also J11.A30 (GPIO15); no longer J11.A29 (GPIO14)
- net MBRD_GPIO15: no longer J11.A30 (GPIO15)
- net MBRD_GPIO6: now also J11.B16 (GPIO6/BCM27); no longer J11.B17 (GPIO7/BCM28)
- net MBRD_GPIO7: now also J11.B17 (GPIO7/BCM28); no longer J11.B18 (GPIO8/BCM34)
- net MBRD_PWM8: now also J11.B18 (GPIO8/BCM34); no longer J11.B19 (GND)
- net at J13.4 (Pin_4): now also F?.2
- new net: F?.1, J13.1 (Pin_1)
- new net: F?.1, J13.2 (Pin_2)
- new net MBRD_SPI1_CS2: J11.A29 (GPIO14)
Changed lines of the file:
@@
 $Descr A4 11693 8268
 encoding utf-8
-Sheet 6 6
+Sheet 5 6
 Title ""
 Date ""
@@
 	2625 2675 2350 2675
 Wire Wire Line
-	2625 2975 2350 2975
-Wire Wire Line
-	2625 3075 2350 3075
-Wire Wire Line
-	2625 3175 2350 3175
-Wire Wire Line
 	2625 3275 2350 3275
 Wire Wire Line
@@
 Wire Wire Line
 	2500 1675 2500 1975
-Wire Wire Line
-	2500 2875 2500 3475
-Connection ~ 2500 2875
-Wire Wire Line
-	2500 2875 2625 2875
 Connection ~ 2500 3475
 Wire Wire Line
@@
 Text HLabel 2350 4375 0    60   Input ~ 0
 MBRD_GPIO13
-Text HLabel 4850 4175 2    60   Input ~ 0
+Text HLabel 4850 4275 2    60   Input ~ 0
 MBRD_GPIO14
-Text HLabel 4850 4275 2    60   Input ~ 0
+Text HLabel 4850 4375 2    60   Input ~ 0
 MBRD_GPIO15
-Text HLabel 4850 4375 2    60   Input ~ 0
-MBRD_GPIO16
 Wire Wire Line
 	4650 1175 4650 1475
@@
 Text HLabel 2350 2675 0    60   Input ~ 0
 MBRD_GPIO5
+Text HLabel 2350 2875 0    60   Input ~ 0
+MBRD_GPIO6
 Text HLabel 2350 2975 0    60   Input ~ 0
-MBRD_GPIO6
+MBRD_GPIO7
 Text HLabel 2350 3075 0    60   Input ~ 0
-MBRD_GPIO7
-Text HLabel 2350 3175 0    60   Input ~ 0
 MBRD_PWM8
 Text HLabel 2350 3275 0    60   Input ~ 0
@@
 -5V
 $Comp
-L hiltop_backplane_brd-rescue:HILTOP_PCIE-64_CONN-hiltop_pcie-64_conn J11
+L gti_Lattice:HILTOP_PCIE-64_CONN J11
 U 1 1 5C13457D
 P 3575 2725
@@
 Wire Wire Line
 	2350 2575 2625 2575
-Wire Wire Line
-	2500 1975 2500 2875
 Connection ~ 2500 1975
 Wire Wire Line
@@
 Connection ~ 4650 2175
 $Comp
-L hiltop_backplane_brd-rescue:Conn_02x04_Odd_Even-Connector1 J12
+L Connector1:Conn_02x04_Odd_Even J12
 U 1 1 5C155D60
 P 8400 1825
@@
 $EndComp
 $Comp
-L hiltop_backplane_brd-rescue:Conn_02x02_Counter_Clockwise-Connector1 J13
+L Connector1:Conn_02x02_Counter_Clockwise J13
 U 1 1 5C155E73
 P 8425 2700
-F 0 "J13" H 8475 2917 50  0000 C CNN
-F 1 "Conn_02x02_Counter_Clockwise" H 8475 2826 50  0000 C CNN
+F 0 "J13" H 8425 2800 50  0000 C CNN
+F 1 "Conn_02x02_Counter_Clockwise" H 8425 2925 50  0000 C CNN
 F 2 "" H 8425 2700 50  0001 C CNN
 F 3 "~" H 8425 2700 50  0001 C CNN
@@
 $EndComp
 $Comp
-L hiltop_backplane_brd-rescue:Conn_01x02-Connector1 J14
+L Connector1:Conn_01x02 J14
 U 1 1 5C155F47
 P 8475 3425
@@
 Wire Wire Line
 	8825 2800 8825 2875
-Text HLabel 7875 2700 0    60   Input ~ 0
+Text HLabel 7500 2700 0    60   Input ~ 0
 +2V5
-Text HLabel 7875 2800 0    60   Input ~ 0
+Text HLabel 7500 2800 0    60   Input ~ 0
 +1V8
 Text HLabel 9625 2700 2    60   Input ~ 0
@@
 	8725 2700 8950 2700
 $Comp
-L hiltop_backplane_brd-rescue:R-device R?
+L device:R R?
 U 1 1 602962E5
 P 6100 5100
@@
 $EndComp
 $Comp
-L hiltop_backplane_brd-rescue:R-device R?
+L device:R R?
 U 1 1 602962EC
 P 6100 5200
@@
 $EndComp
 $Comp
-L hiltop_backplane_brd-rescue:R-device R?
+L device:R R?
 U 1 1 602962F3
 P 6100 5300
@@
 $EndComp
 $Comp
-L hiltop_backplane_brd-rescue:R-device R?
+L device:R R?
 U 1 1 602962FA
 P 6100 5400
@@
 $EndComp
 $Comp
-L hiltop_backplane_brd-rescue:R-device R?
+L device:R R?
 U 1 1 60296301
 P 6100 5500
@@
 $EndComp
 $Comp
-L hiltop_backplane_brd-rescue:R-device R?
+L device:R R?
 U 1 1 60296308
 P 6100 5600
@@
 $EndComp
 $Comp
-L hiltop_backplane_brd-rescue:R-device R?
+L device:R R?
 U 1 1 6029630F
 P 6100 5700
@@
 $EndComp
 $Comp
-L hiltop_backplane_brd-rescue:R-device R?
+L device:R R?
 U 1 1 60296316
 P 6100 5800
@@
 $EndComp
 $Comp
-L hiltop_backplane_brd-rescue:R-device R?
+L device:R R?
 U 1 1 6029631D
 P 6100 6000
@@
 $EndComp
 $Comp
-L hiltop_backplane_brd-rescue:R-device R?
+L device:R R?
 U 1 1 60296324
 P 6100 6100
@@
 $EndComp
 $Comp
-L hiltop_backplane_brd-rescue:R-device R?
+L device:R R?
 U 1 1 6029632B
 P 6100 6200
@@
 $EndComp
 $Comp
-L hiltop_backplane_brd-rescue:R-device R?
+L device:R R?
 U 1 1 60296332
 P 6100 6300
@@
 $EndComp
 $Comp
-L hiltop_backplane_brd-rescue:R-device R?
+L device:R R?
 U 1 1 60296339
 P 6100 6800
@@
 $EndComp
 $Comp
-L hiltop_backplane_brd-rescue:R-device R?
+L device:R R?
 U 1 1 60296340
 P 6100 6900
@@
 $EndComp
 $Comp
-L hiltop_backplane_brd-rescue:R-device R?
+L device:R R?
 U 1 1 60296347
 P 6100 7075
@@
 $EndComp
 $Comp
-L hiltop_backplane_brd-rescue:R-device R?
+L device:R R?
 U 1 1 6029634E
 P 6100 7175
@@
 $EndComp
 $Comp
-L hiltop_backplane_brd-rescue:R-device R?
+L device:R R?
 U 1 1 60296355
 P 6100 7275
@@
 $EndComp
 $Comp
-L hiltop_backplane_brd-rescue:R-device R?
+L device:R R?
 U 1 1 6029635C
 P 6100 7375
@@
 $EndComp
 $Comp
-L hiltop_backplane_brd-rescue:R-device R?
+L device:R R?
 U 1 1 60296363
 P 6100 7475
@@
 $EndComp
 $Comp
-L hiltop_backplane_brd-rescue:R-device R?
+L device:R R?
 U 1 1 6029636A
 P 6100 7575
@@
 $EndComp
 $Comp
-L hiltop_backplane_brd-rescue:R-device R?
+L device:R R?
 U 1 1 60296371
 P 5650 5100
@@
 $EndComp
 $Comp
-L hiltop_backplane_brd-rescue:R-device R?
+L device:R R?
 U 1 1 60296378
 P 5650 5300
@@
 $EndComp
 $Comp
-L hiltop_backplane_brd-rescue:R-device R?
+L device:R R?
 U 1 1 6029637F
 P 5650 5500
@@
 $EndComp
 $Comp
-L hiltop_backplane_brd-rescue:R-device R?
+L device:R R?
 U 1 1 60296386
 P 5650 5700
@@
 $EndComp
 $Comp
-L hiltop_backplane_brd-rescue:R-device R?
+L device:R R?
 U 1 1 6029638D
 P 5650 6000
@@
 $EndComp
 $Comp
-L hiltop_backplane_brd-rescue:R-device R?
+L device:R R?
 U 1 1 60296394
 P 5650 6200
@@
 $EndComp
 $Comp
-L hiltop_backplane_brd-rescue:R-device R?
+L device:R R?
 U 1 1 6029639B
 P 5650 6900
@@
 $EndComp
 $Comp
-L hiltop_backplane_brd-rescue:R-device R?
+L device:R R?
 U 1 1 602963A2
 P 5650 7075
@@
 $EndComp
 $Comp
-L hiltop_backplane_brd-rescue:R-device R?
+L device:R R?
 U 1 1 602963A9
 P 5650 7275
@@
 $EndComp
 $Comp
-L hiltop_backplane_brd-rescue:R-device R?
+L device:R R?
 U 1 1 602963B0
 P 5650 7475
@@
 	5450 5700 5500 5700
 Wire Wire Line
-	7875 2700 8225 2700
-Wire Wire Line
-	7875 2800 8225 2800
-Wire Wire Line
 	7900 3425 8275 3425
 Wire Wire Line
@@
 Wire Wire Line
 	8700 2025 8925 2025
+$Comp
+L device:Polyfuse F?
+U 1 1 5C36D98A
+P 9100 2700
+F 0 "F?" V 8875 2700 50  0000 C CNN
+F 1 "Polyfuse" V 8966 2700 50  0000 C CNN
+F 2 "" H 9150 2500 50  0001 L CNN
+F 3 "" H 9100 2700 50  0001 C CNN
+	1    9100 2700
+	0    1    1    0
+$EndComp
+$Comp
+L device:Polyfuse F?
+U 1 1 5C36DB02
+P 7950 2700
+F 0 "F?" V 7850 2550 50  0000 C CNN
+F 1 "Polyfuse" V 7900 2425 50  0000 C CNN
+F 2 "" H 8000 2500 50  0001 L CNN
+F 3 "" H 7950 2700 50  0001 C CNN
+	1    7950 2700
+	0    1    1    0
+$EndComp
+$Comp
+L device:Polyfuse F?
+U 1 1 5C36DBE2
+P 7950 2800
+F 0 "F?" V 8075 2650 50  0000 C CNN
+F 1 "Polyfuse" V 8000 2525 50  0000 C CNN
+F 2 "" H 8000 2600 50  0001 L CNN
+F 3 "" H 7950 2800 50  0001 C CNN
+	1    7950 2800
+	0    1    1    0
+$EndComp
+Wire Wire Line
+	8100 2700 8225 2700
+Wire Wire Line
+	8100 2800 8225 2800
+Wire Wire Line
+	7500 2700 7800 2700
+Wire Wire Line
+	7500 2800 7800 2800
+Wire Wire Line
+	2500 1975 2500 2775
+Wire Wire Line
+	2625 2775 2500 2775
+Connection ~ 2500 2775
+Wire Wire Line
+	2500 2775 2500 3175
+Wire Wire Line
+	2625 3175 2500 3175
+Connection ~ 2500 3175
+Wire Wire Line
+	2500 3175 2500 3475
+Wire Wire Line
+	2625 2875 2350 2875
+Wire Wire Line
+	2625 2975 2350 2975
+Wire Wire Line
+	2625 3075 2350 3075
+Text HLabel 4850 4175 2    59   Input ~ 0
+MBRD_SPI1_CS2
 $EndSCHEMATC

Commit message: Schematic updated to reflect USB logic and Global nets changed to local nets, renamed signals in motherboard connector
Parts:
- removed R31, R44, R45, R46, R47, R48, R49, R50, R51, R52: 100, Resistor_SMD:R_0402_1005Metric, symbol device:R
- removed R53, R54, R55, R58, R59, R66, R67, R68, R69, R70, R71, R75, R76, R77, R78, R79, R80, R81, R82, R83: 150, Resistor_SMD:R_0402_1005Metric, symbol device:R
Connections:
- net MBRD_GPIO11 is gone; now on net MBRD_SPI1_CS2: J11.B29 (GPIO11)
- net MBRD_GPIO14: now also J11.A29 (GPIO14); no longer J11.A30 (GPIO15)
- net MBRD_GPIO15: now also J11.A30 (GPIO15); no longer J11.A31 (GPIO16)
- net MBRD_SPI1_CS2: no longer J11.A29 (GPIO14)
- net MBRD_PWM10 renamed MBRD_GPIO10
- net MBRD_PWM8 renamed MBRD_GPIO8
- net MBRD_PWM9 renamed MBRD_GPIO9
- new net MBRD_GPIO16: J11.A31 (GPIO16)

Commit message: lables connected to end of net, each component mapped to footprint, working on reducing error
Parts:
- J10: renamed from J14; footprint (none) -> Connector_Molex:Molex_Mini-Fit_Jr_5566-02A2_2x01_P4.20mm_Vertical
- J7: renamed from J11; footprint (none) -> GTI_Footprint_Lib:SO_DIMM_200
- J8: renamed from J12; footprint (none) -> Connector_Molex:Molex_Mini-Fit_Jr_5566-08A_2x04_P4.20mm_Vertical
- J9: renamed from J13; footprint (none) -> Connector_Molex:Molex_Mini-Fit_Jr_5566-04A_2x02_P4.20mm_Vertical
- R45: renamed from F?; value Polyfuse -> 0R; footprint (none) -> Resistor_SMD:R_0402_1005Metric
- R46, R47: renamed from F?; value Polyfuse -> 0R; footprint (none) -> Resistor_SMD:R_1206_3216Metric
Changed lines of the file:
@@
 Connection ~ 2500 4475
 $Comp
-L power:GND #PWR031
+L power:GND #PWR030
 U 1 1 5C0B72CD
 P 2500 4575
-F 0 "#PWR031" H 2500 4325 50  0001 C CNN
+F 0 "#PWR030" H 2500 4325 50  0001 C CNN
 F 1 "GND" H 2505 4402 50  0000 C CNN
 F 2 "" H 2500 4575 50  0001 C CNN
@@
 	4650 4475 4650 4575
 $Comp
-L power:GND #PWR032
+L power:GND #PWR031
 U 1 1 5C0C4F5C
 P 4650 4575
-F 0 "#PWR032" H 4650 4325 50  0001 C CNN
+F 0 "#PWR031" H 4650 4325 50  0001 C CNN
 F 1 "GND" H 4655 4402 50  0000 C CNN
 F 2 "" H 4650 4575 50  0001 C CNN
@@
 -5V
 $Comp
-L gti_Lattice:HILTOP_PCIE-64_CONN J11
+L gti_Lattice:HILTOP_PCIE-64_CONN J7
 U 1 1 5C13457D
 P 3575 2725
-F 0 "J11" H 3575 4640 50  0000 C CNN
+F 0 "J7" H 3575 4640 50  0000 C CNN
 F 1 "HILTOP_PCIE-64_CONN" H 3575 4549 50  0000 C CNN
-F 2 "" H 2925 4575 50  0001 C CNN
+F 2 "GTI_Footprint_Lib:SO_DIMM_200" H 2925 4575 50  0001 C CNN
 F 3 "" H 3075 4675 50  0001 C CNN
 	1    3575 2725
@@
 Connection ~ 4650 2175
 $Comp
-L Connector1:Conn_02x04_Odd_Even J12
+L Connector1:Conn_02x04_Odd_Even J8
 U 1 1 5C155D60
 P 8400 1825
-F 0 "J12" H 8450 2142 50  0000 C CNN
+F 0 "J8" H 8450 2142 50  0000 C CNN
 F 1 "Conn_02x04_Odd_Even" H 8450 2051 50  0000 C CNN
-F 2 "" H 8400 1825 50  0001 C CNN
+F 2 "Connector_Molex:Molex_Mini-Fit_Jr_5566-08A_2x04_P4.20mm_Vertical" H 8400 1825 50  0001 C CNN
 F 3 "~" H 8400 1825 50  0001 C CNN
 	1    8400 1825
@@
 $EndComp
 $Comp
-L Connector1:Conn_02x02_Counter_Clockwise J13
+L Connector1:Conn_02x02_Counter_Clockwise J9
 U 1 1 5C155E73
 P 8425 2700
-F 0 "J13" H 8425 2800 50  0000 C CNN
+F 0 "J9" H 8425 2800 50  0000 C CNN
 F 1 "Conn_02x02_Counter_Clockwise" H 8425 2925 50  0000 C CNN
-F 2 "" H 8425 2700 50  0001 C CNN
+F 2 "Connector_Molex:Molex_Mini-Fit_Jr_5566-04A_2x02_P4.20mm_Vertical" H 8425 2700 50  0001 C CNN
 F 3 "~" H 8425 2700 50  0001 C CNN
 	1    8425 2700
@@
 $EndComp
 $Comp
-L Connector1:Conn_01x02 J14
+L Connector1:Conn_01x02 J10
 U 1 1 5C155F47
 P 8475 3425
-F 0 "J14" H 8450 3600 50  0000 L CNN
+F 0 "J10" H 8450 3600 50  0000 L CNN
 F 1 "Conn_01x02" H 8275 3525 50  0000 L CNN
-F 2 "" H 8475 3425 50  0001 C CNN
+F 2 "Connector_Molex:Molex_Mini-Fit_Jr_5566-02A2_2x01_P4.20mm_Vertical" H 8475 3425 50  0001 C CNN
 F 3 "~" H 8475 3425 50  0001 C CNN
 	1    8475 3425
@@
 $EndComp
 $Comp
-L power:GND #PWR033
+L power:GND #PWR032
 U 1 1 5C1D8414
 P 8100 2125
-F 0 "#PWR033" H 8100 1875 50  0001 C CNN
+F 0 "#PWR032" H 8100 1875 50  0001 C CNN
 F 1 "GND" H 8105 1952 50  0000 C CNN
 F 2 "" H 8100 2125 50  0001 C CNN
@@
 +1V2
 $Comp
-L power:GND #PWR035
+L power:GND #PWR034
 U 1 1 5C1EE135
 P 8825 2875
-F 0 "#PWR035" H 8825 2625 50  0001 C CNN
+F 0 "#PWR034" H 8825 2625 50  0001 C CNN
 F 1 "GND" H 8830 2702 50  0000 C CNN
 F 2 "" H 8825 2875 50  0001 C CNN
@@
 VADJ_DC
 $Comp
-L power:GND #PWR034
+L power:GND #PWR033
 U 1 1 5C1F5843
 P 8150 3575
-F 0 "#PWR034" H 8150 3325 50  0001 C CNN
+F 0 "#PWR033" H 8150 3325 50  0001 C CNN
 F 1 "GND" H 8155 3402 50  0000 C CNN
 F 2 "" H 8150 3575 50  0001 C CNN
@@
 	8700 2025 8925 2025
 $Comp
-L device:Polyfuse F?
+L device:Polyfuse R47
 U 1 1 5C36D98A
 P 9100 2700
-F 0 "F?" V 8875 2700 50  0000 C CNN
-F 1 "Polyfuse" V 8966 2700 50  0000 C CNN
-F 2 "" H 9150 2500 50  0001 L CNN
+F 0 "R47" V 9025 2525 50  0000 C CNN
+F 1 "0R" V 9025 2700 50  0000 C CNN
+F 2 "Resistor_SMD:R_1206_3216Metric" H 9150 2500 50  0001 L CNN
 F 3 "" H 9100 2700 50  0001 C CNN
 	1    9100 2700
@@
 $EndComp
 $Comp
-L device:Polyfuse F?
+L device:Polyfuse R45
 U 1 1 5C36DB02
 P 7950 2700
-F 0 "F?" V 7850 2550 50  0000 C CNN
-F 1 "Polyfuse" V 7900 2425 50  0000 C CNN
-F 2 "" H 8000 2500 50  0001 L CNN
+F 0 "R45" V 7850 2550 50  0000 C CNN
+F 1 "0R" V 7875 2700 50  0000 C CNN
+F 2 "Resistor_SMD:R_0402_1005Metric" H 8000 2500 50  0001 L CNN
 F 3 "" H 7950 2700 50  0001 C CNN
 	1    7950 2700
@@
 $EndComp
 $Comp
-L device:Polyfuse F?
+L device:Polyfuse R46
 U 1 1 5C36DBE2
 P 7950 2800
-F 0 "F?" V 8075 2650 50  0000 C CNN
-F 1 "Polyfuse" V 8000 2525 50  0000 C CNN
-F 2 "" H 8000 2600 50  0001 L CNN
+F 0 "R46" V 8075 2650 50  0000 C CNN
+F 1 "0R" V 8025 2800 50  0000 C CNN
+F 2 "Resistor_SMD:R_1206_3216Metric" H 8000 2600 50  0001 L CNN
 F 3 "" H 7950 2800 50  0001 C CNN
 	1    7950 2800

Commit message: first pass schematic placement
Parts:
- J7: footprint GTI_Footprint_Lib:SO_DIMM_200 -> GTI_Footprint_Lib:CONN PCI EXP FEMALE 64POS 0.039
- R45: footprint Resistor_SMD:R_0402_1005Metric -> Resistor_SMD:R_0603_1608Metric
Changed lines of the file:
@@
 F 0 "J7" H 3575 4640 50  0000 C CNN
 F 1 "HILTOP_PCIE-64_CONN" H 3575 4549 50  0000 C CNN
-F 2 "GTI_Footprint_Lib:SO_DIMM_200" H 2925 4575 50  0001 C CNN
+F 2 "GTI_Footprint_Lib:CONN PCI EXP FEMALE 64POS 0.039" H 2925 4575 50  0001 C CNN
 F 3 "" H 3075 4675 50  0001 C CNN
 	1    3575 2725
@@
 F 0 "R45" V 7850 2550 50  0000 C CNN
 F 1 "0R" V 7875 2700 50  0000 C CNN
-F 2 "Resistor_SMD:R_0402_1005Metric" H 8000 2500 50  0001 L CNN
+F 2 "Resistor_SMD:R_0603_1608Metric" H 8000 2500 50  0001 L CNN
 F 3 "" H 7950 2700 50  0001 C CNN
 	1    7950 2700

Commit message: routing os SODIM and GPIO
Connections:
- net MBRD_RESERVED_2 renamed MBRD_RESERVED_2+
- net MBRD_RESERVED_3 renamed MBRD_RESERVED_2-
Changed lines of the file:
@@
 MBRD_RESERVED_1
 Text HLabel 4850 2675 2    60   Input ~ 0
-MBRD_RESERVED_2
+MBRD_RESERVED_2+
 Text HLabel 4850 2775 2    60   Input ~ 0
-MBRD_RESERVED_3
+MBRD_RESERVED_2-
 Text HLabel 4850 1575 2    60   Input ~ 0
 MBRD_PSEL_0
