File: kicad_hiltop_63hp_backplane/USB_FTDI.sch (KiCad schematic (older format))
At the start: 53 parts, among them J1 USB_B_Micro, J2 3pos_Jumper, J3 3pos_Jumper, U5 93LCxxC, U6 FT2232H, Y1 ABM10AIG-12.000MHZ-4Z-T3

Commit message: PCI EXPRESS 96
Parts:
- gave numbers to parts that had none: 1
Changed lines of the file:
@@
 $Descr A4 11693 8268
 encoding utf-8
-Sheet 3 6
+Sheet 2 6
 Title ""
 Date ""
@@
 +3V3_IN
 $Comp
-L Connector:TestPoint TP?
+L Connector:TestPoint TP1
 U 1 1 5D0D4D61
 P 5400 2050
-F 0 "TP?" V 5425 2300 50  0000 C CNN
+F 0 "TP1" V 5425 2300 50  0000 C CNN
 F 1 "+1V8_REG_OUT" V 5350 2525 50  0000 C CNN
 F 2 "" H 5600 2050 50  0001 C CNN

Commit message: Added new PCB outline for the backplane
Parts:
- C22, C23, C24, C25, C26, C27, C28, C29, C30, C31, C32, C33, C34, C35, C36, C37, C38, C39, C40: symbol device:C -> hiltop_backplane_brd-rescue:C-device
- D2: symbol device:D_Schottky -> hiltop_backplane_brd-rescue:D_Schottky-device
- D3: symbol ESD_Protection:NUP2105L -> hiltop_backplane_brd-rescue:NUP2105L-ESD_Protection
- D4, D5: symbol device:LED -> hiltop_backplane_brd-rescue:LED-device
- J1: symbol Connector1:USB_B_Micro -> hiltop_backplane_brd-rescue:USB_B_Micro-Connector1
- J2, J3: symbol gti_Lattice:3pos_Jumper -> hiltop_backplane_brd-rescue:3pos_Jumper-gti_Lattice
- L1, L2, L3, L4, L5: symbol device:Ferrite_Bead -> hiltop_backplane_brd-rescue:Ferrite_Bead-device
- R110, R111, R112, R113, R114, R115, R116, R117, R118, R119, R120, R121, R122, R123, R124, R125, R126: symbol device:R -> hiltop_backplane_brd-rescue:R-device
- TP1: symbol Connector:TestPoint -> hiltop_backplane_brd-rescue:TestPoint-Connector
- TP11: symbol Connector1:Test_Point -> hiltop_backplane_brd-rescue:Test_Point-Connector1
- U5: symbol memory:93LCxxC -> hiltop_backplane_brd-rescue:93LCxxC-memory
- U6: symbol ftdi:FT2232H -> hiltop_backplane_brd-rescue:FT2232H-ftdi
- Y1: symbol device:Crystal_GND24 -> hiltop_backplane_brd-rescue:Crystal_GND24-device
Changed lines of the file:
@@
 $EndDescr
 $Comp
-L Connector1:USB_B_Micro J1
+L hiltop_backplane_brd-rescue:USB_B_Micro-Connector1 J1
 U 1 1 5A0CEDE1
 P 1550 2750
@@
 $EndComp
 $Comp
-L ESD_Protection:NUP2105L D3
+L hiltop_backplane_brd-rescue:NUP2105L-ESD_Protection D3
 U 1 1 5A0CEFF4
 P 4500 3150
@@
 $EndComp
 $Comp
-L device:C C22
+L hiltop_backplane_brd-rescue:C-device C22
 U 1 1 5A0CF19D
 P 2250 1500
@@
 $EndComp
 $Comp
-L device:C C23
+L hiltop_backplane_brd-rescue:C-device C23
 U 1 1 5A0CF48E
 P 3150 4800
@@
 $EndComp
 $Comp
-L device:C C37
+L hiltop_backplane_brd-rescue:C-device C37
 U 1 1 5A0CF61F
 P 8850 1250
@@
 $EndComp
 $Comp
-L device:C C39
+L hiltop_backplane_brd-rescue:C-device C39
 U 1 1 5A0CF7C6
 P 9450 1250
@@
 $EndComp
 $Comp
-L device:C C36
+L hiltop_backplane_brd-rescue:C-device C36
 U 1 1 5A0CF9B8
 P 8550 1250
@@
 $EndComp
 $Comp
-L device:C C40
+L hiltop_backplane_brd-rescue:C-device C40
 U 1 1 5A0CFC0B
 P 9750 1250
@@
 $EndComp
 $Comp
-L device:C C35
+L hiltop_backplane_brd-rescue:C-device C35
 U 1 1 5A0CFCE6
 P 8250 1250
@@
 $EndComp
 $Comp
-L device:C C34
+L hiltop_backplane_brd-rescue:C-device C34
 U 1 1 5A0CFD9F
 P 7950 1250
@@
 $EndComp
 $Comp
-L device:C C27
+L hiltop_backplane_brd-rescue:C-device C27
 U 1 1 5A0CFDD2
 P 5550 1200
@@
 $EndComp
 $Comp
-L device:C C30
+L hiltop_backplane_brd-rescue:C-device C30
 U 1 1 5A0CFE07
 P 5850 1200
@@
 $EndComp
 $Comp
-L device:C C32
+L hiltop_backplane_brd-rescue:C-device C32
 U 1 1 5A0CFE36
 P 6150 1200
@@
 $EndComp
 $Comp
-L device:C C33
+L hiltop_backplane_brd-rescue:C-device C33
 U 1 1 5A0CFE71
 P 6450 1200
@@
 $EndComp
 $Comp
-L device:C C38
+L hiltop_backplane_brd-rescue:C-device C38
 U 1 1 5A0CFEAA
 P 9150 1250
@@
 $EndComp
 $Comp
-L device:C C25
+L hiltop_backplane_brd-rescue:C-device C25
 U 1 1 5A0CFFD0
 P 5500 2300
@@
 $EndComp
 $Comp
-L device:C C29
+L hiltop_backplane_brd-rescue:C-device C29
 U 1 1 5A0D0317
 P 5750 2300
@@
 $EndComp
 $Comp
-L device:C C26
+L hiltop_backplane_brd-rescue:C-device C26
 U 1 1 5A0D035A
 P 5500 5850
@@
 $EndComp
 $Comp
-L device:C C24
+L hiltop_backplane_brd-rescue:C-device C24
 U 1 1 5A0D03B9
 P 4950 5850
@@
 $EndComp
 $Comp
-L device:Ferrite_Bead L2
+L hiltop_backplane_brd-rescue:Ferrite_Bead-device L2
 U 1 1 5A0D0483
 P 4850 650
@@
 $EndComp
 $Comp
-L device:Ferrite_Bead L3
+L hiltop_backplane_brd-rescue:Ferrite_Bead-device L3
 U 1 1 5A0D07F0
 P 4850 950
@@
 $EndComp
 $Comp
-L device:Ferrite_Bead L4
+L hiltop_backplane_brd-rescue:Ferrite_Bead-device L4
 U 1 1 5A0D0852
 P 10250 750
@@
 $EndComp
 $Comp
-L device:Ferrite_Bead L1
+L hiltop_backplane_brd-rescue:Ferrite_Bead-device L1
 U 1 1 5A0D09B1
 P 2000 2300
@@
 $EndComp
 $Comp
-L ftdi:FT2232H U6
+L hiltop_backplane_brd-rescue:FT2232H-ftdi U6
 U 1 1 5A0D0CDB
 P 7250 3750
@@
 $EndComp
 $Comp
-L memory:93LCxxC U5
+L hiltop_backplane_brd-rescue:93LCxxC-memory U5
 U 1 1 5A0D27FD
 P 3800 4750
@@
 $EndComp
 $Comp
-L device:R R111
+L hiltop_backplane_brd-rescue:R-device R111
 U 1 1 5A0E2040
 P 4000 3850
@@
 $EndComp
 $Comp
-L device:R R110
+L hiltop_backplane_brd-rescue:R-device R110
 U 1 1 5A0E22F5
 P 3800 3850
@@
 $EndComp
 $Comp
-L device:R R112
+L hiltop_backplane_brd-rescue:R-device R112
 U 1 1 5A0E2366
 P 4200 3850
@@
 $EndComp
 $Comp
-L device:R R113
+L hiltop_backplane_brd-rescue:R-device R113
 U 1 1 5A0E23C5
 P 4500 4650
@@
 $EndComp
 $Comp
-L device:R R114
+L hiltop_backplane_brd-rescue:R-device R114
 U 1 1 5A0E253E
 P 5050 2750
@@
 $EndComp
 $Comp
-L device:R R115
+L hiltop_backplane_brd-rescue:R-device R115
 U 1 1 5A0E2735
 P 5050 2850
@@
 $EndComp
 $Comp
-L device:R R117
+L hiltop_backplane_brd-rescue:R-device R117
 U 1 1 5A0E4574
 P 5850 3600
@@
 $EndComp
 $Comp
-L device:R R116
+L hiltop_backplane_brd-rescue:R-device R116
 U 1 1 5A0E467B
 P 5300 3350
@@
 $EndComp
 $Comp
-L device:C C28
+L hiltop_backplane_brd-rescue:C-device C28
 U 1 1 5A0E7988
 P 5550 3600
@@
 $EndComp
 $Comp
-L device:D_Schottky D2
+L hiltop_backplane_brd-rescue:D_Schottky-device D2
 U 1 1 5A0E9377
 P 2000 1800
@@
 $EndComp
 $Comp
-L device:R R118
+L hiltop_backplane_brd-rescue:R-device R118
 U 1 1 5A286A3D
 P 8800 1850
@@
 $EndComp
 $Comp
-L device:R R119
+L hiltop_backplane_brd-rescue:R-device R119
 U 1 1 5A286C57
 P 8800 1950
@@
 $EndComp
 $Comp
-L device:R R120
+L hiltop_backplane_brd-rescue:R-device R120
 U 1 1 5A286CD9
 P 8800 2050
@@
 $EndComp
 $Comp
-L device:R R121
+L hiltop_backplane_brd-rescue:R-device R121
 U 1 1 5A286D5E
 P 8800 2150
@@
 $EndComp
 $Comp
-L device:R R123
+L hiltop_backplane_brd-rescue:R-device R123
 U 1 1 5A286F0C
 P 8800 2450
@@
 $EndComp
 $Comp
-L device:R R124
+L hiltop_backplane_brd-rescue:R-device R124
 U 1 1 5A286F9B
 P 8800 2550
@@
 $EndComp
 $Comp
-L device:C C31
+L hiltop_backplane_brd-rescue:C-device C31
 U 1 1 5A28A03B
 P 6000 2300
@@
 $EndComp
 $Comp
-L device:R R122
+L hiltop_backplane_brd-rescue:R-device R122
 U 1 1 5A28A99D
 P 8800 2250
@@
 iCE40 CRESET
 $Comp
-L device:R R125
+L hiltop_backplane_brd-rescue:R-device R125
 U 1 1 5A432905
 P 9550 4800
@@
 $EndComp
 $Comp
-L device:R R126
+L hiltop_backplane_brd-rescue:R-device R126
 U 1 1 5A432C01
 P 9550 5000
@@
 $EndComp
 $Comp
-L device:LED D4
+L hiltop_backplane_brd-rescue:LED-device D4
 U 1 1 5A432D8D
 P 9000 4800
@@
 $EndComp
 $Comp
-L device:LED D5
+L hiltop_backplane_brd-rescue:LED-device D5
 U 1 1 5A432E41
 P 9000 5000
@@
 $EndComp
 $Comp
-L device:Crystal_GND24 Y1
+L hiltop_backplane_brd-rescue:Crystal_GND24-device Y1
 U 1 1 5A2C1F7D
 P 5250 5350
@@
 $EndComp
 $Comp
-L gti_Lattice:3pos_Jumper J3
+L hiltop_backplane_brd-rescue:3pos_Jumper-gti_Lattice J3
 U 1 1 5A2C5B3A
 P 2800 2900
@@
 $EndComp
 $Comp
-L gti_Lattice:3pos_Jumper J2
+L hiltop_backplane_brd-rescue:3pos_Jumper-gti_Lattice J2
 U 1 1 5A2C5C1B
 P 2800 2700
@@
 $EndComp
 $Comp
-L Connector1:Test_Point TP11
+L hiltop_backplane_brd-rescue:Test_Point-Connector1 TP11
 U 1 1 5A2FCE0A
 P 2000 1350
@@
 +1V8_IN
 $Comp
-L device:Ferrite_Bead L5
+L hiltop_backplane_brd-rescue:Ferrite_Bead-device L5
 U 1 1 5A0D0A0A
 P 10250 1000
@@
 +3V3_IN
 $Comp
-L Connector:TestPoint TP1
+L hiltop_backplane_brd-rescue:TestPoint-Connector TP1
 U 1 1 5D0D4D61
 P 5400 2050
+AR Path="/5D0D4D61" Ref="TP1"  Part="1"
+AR Path="/5A077B59/5D0D4D61" Ref="TP1"  Part="1"
 F 0 "TP1" V 5425 2300 50  0000 C CNN
 F 1 "+1V8_REG_OUT" V 5350 2525 50  0000 C CNN

Commit message: first pass draft for review
Parts:
- removed J2, J3: 3pos_Jumper, Connector_PinHeader_2.00mm:PinHeader_1x03_P2.00mm_Vertical, symbol hiltop_backplane_brd-rescue:3pos_Jumper-gti_Lattice
- added J? (x2): 3pos_Jumper, symbol gti_Lattice:3pos_Jumper
- C22, C23, C24, C25, C26, C27, C28, C29, C30, C31, C32, C33, C34, C35, C36, C37, C38, C39, C40: symbol hiltop_backplane_brd-rescue:C-device -> device:C
- D2: symbol hiltop_backplane_brd-rescue:D_Schottky-device -> device:D_Schottky
- D3: symbol hiltop_backplane_brd-rescue:NUP2105L-ESD_Protection -> ESD_Protection:NUP2105L
- D4, D5: symbol hiltop_backplane_brd-rescue:LED-device -> device:LED
- J1: symbol hiltop_backplane_brd-rescue:USB_B_Micro-Connector1 -> Connector:USB_B_Micro
- L1, L2, L3, L4, L5: symbol hiltop_backplane_brd-rescue:Ferrite_Bead-device -> device:Ferrite_Bead
- R110, R111, R112, R113, R114, R115, R116, R117, R118, R119, R120, R121, R122, R123, R124, R125, R126: symbol hiltop_backplane_brd-rescue:R-device -> device:R
- TP1: symbol hiltop_backplane_brd-rescue:TestPoint-Connector -> Connector:TestPoint
- TP11: symbol hiltop_backplane_brd-rescue:Test_Point-Connector1 -> Connector:TestPoint
- U5: symbol hiltop_backplane_brd-rescue:93LCxxC-memory -> memory:93LCxxC
- U6: symbol hiltop_backplane_brd-rescue:FT2232H-ftdi -> ftdi:FT2232H
- Y1: symbol hiltop_backplane_brd-rescue:Crystal_GND24-device -> device:Crystal_GND24

Commit message: lables connected to end of net, each component mapped to footprint, working on reducing error
Parts:
- J2, J3: renamed from J?; footprint (none) -> GTI_Footprint_Lib:3POS_JUMPER_R_0603_1608Metric
- TP15: renamed from TP1; footprint (none) -> TestPoint:TestPoint_Pad_D1.0mm
- renumbered C22 to C1, C31 to C10, C32 to C11, C33 to C12, C34 to C13, C35 to C14, C36 to C15, C37 to C16, C38 to C17, C39 to C18, C40 to C19, C23 to C2, C24 to C3, C25 to C4, C26 to C5, C27 to C6, C28 to C7, C29 to C8, C30 to C9, D2 to D1, D3 to D2, D4 to D3, D5 to D4, R110 to R1, R119 to R10, R120 to R11, R121 to R12, R122 to R13, R123 to R14, R124 to R15, R125 to R16, R126 to R17, R111 to R2, R112 to R3, R113 to R4, R114 to R5, R115 to R6, R116 to R7, R117 to R8, R118 to R9, TP11 to TP14, U5 to U1, U6 to U2
Connections:
- no-connect marks 0 -> 22

Commit message: added keepout to differential pair and trace clean up
Parts:
- J2, J3: symbol gti_Lattice:3pos_Jumper -> hiltop_backplane_brd-rescue:3pos_Jumper-gti_Lattice
Changed lines of the file:
@@
 $EndComp
 $Comp
-L gti_Lattice:3pos_Jumper J2
+L hiltop_backplane_brd-rescue:3pos_Jumper-gti_Lattice J2
 U 1 1 5C690C56
 P 3200 2400
@@
 $EndComp
 $Comp
-L gti_Lattice:3pos_Jumper J3
+L hiltop_backplane_brd-rescue:3pos_Jumper-gti_Lattice J3
 U 1 1 5C690DBE
 P 3200 2700

Commit message: final design checkin
Parts:
- removed U2: FT2232H, Package_DFN_QFN:QFN-64-1EP_9x9mm_P0.5mm_EP7.35x7.35mm, symbol ftdi:FT2232H
- added U2: FT2232H, Package_DFN_QFN:QFN-64-1EP_9x9mm_P0.5mm_EP7.35x7.35mm, symbol gti_Lattice:FT2232H
Connections:
- net +3V3_IN: now also U2.50 (VREGIN)
- net FTDI_UART_RXD: now also U2.39 (BDBUS1)
- net FTDI_UART_TXD: now also U2.38 (BDBUS0)
- net FTDI_UART_TXEN: now also U2.48 (BCBUS0)
- net FTDI_UART_~CTS: now also U2.41 (BDBUS3)
- net FTDI_UART_~RTS: now also U2.40 (BDBUS2)
- net GND: now also U2.1 (GND), U2.10 (AGND), U2.11 (GND), U2.13 (TEST), U2.15 (GND), U2.25 (GND), U2.35 (GND), U2.47 (GND), U2.5 (GND), U2.51 (GND), U2.65 (PAD)
- net at C16.1, C17.2, C18.2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: now also U2.20 (VCCIO), U2.31 (VCCIO), U2.42 (VCCIO), U2.56 (VCCIO)
- net at C13.2, C14.2, C15.2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: now also U2.12 (VCORE), U2.37 (VCORE), U2.64 (VCORE)
- net at C6.1, C9.1, L2.1: now also U2.9 (VPLL)
- net at C11.1, C12.1, L3.1: now also U2.4 (VPHY)
- net at C10.2, C8.2, TP15.1: now also U2.49 (VREGOUT)
- net at C5.2, Y1.3: now also U2.3 (OSCO)
- net at C3.2, Y1.1: now also U2.2 (OSCI)
- net at C7.2, R7.1: now also U2.14 (~RESET)
- net at R9.2: now also U2.16 (ADBUS0)
- net at R10.2: now also U2.17 (ADBUS1)
- net at R11.2: now also U2.18 (ADBUS2)
- net at R12.2: now also U2.19 (ADBUS3)
- net at R13.2: now also U2.21 (ADBUS4)
- net at R14.2: now also U2.23 (ADBUS6)
- net at R15.2: now also U2.24 (ADBUS7)
- net at D3.1 (K): now also U2.54 (BCBUS3)
- net at D4.1 (K): now also U2.55 (BCBUS4)
- net at R8.2: now also U2.6 (REF)
- net at R4.1, U1.3 (DI): now also U2.61 (EEDATA)
- net at R2.1, U1.2 (SCLK): now also U2.62 (EECLK)
- net at R1.2, U1.1 (CS): now also U2.63 (EECS)
- net at R6.1: now also U2.7 (DM)
- net at R5.1: now also U2.8 (DP)
Changed lines of the file:
@@
-$EndComp
-$Comp
-L ftdi:FT2232H U2
-U 1 1 5A0D0CDB
-P 7250 3750
-F 0 "U2" H 6200 5850 50  0000 L CNN
-F 1 "FT2232H" H 8000 5850 50  0000 L CNN
-F 2 "Package_DFN_QFN:QFN-64-1EP_9x9mm_P0.5mm_EP7.35x7.35mm" H 7250 3750 50  0001 C CNN
-F 3 "" H 7250 3750 50  0001 C CNN
-	1    7250 3750
-	1    0    0    -1
 $EndComp
 $Comp
@@
 NoConn ~ 4100 4750
 NoConn ~ 8450 2350
+$Comp
+L gti_Lattice:FT2232H U2
+U 1 1 5C716984
+P 7250 3750
+F 0 "U2" H 6250 5875 50  0000 C CNN
+F 1 "FT2232H" H 8125 5850 50  0000 C CNN
+F 2 "Package_DFN_QFN:QFN-64-1EP_9x9mm_P0.5mm_EP7.35x7.35mm" H 7250 3750 50  0001 C CNN
+F 3 "http://www.ftdichip.com/Products/ICs/FT2232H.html" H 7250 3750 50  0001 C CNN
+	1    7250 3750
+	1    0    0    -1
+$EndComp
+Wire Wire Line
+	7650 5950 7650 6050
+Wire Wire Line
+	7650 6050 7550 6050
 $EndSCHEMATC

Commit message: Rev A
Parts:
- C1, C10, C12, C13, C14, C15, C16, C17, C18, C19, C2, C4, C7, C9: value 0.1uF -> 100nF; symbol device:C -> hiltop_backplane_brd-rescue:C-device; Devtank (none) -> 105-019
- C11, C6: symbol device:C -> hiltop_backplane_brd-rescue:C-device; Devtank (none) -> 105-021
- C3, C5: symbol device:C -> hiltop_backplane_brd-rescue:C-device; Devtank (none) -> 106-012
- C8: symbol device:C -> hiltop_backplane_brd-rescue:C-device; Devtank (none) -> 105-022
- D1: value MBR120VLSFT3G -> MBR230LSFT1G; symbol device:D_Schottky -> hiltop_backplane_brd-rescue:D_Schottky-device; Devtank (none) -> 133-006
- D2: symbol ESD_Protection:NUP2105L -> hiltop_backplane_brd-rescue:NUP2105L-ESD_Protection; Devtank (none) -> 136-002
- D3, D4: value LED -> LED RED; symbol device:LED -> hiltop_backplane_brd-rescue:LED-device; Devtank (none) -> 110-004
- J1: Devtank (none) -> 703-005
- L1, L2, L3, L4, L5: symbol device:Ferrite_Bead -> hiltop_backplane_brd-rescue:Ferrite_Bead-device; Devtank (none) -> 113-001
- R1, R2, R3: symbol device:R -> hiltop_backplane_brd-rescue:R-device; Devtank (none) -> 101-501
- R10, R11, R12, R14, R15, R5, R6, R9: symbol device:R -> hiltop_backplane_brd-rescue:R-device; Devtank (none) -> 101-506
- R13: symbol device:R -> hiltop_backplane_brd-rescue:R-device
- R16, R17: symbol device:R -> hiltop_backplane_brd-rescue:R-device; Devtank (none) -> 101-509
- R4: symbol device:R -> hiltop_backplane_brd-rescue:R-device; Devtank (none) -> 101-505
- R7: symbol device:R -> hiltop_backplane_brd-rescue:R-device; Devtank (none) -> 101-507
- R8: symbol device:R -> hiltop_backplane_brd-rescue:R-device; Devtank (none) -> 101-508
- TP14, TP15: symbol Connector:TestPoint -> hiltop_backplane_brd-rescue:TestPoint-Connector
- U1: symbol memory:93LCxxC -> hiltop_backplane_brd-rescue:93LCxxC-memory; Devtank (none) -> 129-004
- U2: symbol gti_Lattice:FT2232H -> hiltop_backplane_brd-rescue:FT2232H-gti_Lattice; Devtank (none) -> 118-011
- Y1: symbol device:Crystal_GND24 -> hiltop_backplane_brd-rescue:Crystal_GND24-device; Devtank (none) -> 181-007
