File: kicad_hiltop_63hp_backplane/FPGA_breakout_brd.sch (KiCad schematic (older format))
At the start: 21 parts, among them J9 SO-DIMM

Commit message: Schematic updated to reflect USB logic and Global nets changed to local nets, renamed signals in motherboard connector
Changed lines of the file:
@@
 $Descr A4 11693 8268
 encoding utf-8
-Sheet 6 6
+Sheet 5 6
 Title ""
 Date ""
@@
 	1    0    0    -1
 $EndComp
-Text GLabel 1350 7100 0    39   Input ~ 0
-+3V3_EXT_IN
-Text GLabel 4050 6525 0    39   Input ~ 0
-+1V2_EXT_IN
-Text GLabel 4050 7075 0    39   Input ~ 0
-+1V8_EXT_IN
-Text GLabel 1350 6500 0    39   Input ~ 0
-+2V5_EXT_IN
 $Comp
 L power:GND #PWR038
@@
 	1700 1500 1700 1700
 Wire Wire Line
-	1500 1350 1500 1600
+	1500 1075 1500 1600
 Wire Wire Line
 	1400 1500 1400 1700
 Wire Wire Line
-	1300 1700 1300 1350
-Wire Wire Line
-	800  1350 800  1600
+	1300 1700 1300 1075
+Wire Wire Line
+	800  1075 800  1600
 Connection ~ 5400 6525
 Connection ~ 2700 7100
@@
 Connection ~ 1500 1600
 Wire Wire Line
-	1800 1350 1800 1600
+	1800 1075 1800 1600
 Wire Wire Line
 	1900 1700 1900 1600
@@
 Connection ~ 1400 4450
 Wire Wire Line
-	1300 4200 1300 4600
-Wire Wire Line
-	4050 6525 4150 6525
-Wire Wire Line
-	4050 7075 4150 7075
-Wire Wire Line
-	1350 6500 1450 6500
-Wire Wire Line
-	1350 7100 1450 7100
+	1300 4200 1300 4825
+Wire Wire Line
+	3550 6525 4150 6525
+Wire Wire Line
+	3550 7075 4150 7075
+Wire Wire Line
+	825  6500 1450 6500
+Wire Wire Line
+	825  7100 1450 7100
 Text HLabel 2800 7100 2    39   Input ~ 0
 +3V3_EXT_OUT
@@
 Text HLabel 10850 1275 1    39   Input ~ 0
 LVPECLK+
-Text GLabel 1800 4600 3    39   Input ~ 0
-+1V2_EXT_IN
-Text GLabel 1500 4600 3    39   Input ~ 0
-+1V8_EXT_IN
-Text GLabel 1300 4600 3    39   Input ~ 0
-+2V5_EXT_IN
-Text GLabel 800  4600 3    39   Input ~ 0
-+3V3_EXT_IN
-Text GLabel 1800 1350 1    39   Input ~ 0
-+1V2_EXT_IN
-Text GLabel 1500 1350 1    39   Input ~ 0
-+1V8_EXT_IN
-Text GLabel 1300 1350 1    39   Input ~ 0
-+2V5_EXT_IN
-Text GLabel 800  1350 1    39   Input ~ 0
-+3V3_EXT_IN
 Text HLabel 10450 1275 1    39   Input ~ 0
 DP1-
@@
 	2700 6500 2800 6500
 Wire Wire Line
-	800  4300 800  4600
+	800  4300 800  4825
 Wire Wire Line
 	900  4300 1100 4300
@@
 	1100 4300 1200 4300
 Wire Wire Line
-	1500 4300 1500 4600
-Wire Wire Line
-	1800 4300 1800 4600
+	1500 4300 1500 4825
+Wire Wire Line
+	1800 4300 1800 4825
 Wire Wire Line
 	1700 4450 2000 4450
@@
 	0    1    1    0
 $EndComp
+Text Label 800  1425 1    28   ~ 0
++3V3_EXT_IN
+Text Label 800  4775 1    28   ~ 0
++3V3_EXT_IN
+Text Label 1300 4775 1    28   ~ 0
++2V5_EXT_IN
+Text Label 1300 1400 1    28   ~ 0
++2V5_EXT_IN
+Text Label 1500 4775 1    28   ~ 0
++1V8_EXT_IN
+Text Label 1800 4750 1    28   ~ 0
++1V2_EXT_IN
+Text Label 1500 1400 1    28   ~ 0
++1V8_EXT_IN
+Text Label 1800 1400 1    28   ~ 0
++1V2_EXT_IN
+Text Label 925  6500 0    28   ~ 0
++2V5_EXT_IN
+Text Label 925  7100 0    28   ~ 0
++3V3_EXT_IN
+Text Label 3700 6525 0    28   ~ 0
++1V2_EXT_IN
+Text Label 3700 7075 0    28   ~ 0
++1V8_EXT_IN
 $EndSCHEMATC

Commit message: lables connected to end of net, each component mapped to footprint, working on reducing error
Parts:
- F16: renamed from F9; value Polyfuse -> 1206L050; footprint (none) -> Fuse:Fuse_1206_3216Metric
- F17: renamed from F10; value Polyfuse -> 1206L050; footprint (none) -> Fuse:Fuse_1206_3216Metric
- F18: renamed from F11; value Polyfuse -> 1206L050; footprint (none) -> Fuse:Fuse_1206_3216Metric
- F19: renamed from F?; value Polyfuse -> 1206L050; footprint (none) -> Fuse:Fuse_1206_3216Metric
- renumbered C61 to C22, C62 to C23, C64 to C24, C65 to C25, C68 to C26, C69 to C27, C72 to C28, C73 to C29, C58 to C30, C60 to C31, C59 to C32, C63 to C33, C66 to C34, C67 to C35, C70 to C36, C71 to C37, J9 to J11
Connections:
- no-connect marks 0 -> 2
Changed lines of the file:
@@
 $EndDescr
 $Comp
-L device:C C58
+L device:C C30
 U 1 1 5A418459
 P 4650 6725
-F 0 "C58" H 4675 6825 50  0000 L CNN
+F 0 "C30" H 4675 6825 50  0000 L CNN
 F 1 "10uF" H 4675 6625 50  0000 L CNN
 F 2 "Capacitor_SMD:C_0603_1608Metric" H 4688 6575 50  0001 C CNN
@@
 $EndComp
 $Comp
-L device:C C59
+L device:C C32
 U 1 1 5A4184EA
 P 4900 6725
-F 0 "C59" H 4925 6825 50  0000 L CNN
+F 0 "C32" H 4925 6825 50  0000 L CNN
 F 1 "1uF" H 4925 6625 50  0000 L CNN
 F 2 "Capacitor_SMD:C_0603_1608Metric" H 4938 6575 50  0001 C CNN
@@
 $EndComp
 $Comp
-L device:C C66
+L device:C C34
 U 1 1 5A41850F
 P 5150 6725
-F 0 "C66" H 5175 6825 50  0000 L CNN
+F 0 "C34" H 5175 6825 50  0000 L CNN
 F 1 "0.1uF" H 5175 6625 50  0000 L CNN
 F 2 "Capacitor_SMD:C_0402_1005Metric" H 5188 6575 50  0001 C CNN
@@
 $EndComp
 $Comp
-L device:C C70
+L device:C C36
 U 1 1 5A418541
 P 5400 6725
-F 0 "C70" H 5425 6825 50  0000 L CNN
+F 0 "C36" H 5425 6825 50  0000 L CNN
 F 1 "0.01uF" H 5425 6625 50  0000 L CNN
 F 2 "Capacitor_SMD:C_0402_1005Metric" H 5438 6575 50  0001 C CNN
@@
 $EndComp
 $Comp
-L device:C C60
+L device:C C31
 U 1 1 5A41856A
 P 4650 7275
-F 0 "C60" H 4675 7375 50  0000 L CNN
+F 0 "C31" H 4675 7375 50  0000 L CNN
 F 1 "10uF" H 4675 7175 50  0000 L CNN
 F 2 "Capacitor_SMD:C_0603_1608Metric" H 4688 7125 50  0001 C CNN
@@
 $EndComp
 $Comp
-L device:C C63
+L device:C C33
 U 1 1 5A4185BC
 P 4900 7275
-F 0 "C63" H 4925 7375 50  0000 L CNN
+F 0 "C33" H 4925 7375 50  0000 L CNN
 F 1 "1uF" H 4925 7175 50  0000 L CNN
 F 2 "Capacitor_SMD:C_0603_1608Metric" H 4938 7125 50  0001 C CNN
@@
 $EndComp
 $Comp
-L device:C C67
+L device:C C35
 U 1 1 5A4185F9
 P 5150 7275
-F 0 "C67" H 5175 7375 50  0000 L CNN
+F 0 "C35" H 5175 7375 50  0000 L CNN
 F 1 "0.1uF" H 5175 7175 50  0000 L CNN
 F 2 "Capacitor_SMD:C_0402_1005Metric" H 5188 7125 50  0001 C CNN
@@
 $EndComp
 $Comp
-L device:C C71
+L device:C C37
 U 1 1 5A41862F
 P 5400 7275
-F 0 "C71" H 5425 7375 50  0000 L CNN
+F 0 "C37" H 5425 7375 50  0000 L CNN
 F 1 "0.01uF" H 5425 7175 50  0000 L CNN
 F 2 "Capacitor_SMD:C_0402_1005Metric" H 5438 7125 50  0001 C CNN
@@
 $EndComp
 $Comp
-L device:C C61
+L device:C C22
 U 1 1 5A418664
 P 1950 6700
-F 0 "C61" H 1975 6800 50  0000 L CNN
+F 0 "C22" H 1975 6800 50  0000 L CNN
 F 1 "10uF" H 1975 6600 50  0000 L CNN
 F 2 "Capacitor_SMD:C_0603_1608Metric" H 1988 6550 50  0001 C CNN
@@
 $EndComp
 $Comp
-L device:C C64
+L device:C C24
 U 1 1 5A4186B2
 P 2200 6700
-F 0 "C64" H 2225 6800 50  0000 L CNN
+F 0 "C24" H 2225 6800 50  0000 L CNN
 F 1 "1uF" H 2225 6600 50  0000 L CNN
 F 2 "Capacitor_SMD:C_0603_1608Metric" H 2238 6550 50  0001 C CNN
@@
 $EndComp
 $Comp
-L device:C C68
+L device:C C26
 U 1 1 5A4186E9
 P 2450 6700
-F 0 "C68" H 2475 6800 50  0000 L CNN
+F 0 "C26" H 2475 6800 50  0000 L CNN
 F 1 "0.1uF" H 2475 6600 50  0000 L CNN
 F 2 "Capacitor_SMD:C_0402_1005Metric" H 2488 6550 50  0001 C CNN
@@
 $EndComp
 $Comp
-L device:C C72
+L device:C C28
 U 1 1 5A418729
 P 2700 6700
-F 0 "C72" H 2725 6800 50  0000 L CNN
+F 0 "C28" H 2725 6800 50  0000 L CNN
 F 1 "0.01uF" H 2725 6600 50  0000 L CNN
 F 2 "Capacitor_SMD:C_0402_1005Metric" H 2738 6550 50  0001 C CNN
@@
 $EndComp
 $Comp
-L device:C C62
+L device:C C23
 U 1 1 5A418776
 P 1950 7300
-F 0 "C62" H 1975 7400 50  0000 L CNN
+F 0 "C23" H 1975 7400 50  0000 L CNN
 F 1 "10uF" H 1975 7200 50  0000 L CNN
 F 2 "Capacitor_SMD:C_0603_1608Metric" H 1988 7150 50  0001 C CNN
@@
 $EndComp
 $Comp
-L device:C C65
+L device:C C25
 U 1 1 5A418B7E
 P 2200 7300
-F 0 "C65" H 2225 7400 50  0000 L CNN
+F 0 "C25" H 2225 7400 50  0000 L CNN
 F 1 "1uF" H 2225 7200 50  0000 L CNN
 F 2 "Capacitor_SMD:C_0603_1608Metric" H 2238 7150 50  0001 C CNN
@@
 $EndComp
 $Comp
-L device:C C69
+L device:C C27
 U 1 1 5A418BC9
 P 2450 7300
-F 0 "C69" H 2475 7400 50  0000 L CNN
+F 0 "C27" H 2475 7400 50  0000 L CNN
 F 1 "0.1uF" H 2475 7200 50  0000 L CNN
 F 2 "Capacitor_SMD:C_0402_1005Metric" H 2488 7150 50  0001 C CNN
@@
 $EndComp
 $Comp
-L device:C C73
+L device:C C29
 U 1 1 5A418C13
 P 2700 7300
-F 0 "C73" H 2725 7400 50  0000 L CNN
+F 0 "C29" H 2725 7400 50  0000 L CNN
 F 1 "0.01uF" H 2725 7200 50  0000 L CNN
 F 2 "Capacitor_SMD:C_0402_1005Metric" H 2738 7150 50  0001 C CNN
@@
 $EndComp
 $Comp
-L power:GND #PWR038
+L power:GND #PWR037
 U 1 1 5A41B6AD
 P 5550 6925
-F 0 "#PWR038" H 5550 6675 50  0001 C CNN
+F 0 "#PWR037" H 5550 6675 50  0001 C CNN
 F 1 "GND" H 5650 6925 50  0000 C CNN
 F 2 "" H 5550 6925 50  0001 C CNN
@@
 $EndComp
 $Comp
-L power:GND #PWR039
+L power:GND #PWR038
 U 1 1 5A41B7D9
 P 5550 7475
-F 0 "#PWR039" H 5550 7225 50  0001 C CNN
+F 0 "#PWR038" H 5550 7225 50  0001 C CNN
 F 1 "GND" H 5650 7475 50  0000 C CNN
 F 2 "" H 5550 7475 50  0001 C CNN
@@
 $EndComp
 $Comp
-L power:GND #PWR040
+L power:GND #PWR036
 U 1 1 5A41B927
 P 2850 7500
-F 0 "#PWR040" H 2850 7250 50  0001 C CNN
+F 0 "#PWR036" H 2850 7250 50  0001 C CNN
 F 1 "GND" H 2950 7500 50  0000 C CNN
 F 2 "" H 2850 7500 50  0001 C CNN
@@
 $EndComp
 $Comp
-L power:GND #PWR041
+L power:GND #PWR035
 U 1 1 5A41B976
 P 2850 6900
-F 0 "#PWR041" H 2850 6650 50  0001 C CNN
+F 0 "#PWR035" H 2850 6650 50  0001 C CNN
 F 1 "GND" H 2950 6900 50  0000 C CNN
 F 2 "" H 2850 6900 50  0001 C CNN
@@
 $EndComp
 $Comp
-L power:GND #PWR042
+L power:GND #PWR039
 U 1 1 5A41CA24
 P 11050 4500
-F 0 "#PWR042" H 11050 4250 50  0001 C CNN
+F 0 "#PWR039" H 11050 4250 50  0001 C CNN
 F 1 "GND" H 11050 4350 50  0000 C CNN
 F 2 "" H 11050 4500 50  0001 C CNN
@@
 Connection ~ 10950 1500
 $Comp
-L power:GND #PWR043
+L power:GND #PWR040
 U 1 1 5A421824
 P 11100 1550
-F 0 "#PWR043" H 11100 1300 50  0001 C CNN
+F 0 "#PWR040" H 11100 1300 50  0001 C CNN
 F 1 "GND" H 11100 1400 50  0000 C CNN
 F 2 "" H 11100 1550 50  0001 C CNN
@@
 	8600 1500 9150 1500
 $Comp
-L gti_Lattice:SO-DIMM J9
+L gti_Lattice:SO-DIMM J11
 U 1 1 5A3A8985
 P 11200 2950
-F 0 "J9" H 10250 3100 60  0000 C CNN
+F 0 "J11" H 10250 3100 60  0000 C CNN
 F 1 "SO-DIMM" H 11300 2800 60  0000 C CNN
 F 2 "Devtank_PCB_Lib:Conn_TE-DDR2-SODIMM-0.6-200P-ComputeModule" H 11350 2950 60  0001 C CNN
@@
 GPIO_55
 $Comp
-L device:Polyfuse F9
+L device:Polyfuse F16
 U 1 1 5CEC5F97
 P 1600 6500
-F 0 "F9" V 1375 6500 50  0000 C CNN
-F 1 "Polyfuse" V 1466 6500 50  0000 C CNN
-F 2 "" H 1650 6300 50  0001 L CNN
+F 0 "F16" V 1375 6500 50  0000 C CNN
+F 1 "1206L050" V 1466 6500 50  0000 C CNN
+F 2 "Fuse:Fuse_1206_3216Metric" H 1650 6300 50  0001 L CNN
 F 3 "" H 1600 6500 50  0001 C CNN
 	1    1600 6500
@@
 $EndComp
 $Comp
-L device:Polyfuse F10
+L device:Polyfuse F17
 U 1 1 5CEC61F6
 P 1600 7100
-F 0 "F10" V 1375 7100 50  0000 C CNN
-F 1 "Polyfuse" V 1466 7100 50  0000 C CNN
-F 2 "" H 1650 6900 50  0001 L CNN
+F 0 "F17" V 1375 7100 50  0000 C CNN
+F 1 "1206L050" V 1466 7100 50  0000 C CNN
+F 2 "Fuse:Fuse_1206_3216Metric" H 1650 6900 50  0001 L CNN
 F 3 "" H 1600 7100 50  0001 C CNN
 	1    1600 7100
@@
 $EndComp
 $Comp
-L device:Polyfuse F11
+L device:Polyfuse F18
 U 1 1 5CEC625C
 P 4300 6525
-F 0 "F11" V 4075 6525 50  0000 C CNN
-F 1 "Polyfuse" V 4166 6525 50  0000 C CNN
-F 2 "" H 4350 6325 50  0001 L CNN
+F 0 "F18" V 4075 6525 50  0000 C CNN
+F 1 "1206L050" V 4166 6525 50  0000 C CNN
+F 2 "Fuse:Fuse_1206_3216Metric" H 4350 6325 50  0001 L CNN
 F 3 "" H 4300 6525 50  0001 C CNN
 	1    4300 6525
@@
 $EndComp
 $Comp
-L device:Polyfuse F?
+L device:Polyfuse F19
 U 1 1 5C2D630E
 P 4300 7075
-F 0 "F?" V 4075 7075 50  0000 C CNN
-F 1 "Polyfuse" V 4166 7075 50  0000 C CNN
-F 2 "" H 4350 6875 50  0001 L CNN
+F 0 "F19" V 4075 7075 50  0000 C CNN
+F 1 "1206L050" V 4166 7075 50  0000 C CNN
+F 2 "Fuse:Fuse_1206_3216Metric" H 4350 6875 50  0001 L CNN
 F 3 "" H 4300 7075 50  0001 C CNN
 	1    4300 7075
@@
 Text Label 1800 1400 1    28   ~ 0
 +1V2_EXT_IN
-Text Label 925  6500 0    28   ~ 0
+Text Label 825  6500 0    28   ~ 0
 +2V5_EXT_IN
-Text Label 925  7100 0    28   ~ 0
+Text Label 825  7100 0    28   ~ 0
 +3V3_EXT_IN
-Text Label 3700 6525 0    28   ~ 0
+Text Label 3550 6525 0    28   ~ 0
 +1V2_EXT_IN
-Text Label 3700 7075 0    28   ~ 0
+Text Label 3550 7075 0    28   ~ 0
 +1V8_EXT_IN
+NoConn ~ 8700 1700
+NoConn ~ 9050 1700
 $EndSCHEMATC

Commit message: schematic error reduced and footprint mapped
Parts:
- J11: symbol gti_Lattice:SO-DIMM -> hiltop_backplane_brd-rescue:SO-DIMM-gti_Lattice
Changed lines of the file:
@@
 $Descr A4 11693 8268
 encoding utf-8
-Sheet 5 6
+Sheet 6 6
 Title ""
 Date ""
@@
 	8600 1500 9150 1500
 $Comp
-L gti_Lattice:SO-DIMM J11
+L hiltop_backplane_brd-rescue:SO-DIMM-gti_Lattice J11
 U 1 1 5A3A8985
 P 11200 2950
@@
 	0    1    1    0
 $EndComp
-Text Label 800  1425 1    28   ~ 0
+Text Label 800  1075 3    28   ~ 0
 +3V3_EXT_IN
-Text Label 800  4775 1    28   ~ 0
+Text Label 800  4825 1    28   ~ 0
 +3V3_EXT_IN
-Text Label 1300 4775 1    28   ~ 0
+Text Label 1300 4825 1    28   ~ 0
 +2V5_EXT_IN
-Text Label 1300 1400 1    28   ~ 0
+Text Label 1300 1075 3    28   ~ 0
 +2V5_EXT_IN
-Text Label 1500 4775 1    28   ~ 0
+Text Label 1500 4825 1    28   ~ 0
 +1V8_EXT_IN
-Text Label 1800 4750 1    28   ~ 0
+Text Label 1800 4825 1    28   ~ 0
 +1V2_EXT_IN
-Text Label 1500 1400 1    28   ~ 0
+Text Label 1500 1075 3    28   ~ 0
 +1V8_EXT_IN
-Text Label 1800 1400 1    28   ~ 0
+Text Label 1800 1075 3    28   ~ 0
 +1V2_EXT_IN
 Text Label 825  6500 0    28   ~ 0

Commit message: pci connector connection moved to bottom layer, FTDI routing and FPGA power routing
Parts:
- J11: symbol hiltop_backplane_brd-rescue:SO-DIMM-gti_Lattice -> hiltop_backplane_brd-rescue:SO-DIMM-gti_Lattice-hiltop_backplane_brd-rescue
Changed lines of the file:
@@
 	8600 1500 9150 1500
 $Comp
-L hiltop_backplane_brd-rescue:SO-DIMM-gti_Lattice J11
+L hiltop_backplane_brd-rescue:SO-DIMM-gti_Lattice-hiltop_backplane_brd-rescue J11
 U 1 1 5A3A8985
 P 11200 2950
+AR Path="/5A3A8985" Ref="J11"  Part="1"
+AR Path="/5A077BA2/5A3A8985" Ref="J11"  Part="1"
 F 0 "J11" H 10250 3100 60  0000 C CNN
 F 1 "SO-DIMM" H 11300 2800 60  0000 C CNN

Commit message: Rev A
Parts:
- C22, C23, C30, C31: symbol device:C -> hiltop_backplane_brd-rescue:C-device; Devtank (none) -> 105-023
- C24, C25, C32, C33: symbol device:C -> hiltop_backplane_brd-rescue:C-device; Devtank (none) -> 105-014
- C26, C27, C34, C35: value 0.1uF -> 100nF; symbol device:C -> hiltop_backplane_brd-rescue:C-device; Devtank (none) -> 105-019
- C28, C29, C36, C37: value 0.01uF -> 10nF; symbol device:C -> hiltop_backplane_brd-rescue:C-device; Devtank (none) -> 105-017
- F16, F17, F18, F19: symbol device:Polyfuse -> hiltop_backplane_brd-rescue:Polyfuse-device; Devtank (none) -> 190-002
- J11: Devtank (none) -> 712-001
Changed lines of the file:
@@
 $EndDescr
 $Comp
-L device:C C30
+L hiltop_backplane_brd-rescue:C-device C30
 U 1 1 5A418459
 P 4650 6725
@@
 F 2 "Capacitor_SMD:C_0603_1608Metric" H 4688 6575 50  0001 C CNN
 F 3 "" H 4650 6725 50  0001 C CNN
+F 4 "105-023" H 0   0   50  0001 C CNN "Devtank"
 	1    4650 6725
 	1    0    0    -1
 $EndComp
 $Comp
-L device:C C32
+L hiltop_backplane_brd-rescue:C-device C32
 U 1 1 5A4184EA
 P 4900 6725
@@
 F 2 "Capacitor_SMD:C_0603_1608Metric" H 4938 6575 50  0001 C CNN
 F 3 "" H 4900 6725 50  0001 C CNN
+F 4 "105-014" H 0   0   50  0001 C CNN "Devtank"
 	1    4900 6725
 	1    0    0    -1
 $EndComp
 $Comp
-L device:C C34
+L hiltop_backplane_brd-rescue:C-device C34
 U 1 1 5A41850F
 P 5150 6725
 F 0 "C34" H 5175 6825 50  0000 L CNN
-F 1 "0.1uF" H 5175 6625 50  0000 L CNN
+F 1 "100nF" H 5175 6625 50  0000 L CNN
 F 2 "Capacitor_SMD:C_0402_1005Metric" H 5188 6575 50  0001 C CNN
 F 3 "" H 5150 6725 50  0001 C CNN
+F 4 "105-019" H 0   0   50  0001 C CNN "Devtank"
 	1    5150 6725
 	1    0    0    -1
 $EndComp
 $Comp
-L device:C C36
+L hiltop_backplane_brd-rescue:C-device C36
 U 1 1 5A418541
 P 5400 6725
 F 0 "C36" H 5425 6825 50  0000 L CNN
-F 1 "0.01uF" H 5425 6625 50  0000 L CNN
+F 1 "10nF" H 5425 6625 50  0000 L CNN
 F 2 "Capacitor_SMD:C_0402_1005Metric" H 5438 6575 50  0001 C CNN
 F 3 "" H 5400 6725 50  0001 C CNN
+F 4 "105-017" H 0   0   50  0001 C CNN "Devtank"
 	1    5400 6725
 	1    0    0    -1
 $EndComp
 $Comp
-L device:C C31
+L hiltop_backplane_brd-rescue:C-device C31
 U 1 1 5A41856A
 P 4650 7275
@@
 F 2 "Capacitor_SMD:C_0603_1608Metric" H 4688 7125 50  0001 C CNN
 F 3 "" H 4650 7275 50  0001 C CNN
+F 4 "105-023" H 0   0   50  0001 C CNN "Devtank"
 	1    4650 7275
 	1    0    0    -1
 $EndComp
 $Comp
-L device:C C33
+L hiltop_backplane_brd-rescue:C-device C33
 U 1 1 5A4185BC
 P 4900 7275
@@
 F 2 "Capacitor_SMD:C_0603_1608Metric" H 4938 7125 50  0001 C CNN
 F 3 "" H 4900 7275 50  0001 C CNN
+F 4 "105-014" H 0   0   50  0001 C CNN "Devtank"
 	1    4900 7275
 	1    0    0    -1
 $EndComp
 $Comp
-L device:C C35
+L hiltop_backplane_brd-rescue:C-device C35
 U 1 1 5A4185F9
 P 5150 7275
 F 0 "C35" H 5175 7375 50  0000 L CNN
-F 1 "0.1uF" H 5175 7175 50  0000 L CNN
+F 1 "100nF" H 5175 7175 50  0000 L CNN
 F 2 "Capacitor_SMD:C_0402_1005Metric" H 5188 7125 50  0001 C CNN
 F 3 "" H 5150 7275 50  0001 C CNN
+F 4 "105-019" H 0   0   50  0001 C CNN "Devtank"
 	1    5150 7275
 	1    0    0    -1
 $EndComp
 $Comp
-L device:C C37
+L hiltop_backplane_brd-rescue:C-device C37
 U 1 1 5A41862F
 P 5400 7275
 F 0 "C37" H 5425 7375 50  0000 L CNN
-F 1 "0.01uF" H 5425 7175 50  0000 L CNN
+F 1 "10nF" H 5425 7175 50  0000 L CNN
 F 2 "Capacitor_SMD:C_0402_1005Metric" H 5438 7125 50  0001 C CNN
 F 3 "" H 5400 7275 50  0001 C CNN
+F 4 "105-017" H 0   0   50  0001 C CNN "Devtank"
 	1    5400 7275
 	1    0    0    -1
 $EndComp
 $Comp
-L device:C C22
+L hiltop_backplane_brd-rescue:C-device C22
 U 1 1 5A418664
 P 1950 6700
@@
 F 2 "Capacitor_SMD:C_0603_1608Metric" H 1988 6550 50  0001 C CNN
 F 3 "" H 1950 6700 50  0001 C CNN
+F 4 "105-023" H 0   0   50  0001 C CNN "Devtank"
 	1    1950 6700
 	1    0    0    -1
 $EndComp
 $Comp
-L device:C C24
+L hiltop_backplane_brd-rescue:C-device C24
 U 1 1 5A4186B2
 P 2200 6700
@@
 F 2 "Capacitor_SMD:C_0603_1608Metric" H 2238 6550 50  0001 C CNN
 F 3 "" H 2200 6700 50  0001 C CNN
+F 4 "105-014" H 0   0   50  0001 C CNN "Devtank"
 	1    2200 6700
 	1    0    0    -1
 $EndComp
 $Comp
-L device:C C26
+L hiltop_backplane_brd-rescue:C-device C26
 U 1 1 5A4186E9
 P 2450 6700
 F 0 "C26" H 2475 6800 50  0000 L CNN
-F 1 "0.1uF" H 2475 6600 50  0000 L CNN
+F 1 "100nF" H 2475 6600 50  0000 L CNN
 F 2 "Capacitor_SMD:C_0402_1005Metric" H 2488 6550 50  0001 C CNN
 F 3 "" H 2450 6700 50  0001 C CNN
+F 4 "105-019" H 0   0   50  0001 C CNN "Devtank"
 	1    2450 6700
 	1    0    0    -1
 $EndComp
 $Comp
-L device:C C28
+L hiltop_backplane_brd-rescue:C-device C28
 U 1 1 5A418729
 P 2700 6700
 F 0 "C28" H 2725 6800 50  0000 L CNN
-F 1 "0.01uF" H 2725 6600 50  0000 L CNN
+F 1 "10nF" H 2725 6600 50  0000 L CNN
 F 2 "Capacitor_SMD:C_0402_1005Metric" H 2738 6550 50  0001 C CNN
 F 3 "" H 2700 6700 50  0001 C CNN
+F 4 "105-017" H 0   0   50  0001 C CNN "Devtank"
 	1    2700 6700
 	1    0    0    -1
 $EndComp
 $Comp
-L device:C C23
+L hiltop_backplane_brd-rescue:C-device C23
 U 1 1 5A418776
 P 1950 7300
@@
 F 2 "Capacitor_SMD:C_0603_1608Metric" H 1988 7150 50  0001 C CNN
 F 3 "" H 1950 7300 50  0001 C CNN
+F 4 "105-023" H 0   0   50  0001 C CNN "Devtank"
 	1    1950 7300
 	1    0    0    -1
 $EndComp
 $Comp
-L device:C C25
+L hiltop_backplane_brd-rescue:C-device C25
 U 1 1 5A418B7E
 P 2200 7300
@@
 F 2 "Capacitor_SMD:C_0603_1608Metric" H 2238 7150 50  0001 C CNN
 F 3 "" H 2200 7300 50  0001 C CNN
+F 4 "105-014" H 0   0   50  0001 C CNN "Devtank"
 	1    2200 7300
 	1    0    0    -1
 $EndComp
 $Comp
-L device:C C27
+L hiltop_backplane_brd-rescue:C-device C27
 U 1 1 5A418BC9
 P 2450 7300
 F 0 "C27" H 2475 7400 50  0000 L CNN
-F 1 "0.1uF" H 2475 7200 50  0000 L CNN
+F 1 "100nF" H 2475 7200 50  0000 L CNN
 F 2 "Capacitor_SMD:C_0402_1005Metric" H 2488 7150 50  0001 C CNN
 F 3 "" H 2450 7300 50  0001 C CNN
+F 4 "105-019" H 0   0   50  0001 C CNN "Devtank"
 	1    2450 7300
 	1    0    0    -1
 $EndComp
 $Comp
-L device:C C29
+L hiltop_backplane_brd-rescue:C-device C29
 U 1 1 5A418C13
 P 2700 7300
 F 0 "C29" H 2725 7400 50  0000 L CNN
-F 1 "0.01uF" H 2725 7200 50  0000 L CNN
+F 1 "10nF" H 2725 7200 50  0000 L CNN
 F 2 "Capacitor_SMD:C_0402_1005Metric" H 2738 7150 50  0001 C CNN
 F 3 "" H 2700 7300 50  0001 C CNN
+F 4 "105-017" H 0   0   50  0001 C CNN "Devtank"
 	1    2700 7300
 	1    0    0    -1
@@
 F 2 "Devtank_PCB_Lib:Conn_TE-DDR2-SODIMM-0.6-200P-ComputeModule" H 11350 2950 60  0001 C CNN
 F 3 "" H 11350 2950 60  0001 C CNN
+F 4 "712-001" H 0   0   50  0001 C CNN "Devtank"
 	1    11200 2950
 	0    1    1    0
@@
 GPIO_55
 $Comp
-L device:Polyfuse F16
+L hiltop_backplane_brd-rescue:Polyfuse-device F16
 U 1 1 5CEC5F97
 P 1600 6500
@@
 F 2 "Fuse:Fuse_1206_3216Metric" H 1650 6300 50  0001 L CNN
 F 3 "" H 1600 6500 50  0001 C CNN
+F 4 "190-002" H 0   0   50  0001 C CNN "Devtank"
 	1    1600 6500
 	0    1    1    0
 $EndComp
 $Comp
-L device:Polyfuse F17
+L hiltop_backplane_brd-rescue:Polyfuse-device F17
 U 1 1 5CEC61F6
 P 1600 7100
@@
 F 2 "Fuse:Fuse_1206_3216Metric" H 1650 6900 50  0001 L CNN
 F 3 "" H 1600 7100 50  0001 C CNN
+F 4 "190-002" H 0   0   50  0001 C CNN "Devtank"
 	1    1600 7100
 	0    1    1    0
 $EndComp
 $Comp
-L device:Polyfuse F18
+L hiltop_backplane_brd-rescue:Polyfuse-device F18
 U 1 1 5CEC625C
 P 4300 6525
@@
 F 2 "Fuse:Fuse_1206_3216Metric" H 4350 6325 50  0001 L CNN
 F 3 "" H 4300 6525 50  0001 C CNN
+F 4 "190-002" H 0   0   50  0001 C CNN "Devtank"
 	1    4300 6525
 	0    1    1    0
 $EndComp
 $Comp
-L device:Polyfuse F19
+L hiltop_backplane_brd-rescue:Polyfuse-device F19
 U 1 1 5C2D630E
 P 4300 7075
@@
 F 2 "Fuse:Fuse_1206_3216Metric" H 4350 6875 50  0001 L CNN
 F 3 "" H 4300 7075 50  0001 C CNN
+F 4 "190-002" H 0   0   50  0001 C CNN "Devtank"
 	1    4300 7075
 	0    1    1    0

Commit message: add latest changes
Parts:
- added R5, R6, R84, R85, R86, R87, R88, R89, R90, R91: 0R, Resistor_SMD:R_0402_1005Metric, symbol device:R
- C22, C23, C24, C25, C26, C27, C28, C29, C30, C31, C32, C33, C34, C35, C36, C37: symbol hiltop_backplane_brd-rescue:C-device -> hiltop_backplane_brd-rescue:C-device-hiltop_backplane_brd-rescue
- F16, F17, F18, F19: symbol hiltop_backplane_brd-rescue:Polyfuse-device -> hiltop_backplane_brd-rescue:Polyfuse-device-hiltop_backplane_brd-rescue
- J11: symbol hiltop_backplane_brd-rescue:SO-DIMM-gti_Lattice-hiltop_backplane_brd-rescue -> hiltop_backplane_brd-rescue:SO-DIMM-gti_Lattice-hiltop_backplane_brd-rescue-hiltop_backplane_brd-rescue
Connections:
- wire segments 360 -> 380
