File: kicad_hiltop_63hp_backplane/fpga_soc_module.sch (KiCad schematic (older format))
At the start: 31 parts, among them J11 SO-DIMM

Commit message: Rev C ready for review - updated CERN license details
Connections:
- net GND: now also J11.104 (GND), J11.110 (GND), J11.116 (GND), J11.122 (GND), J11.128 (GND), J11.134 (GND), J11.14 (GND), J11.140 (GND), J11.146 (GND), J11.152 (GND), J11.158 (GND), J11.164 (GND), J11.170 (GND), J11.176 (GND), J11.186 (GND), J11.2 (GND), J11.20 (GND), J11.26 (GND), J11.32 (GND), J11.38 (GND), J11.44 (GND), J11.50 (GND), J11.56 (GND), J11.62 (GND), J11.68 (GND), J11.74 (GND), J11.8 (GND), J11.80 (GND), J11.86 (GND), J11.92 (GND), J11.98 (GND)
Changed lines of the file:
@@
 $Descr A3 11693 16535 portrait
 encoding utf-8
-Sheet 5 6
+Sheet 4 6
 Title "63HP HILTOP Backplane"
 Date "2021-02-04"
@@
 Connection ~ 5975 11600
 $Comp
-L power:GND #PWR?
+L power:GND #PWR0125
 U 1 1 614161A1
 P 3025 12100
-F 0 "#PWR?" H 3025 11850 50  0001 C CNN
+F 0 "#PWR0125" H 3025 11850 50  0001 C CNN
 F 1 "GND" H 3025 11950 50  0000 C CNN
 F 2 "" H 3025 12100 50  0001 C CNN
@@
 TRIGGER
 $Comp
-L power:+2V5 #PWR?
+L power:+2V5 #PWR0126
 U 1 1 6192EDC7
 P 10100 1150
-F 0 "#PWR?" H 10100 1000 50  0001 C CNN
+F 0 "#PWR0126" H 10100 1000 50  0001 C CNN
 F 1 "+2V5" H 10115 1323 50  0000 C CNN
 F 2 "" H 10100 1150 50  0001 C CNN
@@
 $EndComp
 $Comp
-L power:+3V3 #PWR?
+L power:+3V3 #PWR0127
 U 1 1 619303FE
 P 10100 2400
-F 0 "#PWR?" H 10100 2250 50  0001 C CNN
+F 0 "#PWR0127" H 10100 2250 50  0001 C CNN
 F 1 "+3V3" H 10115 2573 50  0000 C CNN
 F 2 "" H 10100 2400 50  0001 C CNN
@@
 $EndComp
 $Comp
-L power:+1V2 #PWR?
+L power:+1V2 #PWR0128
 U 1 1 61933A62
 P 10100 3550
-F 0 "#PWR?" H 10100 3400 50  0001 C CNN
+F 0 "#PWR0128" H 10100 3400 50  0001 C CNN
 F 1 "+1V2" H 10115 3723 50  0000 C CNN
 F 2 "" H 10100 3550 50  0001 C CNN
@@
 $EndComp
 $Comp
-L power:+1V8 #PWR?
+L power:+1V8 #PWR0129
 U 1 1 6193C405
 P 10100 4750
-F 0 "#PWR?" H 10100 4600 50  0001 C CNN
+F 0 "#PWR0129" H 10100 4600 50  0001 C CNN
 F 1 "+1V8" H 10115 4923 50  0000 C CNN
 F 2 "" H 10100 4750 50  0001 C CNN
@@
 Text HLabel 2750 8400 0    60   Input ~ 0
 GPIO_60
+Wire Wire Line
+	5975 11100 5975 11400
+Connection ~ 5975 11100
+Connection ~ 5975 11400
 $EndSCHEMATC
