File: kicad_hiltop_84hp_backplane/hiltop_backplane_brd.kicad_sch (KiCad schematic)
At the start: 30 parts

Commit message: Started differential tracking on layout
Other:
- sheet backplane_connector ports: added USB7_N, USB7_P; removed USB6_N, USB6_P
Changed lines of the file:
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@@
     (stroke (width 0) (type default) (color 0 0 0 0))
   )
-  (wire (pts (xy 351.79 160.02) (xy 371.475 160.02))
+  (wire (pts (xy 351.79 122.555) (xy 371.475 122.555))
     (stroke (width 0) (type default) (color 0 0 0 0))
   )
@@
     (stroke (width 0) (type default) (color 0 0 0 0))
   )
-  (wire (pts (xy 46.99 83.82) (xy 33.02 83.82))
+  (wire (pts (xy 46.99 91.44) (xy 33.02 91.44))
     (stroke (width 0) (type default) (color 0 0 0 0))
   )
@@
     (stroke (width 0) (type default) (color 0 0 0 0))
   )
-  (wire (pts (xy 351.79 145.415) (xy 371.475 145.415))
+  (wire (pts (xy 351.79 153.035) (xy 371.475 153.035))
     (stroke (width 0) (type default) (color 0 0 0 0))
   )
@@
     (stroke (width 0) (type default) (color 0 0 0 0))
   )
-  (wire (pts (xy 351.79 153.035) (xy 371.475 153.035))
+  (wire (pts (xy 351.79 145.415) (xy 371.475 145.415))
     (stroke (width 0) (type default) (color 0 0 0 0))
   )
@@
     (stroke (width 0) (type default) (color 0 0 0 0))
   )
-  (wire (pts (xy 351.79 137.795) (xy 371.475 137.795))
+  (wire (pts (xy 351.79 160.02) (xy 371.475 160.02))
     (stroke (width 0) (type default) (color 0 0 0 0))
   )
@@
     (stroke (width 0) (type default) (color 0 0 0 0))
   )
-  (wire (pts (xy 46.99 93.98) (xy 27.94 93.98))
+  (wire (pts (xy 46.99 86.36) (xy 27.94 86.36))
     (stroke (width 0) (type default) (color 0 0 0 0))
   )
@@
     (stroke (width 0) (type default) (color 0 0 0 0))
   )
-  (wire (pts (xy 351.79 125.095) (xy 371.475 125.095))
+  (wire (pts (xy 351.79 132.715) (xy 371.475 132.715))
     (stroke (width 0) (type default) (color 0 0 0 0))
   )
@@
     (stroke (width 0) (type default) (color 0 0 0 0))
   )
-  (wire (pts (xy 351.79 122.555) (xy 371.475 122.555))
+  (wire (pts (xy 351.79 130.175) (xy 371.475 130.175))
     (stroke (width 0) (type default) (color 0 0 0 0))
   )
@@
     (stroke (width 0) (type default) (color 0 0 0 0))
   )
-  (wire (pts (xy 46.99 91.44) (xy 27.94 91.44))
+  (wire (pts (xy 46.99 83.82) (xy 27.94 83.82))
     (stroke (width 0) (type default) (color 0 0 0 0))
   )
-  (wire (pts (xy 351.79 162.56) (xy 371.475 162.56))
+  (wire (pts (xy 351.79 125.095) (xy 371.475 125.095))
     (stroke (width 0) (type default) (color 0 0 0 0))
   )
@@
     (stroke (width 0) (type default) (color 0 0 0 0))
   )
-  (wire (pts (xy 351.79 155.575) (xy 371.475 155.575))
+  (wire (pts (xy 351.79 147.955) (xy 371.475 147.955))
     (stroke (width 0) (type default) (color 0 0 0 0))
   )
@@
     (stroke (width 0) (type default) (color 0 0 0 0))
   )
-  (wire (pts (xy 351.79 147.955) (xy 371.475 147.955))
+  (wire (pts (xy 351.79 155.575) (xy 371.475 155.575))
     (stroke (width 0) (type default) (color 0 0 0 0))
   )
@@
     (stroke (width 0) (type default) (color 0 0 0 0))
   )
-  (wire (pts (xy 351.79 140.335) (xy 371.475 140.335))
+  (wire (pts (xy 351.79 162.56) (xy 371.475 162.56))
     (stroke (width 0) (type default) (color 0 0 0 0))
   )
@@
     (stroke (width 0) (type default) (color 0 0 0 0))
   )
-  (wire (pts (xy 46.99 86.36) (xy 33.02 86.36))
+  (wire (pts (xy 46.99 93.98) (xy 33.02 93.98))
     (stroke (width 0) (type default) (color 0 0 0 0))
   )
@@
     (stroke (width 0) (type default) (color 0 0 0 0))
   )
-  (wire (pts (xy 351.79 130.175) (xy 371.475 130.175))
+  (wire (pts (xy 351.79 137.795) (xy 371.475 137.795))
     (stroke (width 0) (type default) (color 0 0 0 0))
   )
@@
     (stroke (width 0) (type default) (color 0 0 0 0))
   )
-  (wire (pts (xy 351.79 132.715) (xy 371.475 132.715))
+  (wire (pts (xy 351.79 140.335) (xy 371.475 140.335))
     (stroke (width 0) (type default) (color 0 0 0 0))
   )
@@
     (effects (font (size 1.524 1.524)) (justify right bottom))
   )
-  (label "USB6_P" (at 371.475 162.56 180)
+  (label "USB7_P" (at 371.475 125.095 180)
     (effects (font (size 1.524 1.524)) (justify right bottom))
   )
@@
     (effects (font (size 1.524 1.524)) (justify right bottom))
   )
-  (label "USB5_N" (at 371.475 153.035 180)
+  (label "USB5_N" (at 371.475 145.415 180)
     (effects (font (size 1.524 1.524)) (justify right bottom))
   )
@@
     (effects (font (size 1.524 1.524)) (justify left bottom))
   )
-  (label "USB6_N" (at 371.475 160.02 180)
+  (label "USB7_N" (at 371.475 122.555 180)
     (effects (font (size 1.524 1.524)) (justify right bottom))
   )
@@
     (effects (font (size 1.524 1.524)) (justify right bottom))
   )
-  (label "USB6_P" (at 33.02 83.82 0)
+  (label "USB7_P" (at 33.02 91.44 0)
     (effects (font (size 1.524 1.524)) (justify left bottom))
   )
@@
     (effects (font (size 1.524 1.524)) (justify right bottom))
   )
-  (label "USB4_P" (at 371.475 147.955 180)
+  (label "USB4_P" (at 371.475 155.575 180)
     (effects (font (size 1.524 1.524)) (justify right bottom))
   )
@@
     (effects (font (size 1.524 1.524)) (justify right bottom))
   )
-  (label "FTDI_USB_DP" (at 27.94 91.44 0)
+  (label "FTDI_USB_DP" (at 27.94 83.82 0)
     (effects (font (size 1.524 1.524)) (justify left bottom))
   )
@@
     (effects (font (size 1.524 1.524)) (justify right bottom))
   )
-  (label "USB3_N" (at 371.475 137.795 180)
+  (label "USB3_N" (at 371.475 160.02 180)
     (effects (font (size 1.524 1.524)) (justify right bottom))
   )
@@
     (effects (font (size 1.524 1.524)) (justify right bottom))
   )
-  (label "USB3_P" (at 371.475 140.335 180)
+  (label "USB3_P" (at 371.475 162.56 180)
     (effects (font (size 1.524 1.524)) (justify right bottom))
   )
@@
     (effects (font (size 1.524 1.524)) (justify left bottom))
   )
-  (label "USB4_N" (at 371.475 145.415 180)
+  (label "USB4_N" (at 371.475 153.035 180)
     (effects (font (size 1.524 1.524)) (justify right bottom))
   )
@@
     (effects (font (size 1.524 1.524)) (justify right bottom))
   )
-  (label "FTDI_USB_DN" (at 27.94 93.98 0)
+  (label "FTDI_USB_DN" (at 27.94 86.36 0)
     (effects (font (size 1.524 1.524)) (justify left bottom))
   )
@@
     (effects (font (size 1.524 1.524)) (justify left bottom))
   )
-  (label "USB1_P" (at 371.475 125.095 180)
+  (label "USB1_P" (at 371.475 132.715 180)
     (effects (font (size 1.524 1.524)) (justify right bottom))
   )
@@
     (effects (font (size 1.524 1.524)) (justify left bottom))
   )
-  (label "USB2_N" (at 371.475 130.175 180)
+  (label "USB2_N" (at 371.475 137.795 180)
     (effects (font (size 1.524 1.524)) (justify right bottom))
   )
@@
     (effects (font (size 1.524 1.524)) (justify right bottom))
   )
-  (label "USB2_P" (at 371.475 132.715 180)
+  (label "USB2_P" (at 371.475 140.335 180)
     (effects (font (size 1.524 1.524)) (justify right bottom))
   )
@@
     (effects (font (size 1.524 1.524)) (justify right bottom))
   )
-  (label "USB6_N" (at 33.02 86.36 0)
+  (label "USB7_N" (at 33.02 93.98 0)
     (effects (font (size 1.524 1.524)) (justify left bottom))
   )
@@
     (effects (font (size 1.524 1.524)) (justify left bottom))
   )
-  (label "USB1_N" (at 371.475 122.555 180)
+  (label "USB1_N" (at 371.475 130.175 180)
     (effects (font (size 1.524 1.524)) (justify right bottom))
   )
@@
     (effects (font (size 1.524 1.524)) (justify left bottom))
   )
-  (label "USB5_P" (at 371.475 155.575 180)
+  (label "USB5_P" (at 371.475 147.955 180)
     (effects (font (size 1.524 1.524)) (justify right bottom))
   )
@@
       (effects (font (size 1.524 1.524)) (justify left))
     )
-    (pin "USB6_P" bidirectional (at 351.79 162.56 0)
+    (pin "USB7_P" bidirectional (at 351.79 162.56 0)
       (effects (font (size 1.524 1.524)) (justify right))
     )
-    (pin "USB6_N" bidirectional (at 351.79 160.02 0)
+    (pin "USB7_N" bidirectional (at 351.79 160.02 0)
       (effects (font (size 1.524 1.524)) (justify right))
     )
