File: kicad_hiltop_84hp_backplane/hiltop_backplane_brd.kicad_sch (KiCad schematic)
At the start: 30 parts

Commit message: Layout finished and gerbers exported
Other:
- title: 63HP HILTOP Backplane -> 84HP HILTOP Backplane
Changed lines of the file:
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@@
   (paper "A3")
   (title_block
-    (title "63HP HILTOP Backplane")
-    (date "2021-02-04")
-    (rev "C")
+    (title "84HP HILTOP Backplane")
+    (date "2023-04-06")
+    (rev "A")
     (company "Devtank Ltd")
+    (comment 1 "Part No: 304-020")
   )
   (junction (at 102.235 272.415) (diameter 0) (color 0 0 0 0)
@@
       (reference "D27") (unit 1) (value "LED YEL") (footprint "LED_SMD:LED_0402_1005Metric")
     )
+    (path "/00000000-0000-0000-0000-00005a0778ed/cc27150e-5ad7-4abd-8dc3-ec6b94fa55a5"
+      (reference "DNF1") (unit 1) (value "0R") (footprint "Resistor_SMD:R_0402_1005Metric")
+    )
     (path "/00000000-0000-0000-0000-00005a0778ed/00000000-0000-0000-0000-000060455c00"
       (reference "F1") (unit 1) (value "1206L075") (footprint "Fuse:Fuse_1206_3216Metric")
@@
     )
     (path "/00000000-0000-0000-0000-00005a0778ed/6df3799a-fe1c-4659-871e-5c4af289ab1b"
-      (reference "R18") (unit 1) (value "0R") (footprint "Resistor_SMD:R_0402_1005Metric")
+      (reference "R18") (unit 1) (value "DNF") (footprint "Resistor_SMD:R_0402_1005Metric")
     )
     (path "/00000000-0000-0000-0000-00005a0778ed/01f46a0a-05eb-4ab0-baeb-e9ee53c9f507"
-      (reference "R19") (unit 1) (value "DNF") (footprint "Resistor_SMD:R_0402_1005Metric")
-    )
-    (path "/00000000-0000-0000-0000-00005a0778ed/cc27150e-5ad7-4abd-8dc3-ec6b94fa55a5"
-      (reference "R20") (unit 1) (value "0R") (footprint "Resistor_SMD:R_0402_1005Metric")
+      (reference "R19") (unit 1) (value "0R") (footprint "Resistor_SMD:R_0402_1005Metric")
     )
     (path "/00000000-0000-0000-0000-00005a0778ed/3249e85c-84d0-45cd-8916-8f20fa49b399"
@@
     )
     (path "/00000000-0000-0000-0000-00005a0778ed/51b35572-4799-4b23-8303-70cdac3b2085"
-      (reference "R26") (unit 1) (value "0R") (footprint "Resistor_SMD:R_0402_1005Metric")
+      (reference "R26") (unit 1) (value "DNF") (footprint "Resistor_SMD:R_0402_1005Metric")
     )
     (path "/00000000-0000-0000-0000-00005a0778ed/89c8f2eb-aa54-4bbf-89fc-e49f08b0d288"
-      (reference "R27") (unit 1) (value "DNF") (footprint "Resistor_SMD:R_0402_1005Metric")
+      (reference "R27") (unit 1) (value "0R") (footprint "Resistor_SMD:R_0402_1005Metric")
     )
     (path "/00000000-0000-0000-0000-00005a0778ed/df3e6154-2b4e-4234-8b0b-abcf8ccdf7d2"

Commit message: slots replaced with mounting holes and fiducials added
Parts:
- added F35, F36, F37, F38: Fiducial, Fiducial:Fiducial_1mm_Mask2mm, symbol Devtank:Fiducial
Changed lines of the file:
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@@
   (title_block
     (title "84HP HILTOP Backplane")
-    (date "2023-04-06")
+    (date "2023-04-24")
     (rev "A")
     (company "Devtank Ltd")
@@
     (pin "1")
   )
+  (symbol (lib_id "Devtank:Fiducial") (at 375.285 239.395 0) (unit 1)
+    (in_bom yes) (on_board yes) (fields_autoplaced)
+    (property "Reference" "F35" (id 0) (at 378.7648 238.4188 0)
+      (effects (font (size 1.524 1.524)) (justify left))
+    )
+    (property "Value" "Fiducial" (id 1) (at 378.7648 241.4122 0)
+      (effects (font (size 1.524 1.524)) (justify left))
+    )
+    (property "Footprint" "Fiducial:Fiducial_1mm_Mask2mm" (id 2) (at 375.285 239.395 0)
+      (effects (font (size 1.524 1.524)) hide)
+    )
+    (property "Datasheet" "" (id 3) (at 375.285 239.395 0)
+      (effects (font (size 1.524 1.524)) hide)
+    )
+    (property "Manufacturer" "No part required" (id 4) (at 375.285 239.395 0)
+      (effects (font (size 1.27 1.27)) hide)
+    )
+    (property "Manufacturer Part Number" "No part required" (id 5) (at 375.285 239.395 0)
+      (effects (font (size 1.27 1.27)) hide)
+    )
+  )
   (symbol (lib_id "hiltop_backplane_brd-rescue:TestPoint-Connector-hiltop_backplane_brd-rescue") (at 116.84 123.19 270) (unit 1)
     (in_bom yes) (on_board yes)
@@
     (pin "1")
   )
+  (symbol (lib_id "Devtank:Fiducial") (at 392.43 246.38 0) (unit 1)
+    (in_bom yes) (on_board yes) (fields_autoplaced)
+    (property "Reference" "F38" (id 0) (at 395.9098 245.4038 0)
+      (effects (font (size 1.524 1.524)) (justify left))
+    )
+    (property "Value" "Fiducial" (id 1) (at 395.9098 248.3972 0)
+      (effects (font (size 1.524 1.524)) (justify left))
+    )
+    (property "Footprint" "Fiducial:Fiducial_1mm_Mask2mm" (id 2) (at 392.43 246.38 0)
+      (effects (font (size 1.524 1.524)) hide)
+    )
+    (property "Datasheet" "" (id 3) (at 392.43 246.38 0)
+      (effects (font (size 1.524 1.524)) hide)
+    )
+    (property "Manufacturer" "No part required" (id 4) (at 392.43 246.38 0)
+      (effects (font (size 1.27 1.27)) hide)
+    )
+    (property "Manufacturer Part Number" "No part required" (id 5) (at 392.43 246.38 0)
+      (effects (font (size 1.27 1.27)) hide)
+    )
+  )
+  (symbol (lib_id "Devtank:Fiducial") (at 392.43 239.395 0) (unit 1)
+    (in_bom yes) (on_board yes) (fields_autoplaced)
+    (property "Reference" "F37" (id 0) (at 395.9098 238.4188 0)
+      (effects (font (size 1.524 1.524)) (justify left))
+    )
+    (property "Value" "Fiducial" (id 1) (at 395.9098 241.4122 0)
+      (effects (font (size 1.524 1.524)) (justify left))
+    )
+    (property "Footprint" "Fiducial:Fiducial_1mm_Mask2mm" (id 2) (at 392.43 239.395 0)
+      (effects (font (size 1.524 1.524)) hide)
+    )
+    (property "Datasheet" "" (id 3) (at 392.43 239.395 0)
+      (effects (font (size 1.524 1.524)) hide)
+    )
+    (property "Manufacturer" "No part required" (id 4) (at 392.43 239.395 0)
+      (effects (font (size 1.27 1.27)) hide)
+    )
+    (property "Manufacturer Part Number" "No part required" (id 5) (at 392.43 239.395 0)
+      (effects (font (size 1.27 1.27)) hide)
+    )
+  )
+  (symbol (lib_id "Devtank:Fiducial") (at 375.285 246.38 0) (unit 1)
+    (in_bom yes) (on_board yes) (fields_autoplaced)
+    (property "Reference" "F36" (id 0) (at 378.7648 245.4038 0)
+      (effects (font (size 1.524 1.524)) (justify left))
+    )
+    (property "Value" "Fiducial" (id 1) (at 378.7648 248.3972 0)
+      (effects (font (size 1.524 1.524)) (justify left))
+    )
+    (property "Footprint" "Fiducial:Fiducial_1mm_Mask2mm" (id 2) (at 375.285 246.38 0)
+      (effects (font (size 1.524 1.524)) hide)
+    )
+    (property "Datasheet" "" (id 3) (at 375.285 246.38 0)
+      (effects (font (size 1.524 1.524)) hide)
+    )
+    (property "Manufacturer" "No part required" (id 4) (at 375.285 246.38 0)
+      (effects (font (size 1.27 1.27)) hide)
+    )
+    (property "Manufacturer Part Number" "No part required" (id 5) (at 375.285 246.38 0)
+      (effects (font (size 1.27 1.27)) hide)
+    )
+  )
   (symbol (lib_id "power:+3V3") (at 115.57 271.78 0) (unit 1)
     (in_bom yes) (on_board yes)
@@
       (reference "F34") (unit 1) (value "2920L100PR") (footprint "Fuse:Fuse_2920_7451Metric")
     )
+    (path "/63042929-bfd2-48a4-bff1-0ce0b2d6e6db"
+      (reference "F35") (unit 1) (value "Fiducial") (footprint "Fiducial:Fiducial_1mm_Mask2mm")
+    )
+    (path "/e785e341-7eb1-4378-8548-5a51986d1072"
+      (reference "F36") (unit 1) (value "Fiducial") (footprint "Fiducial:Fiducial_1mm_Mask2mm")
+    )
+    (path "/dd0b2d19-3ee9-4923-9e01-3b6a52b9c7b0"
+      (reference "F37") (unit 1) (value "Fiducial") (footprint "Fiducial:Fiducial_1mm_Mask2mm")
+    )
+    (path "/dd05ada4-2269-4ef7-a044-7cb34264c4d9"
+      (reference "F38") (unit 1) (value "Fiducial") (footprint "Fiducial:Fiducial_1mm_Mask2mm")
+    )
     (path "/00000000-0000-0000-0000-00005a0778ed/910eb48a-2d16-415e-b136-e272f98b6cf7"

Commit message: updated layout with mounting holes and better tracking
Parts:
- removed F36, F37: Fiducial, Fiducial:Fiducial_1mm_Mask2mm, symbol Devtank:Fiducial
Other:
- moved on the sheet: F38
Changed lines of the file:
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@@
   (title_block
     (title "84HP HILTOP Backplane")
-    (date "2023-04-24")
+    (date "2023-05-03")
     (rev "A")
     (company "Devtank Ltd")
@@
     (pin "1")
   )
-  (symbol (lib_id "Devtank:Fiducial") (at 392.43 246.38 0) (unit 1)
-    (in_bom yes) (on_board yes) (fields_autoplaced)
-    (property "Reference" "F38" (id 0) (at 395.9098 245.4038 0)
-      (effects (font (size 1.524 1.524)) (justify left))
-    )
-    (property "Value" "Fiducial" (id 1) (at 395.9098 248.3972 0)
-      (effects (font (size 1.524 1.524)) (justify left))
-    )
-    (property "Footprint" "Fiducial:Fiducial_1mm_Mask2mm" (id 2) (at 392.43 246.38 0)
-      (effects (font (size 1.524 1.524)) hide)
-    )
-    (property "Datasheet" "" (id 3) (at 392.43 246.38 0)
-      (effects (font (size 1.524 1.524)) hide)
-    )
-    (property "Manufacturer" "No part required" (id 4) (at 392.43 246.38 0)
-      (effects (font (size 1.27 1.27)) hide)
-    )
-    (property "Manufacturer Part Number" "No part required" (id 5) (at 392.43 246.38 0)
-      (effects (font (size 1.27 1.27)) hide)
-    )
-  )
   (symbol (lib_id "Devtank:Fiducial") (at 392.43 239.395 0) (unit 1)
     (in_bom yes) (on_board yes) (fields_autoplaced)
-    (property "Reference" "F37" (id 0) (at 395.9098 238.4188 0)
+    (property "Reference" "F38" (id 0) (at 395.9098 238.4188 0)
       (effects (font (size 1.524 1.524)) (justify left))
     )
@@
     )
   )
-  (symbol (lib_id "Devtank:Fiducial") (at 375.285 246.38 0) (unit 1)
-    (in_bom yes) (on_board yes) (fields_autoplaced)
-    (property "Reference" "F36" (id 0) (at 378.7648 245.4038 0)
-      (effects (font (size 1.524 1.524)) (justify left))
-    )
-    (property "Value" "Fiducial" (id 1) (at 378.7648 248.3972 0)
-      (effects (font (size 1.524 1.524)) (justify left))
-    )
-    (property "Footprint" "Fiducial:Fiducial_1mm_Mask2mm" (id 2) (at 375.285 246.38 0)
-      (effects (font (size 1.524 1.524)) hide)
-    )
-    (property "Datasheet" "" (id 3) (at 375.285 246.38 0)
-      (effects (font (size 1.524 1.524)) hide)
-    )
-    (property "Manufacturer" "No part required" (id 4) (at 375.285 246.38 0)
-      (effects (font (size 1.27 1.27)) hide)
-    )
-    (property "Manufacturer Part Number" "No part required" (id 5) (at 375.285 246.38 0)
-      (effects (font (size 1.27 1.27)) hide)
-    )
-  )
   (symbol (lib_id "power:+3V3") (at 115.57 271.78 0) (unit 1)
     (in_bom yes) (on_board yes)
@@
       (reference "F35") (unit 1) (value "Fiducial") (footprint "Fiducial:Fiducial_1mm_Mask2mm")
     )
-    (path "/e785e341-7eb1-4378-8548-5a51986d1072"
-      (reference "F36") (unit 1) (value "Fiducial") (footprint "Fiducial:Fiducial_1mm_Mask2mm")
-    )
-    (path "/dd0b2d19-3ee9-4923-9e01-3b6a52b9c7b0"
-      (reference "F37") (unit 1) (value "Fiducial") (footprint "Fiducial:Fiducial_1mm_Mask2mm")
-    )
     (path "/dd05ada4-2269-4ef7-a044-7cb34264c4d9"
