File: kicad_hiltop_84hp_backplane/MotherBoard_Connector.kicad_sch (KiCad schematic)
At the start: 7 parts, among them J10 PSU3, J7 HILTOP_PCIE-64_CONN, J8 PSU1, J9 PSU2

Commit message: Updated layout with throwdown, added slots and resized board
Parts:
- J10: footprint Connector_Molex:Molex_Mini-Fit_Jr_5566-02A2_2x01_P4.20mm_Vertical -> Devtank_PCB_Lib:Molex_Mini-Fit_Jr_5566-02A_2x01_P4.20mm_Vertical
- J8: footprint Connector_Molex:Molex_Mini-Fit_Jr_5566-08A_2x04_P4.20mm_Vertical -> Devtank_PCB_Lib:Molex_Mini-Fit_Jr_5566-08A_2x04_P4.20mm_Vertical
- J9: footprint Connector_Molex:Molex_Mini-Fit_Jr_5566-04A_2x02_P4.20mm_Vertical -> Devtank_PCB_Lib:Molex_Mini-Fit_Jr_5566-04A_2x02_P4.20mm_Vertical
Changed lines of the file:
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@@
     (property "Reference" "J8" (id 0) (at 214.63 41.275 0))
     (property "Value" "PSU1" (id 1) (at 214.63 53.975 0))
-    (property "Footprint" "Connector_Molex:Molex_Mini-Fit_Jr_5566-08A_2x04_P4.20mm_Vertical" (id 2) (at 213.36 46.355 0)
+    (property "Footprint" "Devtank_PCB_Lib:Molex_Mini-Fit_Jr_5566-08A_2x04_P4.20mm_Vertical" (id 2) (at 213.36 46.355 0)
       (effects (font (size 1.27 1.27)) hide)
     )
@@
     (property "Reference" "J9" (id 0) (at 215.265 66.04 0))
     (property "Value" "PSU2" (id 1) (at 215.265 73.66 0))
-    (property "Footprint" "Connector_Molex:Molex_Mini-Fit_Jr_5566-04A_2x02_P4.20mm_Vertical" (id 2) (at 213.995 68.58 0)
+    (property "Footprint" "Devtank_PCB_Lib:Molex_Mini-Fit_Jr_5566-04A_2x02_P4.20mm_Vertical" (id 2) (at 213.995 68.58 0)
       (effects (font (size 1.27 1.27)) hide)
     )
@@
       (effects (font (size 1.27 1.27)) (justify left))
     )
-    (property "Footprint" "Connector_Molex:Molex_Mini-Fit_Jr_5566-02A2_2x01_P4.20mm_Vertical" (id 2) (at 215.265 86.995 0)
+    (property "Footprint" "Devtank_PCB_Lib:Molex_Mini-Fit_Jr_5566-02A_2x01_P4.20mm_Vertical" (id 2) (at 215.265 86.995 0)
       (effects (font (size 1.27 1.27)) hide)
     )

Commit message: Layout finished and gerbers exported
Other:
- title: 63HP HILTOP Backplane -> 84HP HILTOP Backplane
Changed lines of the file:
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@@
   (paper "A4")
   (title_block
-    (title "63HP HILTOP Backplane")
-    (date "2021-02-04")
-    (rev "C")
+    (title "84HP HILTOP Backplane")
+    (date "2023-04-06")
+    (rev "A")
     (company "Devtank Ltd")
+    (comment 1 "Part No: 304-020")
   )
   (junction (at 118.11 37.465) (diameter 0) (color 0 0 0 0)

Commit message: added measurments to layout
Parts:
- J10: Alternative Manufacturer (none) -> Molex; Alternative Manufacturer Part Number (none) -> 39-28-1023; Manufacturer (none) -> Valcon; Manufacturer Part Number (none) -> 5900-W02ST
- J7: Manufacturer (none) -> No part required; Manufacturer Part Number (none) -> No part required
- J8: Alternative Manufacturer (none) -> Molex; Alternative Manufacturer Part Number (none) -> 39-28-1083; Manufacturer (none) -> Valcon; Manufacturer Part Number (none) -> 5900-W08ST
- J9: Manufacturer (none) -> Valcon; Manufacturer Part Number (none) -> 5900-W04ST
- R45, R46, R47: Tolerance (none) -> 1%
Changed lines of the file:
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@@
+      (effects (font (size 1.27 1.27)) hide)
+    )
+    (property "Manufacturer" "No part required" (id 4) (at 90.805 69.215 0)
+      (effects (font (size 1.27 1.27)) hide)
+    )
+    (property "Manufacturer Part Number" "No part required" (id 5) (at 90.805 69.215 0)
       (effects (font (size 1.27 1.27)) hide)
     )
@@
       (effects (font (size 1.27 1.27)) hide)
     )
+    (property "Manufacturer" "Valcon" (id 5) (at 213.36 46.355 0)
+      (effects (font (size 1.27 1.27)) hide)
+    )
+    (property "Manufacturer Part Number" "5900-W08ST" (id 6) (at 213.36 46.355 0)
+      (effects (font (size 1.27 1.27)) hide)
+    )
+    (property "Alternative Manufacturer" "Molex" (id 7) (at 213.36 46.355 0)
+      (effects (font (size 1.27 1.27)) hide)
+    )
+    (property "Alternative Manufacturer Part Number" "39-28-1083" (id 8) (at 213.36 46.355 0)
+      (effects (font (size 1.27 1.27)) hide)
+    )
     (pin "1")
     (pin "2")
@@
       (effects (font (size 1.27 1.27)) hide)
     )
+    (property "Manufacturer" "Valcon" (id 5) (at 213.995 68.58 0)
+      (effects (font (size 1.27 1.27)) hide)
+    )
+    (property "Manufacturer Part Number" "5900-W04ST" (id 6) (at 213.995 68.58 0)
+      (effects (font (size 1.27 1.27)) hide)
+    )
     (pin "1")
     (pin "2")
@@
     )
     (property "Devtank" "709-002" (id 4) (at 0 173.99 0)
+      (effects (font (size 1.27 1.27)) hide)
+    )
+    (property "Manufacturer" "Valcon" (id 5) (at 215.265 86.995 0)
+      (effects (font (size 1.27 1.27)) hide)
+    )
+    (property "Manufacturer Part Number" "5900-W02ST" (id 6) (at 215.265 86.995 0)
+      (effects (font (size 1.27 1.27)) hide)
+    )
+    (property "Alternative Manufacturer" "Molex" (id 7) (at 215.265 86.995 0)
+      (effects (font (size 1.27 1.27)) hide)
+    )
+    (property "Alternative Manufacturer Part Number" "39-28-1023" (id 8) (at 215.265 86.995 0)
       (effects (font (size 1.27 1.27)) hide)
     )
@@
       (effects (font (size 1.27 1.27)) hide)
     )
+    (property "Tolerance" "1%" (id 5) (at 231.14 68.58 0)
+      (effects (font (size 1.27 1.27)) hide)
+    )
     (pin "1")
     (pin "2")
@@
       (effects (font (size 1.27 1.27)) hide)
     )
+    (property "Tolerance" "1%" (id 5) (at 201.93 68.58 0)
+      (effects (font (size 1.27 1.27)) hide)
+    )
     (pin "1")
     (pin "2")
@@
       (effects (font (size 1.27 1.27)) hide)
     )
+    (property "Tolerance" "1%" (id 5) (at 201.93 71.12 0)
+      (effects (font (size 1.27 1.27)) hide)
+    )
