File: kicad_hiltop_84hp_backplane/MotherBoard_Connector.kicad_sch (KiCad schematic)
At the start: 7 parts, among them J10 PSU3, J7 HILTOP_PCIE-64_CONN, J8 PSU1, J9 PSU2

Commit message: updated bom for 304-020 Rev A
Parts:
- J9: Alternative Manufacturer (none) -> Molex; Alternative Manufacturer Part Number (none) -> 39-28-1043
Changed lines of the file:
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@@
+      (effects (font (size 1.27 1.27)) hide)
+    )
+    (property "Alternative Manufacturer" "Molex" (id 7) (at 213.995 68.58 0)
+      (effects (font (size 1.27 1.27)) hide)
+    )
+    (property "Alternative Manufacturer Part Number" "39-28-1043" (id 8) (at 213.995 68.58 0)
       (effects (font (size 1.27 1.27)) hide)
     )
