File: kicad_hiltop_84hp_backplane/USB_FTDI.kicad_sch (KiCad schematic)
At the start: 43 parts, among them U1 93LCxxC, U2 FT2232H, Y1 ABM10AIG-12.000MHZ-4Z-T3

Commit message: Updated files path on kicad for devtank symbols and footprints
Parts:
- R10, R11, R12, R14, R15, R9: value 0 -> 0R
Changed lines of the file:
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@@
     (in_bom yes) (on_board yes)
     (property "Reference" "R9" (id 0) (at 218.44 102.235 90))
-    (property "Value" "0" (id 1) (at 223.52 103.505 90))
+    (property "Value" "0R" (id 1) (at 223.52 103.505 90))
     (property "Footprint" "Resistor_SMD:R_0402_1005Metric" (id 2) (at 223.52 101.727 90)
       (effects (font (size 1.27 1.27)) hide)
@@
     (in_bom yes) (on_board yes)
     (property "Reference" "R10" (id 0) (at 218.44 104.775 90))
-    (property "Value" "0" (id 1) (at 223.52 106.045 90))
+    (property "Value" "0R" (id 1) (at 223.52 106.045 90))
     (property "Footprint" "Resistor_SMD:R_0402_1005Metric" (id 2) (at 223.52 104.267 90)
       (effects (font (size 1.27 1.27)) hide)
@@
     (in_bom yes) (on_board yes)
     (property "Reference" "R11" (id 0) (at 218.44 107.315 90))
-    (property "Value" "0" (id 1) (at 223.52 108.585 90))
+    (property "Value" "0R" (id 1) (at 223.52 108.585 90))
     (property "Footprint" "Resistor_SMD:R_0402_1005Metric" (id 2) (at 223.52 106.807 90)
       (effects (font (size 1.27 1.27)) hide)
@@
     (in_bom yes) (on_board yes)
     (property "Reference" "R12" (id 0) (at 218.44 109.855 90))
-    (property "Value" "0" (id 1) (at 223.52 111.125 90))
+    (property "Value" "0R" (id 1) (at 223.52 111.125 90))
     (property "Footprint" "Resistor_SMD:R_0402_1005Metric" (id 2) (at 223.52 109.347 90)
       (effects (font (size 1.27 1.27)) hide)
@@
     (in_bom yes) (on_board yes)
     (property "Reference" "R14" (id 0) (at 218.44 117.475 90))
-    (property "Value" "0" (id 1) (at 223.52 118.745 90))
+    (property "Value" "0R" (id 1) (at 223.52 118.745 90))
     (property "Footprint" "Resistor_SMD:R_0402_1005Metric" (id 2) (at 223.52 116.967 90)
       (effects (font (size 1.27 1.27)) hide)
@@
     (in_bom yes) (on_board yes)
     (property "Reference" "R15" (id 0) (at 218.44 120.015 90))
-    (property "Value" "0" (id 1) (at 223.52 121.285 90))
+    (property "Value" "0R" (id 1) (at 223.52 121.285 90))
     (property "Footprint" "Resistor_SMD:R_0402_1005Metric" (id 2) (at 223.52 119.507 90)
       (effects (font (size 1.27 1.27)) hide)

Commit message: Added io tracking on the layout
Parts:
- C6: value 4.7uf -> 4.7uF
- R16, R17: value 330 -> 330R
Changed lines of the file:
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@@
       (effects (font (size 1.27 1.27)) (justify left))
     )
-    (property "Value" "4.7uf" (id 1) (at 141.605 89.535 0)
+    (property "Value" "4.7uF" (id 1) (at 141.605 89.535 0)
       (effects (font (size 1.27 1.27)) (justify left))
     )
@@
     (in_bom yes) (on_board yes)
     (property "Reference" "R16" (id 0) (at 242.57 175.895 90))
-    (property "Value" "330" (id 1) (at 242.57 178.435 90))
+    (property "Value" "330R" (id 1) (at 242.57 178.435 90))
     (property "Footprint" "Resistor_SMD:R_0402_1005Metric" (id 2) (at 242.57 176.657 90)
       (effects (font (size 1.27 1.27)) hide)
@@
     (in_bom yes) (on_board yes)
     (property "Reference" "R17" (id 0) (at 242.57 186.055 90))
-    (property "Value" "330" (id 1) (at 242.57 183.515 90))
+    (property "Value" "330R" (id 1) (at 242.57 183.515 90))
     (property "Footprint" "Resistor_SMD:R_0402_1005Metric" (id 2) (at 242.57 181.737 90)
       (effects (font (size 1.27 1.27)) hide)

Commit message: Layout finished and gerbers exported
Other:
- title: 63HP HILTOP Backplane -> 84HP HILTOP Backplane
Changed lines of the file:
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@@
   (paper "A3")
   (title_block
-    (title "63HP HILTOP Backplane")
-    (date "2021-02-04")
-    (rev "C")
+    (title "84HP HILTOP Backplane")
+    (date "2023-04-06")
+    (rev "A")
     (company "Devtank Ltd")
+    (comment 1 "Part No: 304-020")
   )
   (junction (at 167.005 80.645) (diameter 0) (color 0 0 0 0)

Commit message: added measurments to layout
Parts:
- C10, C11, C12, C13, C14, C15, C16, C17, C18, C19, C2, C3, C4, C5, C6, C7, C9: Characteristics (none) -> X5R; Voltage (none) -> 10V
- C8: Characteristics (none) -> X5R; Voltage (none) -> 6.3V
- D3, D4: Manufacturer (none) -> Rohm Semiconductor; Manufacturer Part Number (none) -> SML-P12VTT86R
- L2, L3, L4, L5: Manufacturer (none) -> muRata; Manufacturer Part Number (none) -> BLM18AG121SN1D; Tolerance (none) -> 1%
- R1, R10, R11, R12, R14, R15, R16, R17, R2, R3, R4, R7, R8, R9: Tolerance (none) -> 1%
- R13: value DNP -> DNF; Tolerance (none) -> 1%
- U1: Manufacturer (none) -> Microchip; Manufacturer Part Number (none) -> 93LC46B-I/SN
- U2: Manufacturer (none) -> FTDI; Manufacturer Part Number (none) -> FT2232HQ-REEL
- Y1: Manufacturer (none) -> Abracon LLC; Manufacturer Part Number (none) -> ABM10AIG-12.000MHZ-4Z-T3
