File: kicad_hiltop_84hp_backplane/backplane_connector.kicad_sch (KiCad schematic)
At the start: 56 parts, among them J1 CONN_DIN_HDR_96POS, J2 CONN_DIN_HDR_96POS, J3 CONN_DIN_HDR_96POS, J4 CONN_DIN_HDR_96POS, J5 CONN_DIN_HDR_96POS, J6 CONN_DIN_HDR_96POS, U3 LTC4311, U4 LTC4311, U6 LM75B, U7 LM75B

Commit message: Layout finished and gerbers exported
Parts:
- R18, R26: value 0R -> DNF
- R19, R27: value DNF -> 0R
- renumbered R20 to DNF1
Other:
- title: 63HP HILTOP Backplane -> 84HP HILTOP Backplane
Changed lines of the file:
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@@
   (paper "A2")
   (title_block
-    (title "63HP HILTOP Backplane")
-    (date "2021-02-04")
-    (rev "C")
+    (title "84HP HILTOP Backplane")
+    (date "2023-04-06")
+    (rev "A")
     (company "Devtank Ltd")
+    (comment 1 "Part No: 304-020")
   )
   (junction (at 320.675 374.65) (diameter 0) (color 0 0 0 0)
@@
   (junction (at 200.025 50.165) (diameter 0) (color 0 0 0 0)
   )
-  (junction (at 351.79 38.1) (diameter 0) (color 0 0 0 0)
-  )
   (junction (at 200.025 40.005) (diameter 0) (color 0 0 0 0)
   )
   (junction (at 200.025 45.085) (diameter 0) (color 0 0 0 0)
   )
+  (junction (at 400.05 33.02) (diameter 0) (color 0 0 0 0)
+  )
   (junction (at 445.135 142.875) (diameter 0) (color 0 0 0 0)
   )
@@
   (junction (at 106.68 156.21) (diameter 0) (color 0 0 0 0)
   )
+  (junction (at 351.79 38.1) (diameter 0) (color 0 0 0 0)
+  )
   (junction (at 445.135 137.795) (diameter 0) (color 0 0 0 0)
   )
@@
   (junction (at 445.135 147.955) (diameter 0) (color 0 0 0 0)
   )
-  (junction (at 400.05 189.23) (diameter 0) (color 0 0 0 0)
-  )
   (junction (at 445.135 29.845) (diameter 0) (color 0 0 0 0)
   )
+  (junction (at 400.05 189.23) (diameter 0) (color 0 0 0 0)
+  )
   (junction (at 445.135 34.925) (diameter 0) (color 0 0 0 0)
   )
@@
   (junction (at 400.05 143.51) (diameter 0) (color 0 0 0 0)
   )
-  (junction (at 400.05 33.02) (diameter 0) (color 0 0 0 0)
-  )
   (junction (at 200.025 137.795) (diameter 0) (color 0 0 0 0)
   )
@@
     (stroke (width 0) (type default) (color 0 0 0 0))
   )
+  (wire (pts (xy 448.945 29.845) (xy 445.135 29.845))
+    (stroke (width 0) (type default) (color 0 0 0 0))
+  )
   (wire (pts (xy 111.125 109.22) (xy 102.87 109.22))
     (stroke (width 0) (type default) (color 0 0 0 0))
@@
     (stroke (width 0) (type default) (color 0 0 0 0))
   )
-  (wire (pts (xy 356.235 30.48) (xy 351.79 30.48))
-    (stroke (width 0) (type default) (color 0 0 0 0))
-  )
   (wire (pts (xy 154.94 292.1) (xy 154.94 307.34))
     (stroke (width 0) (type default) (color 0 0 0 0))
@@
     (stroke (width 0) (type default) (color 0 0 0 0))
   )
+  (wire (pts (xy 400.05 30.48) (xy 400.05 33.02))
+    (stroke (width 0) (type default) (color 0 0 0 0))
+  )
   (wire (pts (xy 102.87 189.23) (xy 111.125 189.23))
     (stroke (width 0) (type default) (color 0 0 0 0))
@@
     (stroke (width 0) (type default) (color 0 0 0 0))
   )
-  (wire (pts (xy 400.05 30.48) (xy 400.05 33.02))
-    (stroke (width 0) (type default) (color 0 0 0 0))
-  )
   (wire (pts (xy 314.325 392.43) (xy 320.675 392.43))
     (stroke (width 0) (type default) (color 0 0 0 0))
@@
     (stroke (width 0) (type default) (color 0 0 0 0))
   )
-  (wire (pts (xy 403.225 30.48) (xy 400.05 30.48))
-    (stroke (width 0) (type default) (color 0 0 0 0))
-  )
   (wire (pts (xy 154.94 140.97) (xy 154.94 143.51))
     (stroke (width 0) (type default) (color 0 0 0 0))
@@
     (stroke (width 0) (type default) (color 0 0 0 0))
   )
-  (wire (pts (xy 448.945 29.845) (xy 445.135 29.845))
-    (stroke (width 0) (type default) (color 0 0 0 0))
-  )
   (wire (pts (xy 102.87 279.4) (xy 111.125 279.4))
     (stroke (width 0) (type default) (color 0 0 0 0))
@@
     (stroke (width 0) (type default) (color 0 0 0 0))
   )
+  (wire (pts (xy 351.79 30.48) (xy 351.79 38.1))
+    (stroke (width 0) (type default) (color 0 0 0 0))
+  )
   (wire (pts (xy 346.71 372.11) (xy 363.22 372.11))
     (stroke (width 0) (type default) (color 0 0 0 0))
@@
     (stroke (width 0) (type default) (color 0 0 0 0))
   )
+  (wire (pts (xy 403.225 30.48) (xy 400.05 30.48))
+    (stroke (width 0) (type default) (color 0 0 0 0))
+  )
   (wire (pts (xy 403.225 254) (xy 394.335 254))
     (stroke (width 0) (type default) (color 0 0 0 0))
@@
     (stroke (width 0) (type default) (color 0 0 0 0))
   )
-  (wire (pts (xy 351.79 30.48) (xy 351.79 38.1))
-    (stroke (width 0) (type default) (color 0 0 0 0))
-  )
   (wire (pts (xy 106.68 38.1) (xy 111.125 38.1))
     (stroke (width 0) (type default) (color 0 0 0 0))
@@
     (stroke (width 0) (type default) (color 0 0 0 0))
   )
+  (wire (pts (xy 356.235 30.48) (xy 351.79 30.48))
+    (stroke (width 0) (type default) (color 0 0 0 0))
+  )
   (wire (pts (xy 448.945 55.245) (xy 445.77 55.245))
     (stroke (width 0) (type default) (color 0 0 0 0))
@@
     (in_bom yes) (on_board yes)
     (property "Reference" "R19" (id 0) (at 238.76 393.065 90))
-    (property "Value" "DNF" (id 1) (at 238.76 382.27 90))
+    (property "Value" "0R" (id 1) (at 238.76 382.27 90))
     (property "Footprint" "Resistor_SMD:R_0402_1005Metric" (id 2) (at 238.252 387.35 90)
       (effects (font (size 1.27 1.27)) hide)
@@
     (in_bom yes) (on_board yes)
     (property "Reference" "R26" (id 0) (at 313.055 374.015 90))
-    (property "Value" "0R" (id 1) (at 313.055 363.855 90))
+    (property "Value" "DNF" (id 1) (at 313.055 363.855 90))
     (property "Footprint" "Resistor_SMD:R_0402_1005Metric" (id 2) (at 312.547 368.3 90)
       (effects (font (size 1.27 1.27)) hide)
@@
     (in_bom yes) (on_board yes)
     (property "Reference" "R18" (id 0) (at 238.76 374.65 90))
-    (property "Value" "0R" (id 1) (at 238.76 364.49 90))
+    (property "Value" "DNF" (id 1) (at 238.76 364.49 90))
     (property "Footprint" "Resistor_SMD:R_0402_1005Metric" (id 2) (at 238.252 368.935 90)
       (effects (font (size 1.27 1.27)) hide)
@@
     (in_bom yes) (on_board yes)
     (property "Reference" "R27" (id 0) (at 313.055 392.43 90))
-    (property "Value" "DNF" (id 1) (at 313.055 381.635 90))
+    (property "Value" "0R" (id 1) (at 313.055 381.635 90))
     (property "Footprint" "Resistor_SMD:R_0402_1005Metric" (id 2) (at 312.547 386.715 90)
       (effects (font (size 1.27 1.27)) hide)
@@
   (symbol (lib_id "Device:R") (at 246.38 368.935 0) (unit 1)
     (in_bom yes) (on_board yes)
-    (property "Reference" "R20" (id 0) (at 245.11 374.65 90))
+    (property "Reference" "DNF1" (id 0) (at 245.11 374.65 90))
     (property "Value" "0R" (id 1) (at 245.11 364.49 90))
     (property "Footprint" "Resistor_SMD:R_0402_1005Metric" (id 2) (at 244.602 368.935 90)

Commit message: added measurments to layout
Parts:
- C1, C20, C21, C55: Characteristics (none) -> X5R; Voltage (none) -> 10V
- F1, F11, F14, F4, F6, F9: Manufacturer (none) -> Littlefuse; Manufacturer Part Number (none) -> 1206L075/13.2WR
- F10, F15, F24, F29, F34, F5: Manufacturer (none) -> Littlefuse; Manufacturer Part Number (none) -> 2920L100PR
- F12, F13, F2, F20, F21, F22, F23, F25, F26, F27, F28, F3, F30, F31, F32, F33, F7, F8: Manufacturer (none) -> Littlefuse; Manufacturer Part Number (none) -> 1206L050/15YR
- J1, J2, J3, J4, J5, J6: Manufacturer (none) -> Valcon; Manufacturer Part Number (none) -> 406AF-96-FSS-AAB4
- R18, R19, R21, R22, R23, R24, R25, R26, R27, R28, R29: Tolerance (none) -> 1%
- R20: renamed from DNF1; Tolerance (none) -> 1%
- U3, U4: Manufacturer (none) -> Linear Technology; Manufacturer Part Number (none) -> LTC4311CDC
