File: kicad_hiltop_84hp_backplane/backplane_connector.kicad_sch (KiCad schematic)
At the start: 56 parts, among them J1 CONN_DIN_HDR_96POS, J2 CONN_DIN_HDR_96POS, J3 CONN_DIN_HDR_96POS, J4 CONN_DIN_HDR_96POS, J5 CONN_DIN_HDR_96POS, J6 CONN_DIN_HDR_96POS, U3 LTC4311, U4 LTC4311, U6 LM75B, U7 LM75B

Commit message: updated bom for 304-020 Rev A
Parts:
- J1, J2, J3, J4, J5, J6: Alternative Manufacturer Part Number (none) -> 3511396AFSS1BNA1
Changed lines of the file:
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@@
       (effects (font (size 1.27 1.27)) hide)
     )
+    (property "Alternative Manufacturer Part Number" "3511396AFSS1BNA1" (id 7) (at 125.095 26.67 0)
+      (effects (font (size 1.27 1.27)) hide)
+    )
     (pin "10a")
     (pin "11a")
@@
       (effects (font (size 1.27 1.27)) hide)
     )
+    (property "Alternative Manufacturer Part Number" "3511396AFSS1BNA1" (id 7) (at 125.095 129.54 0)
+      (effects (font (size 1.27 1.27)) hide)
+    )
     (pin "10a")
     (pin "11a")
@@
       (effects (font (size 1.27 1.27)) hide)
     )
+    (property "Alternative Manufacturer Part Number" "3511396AFSS1BNA1" (id 7) (at 125.095 232.41 0)
+      (effects (font (size 1.27 1.27)) hide)
+    )
     (pin "10a")
     (pin "11a")
@@
       (effects (font (size 1.27 1.27)) hide)
     )
+    (property "Alternative Manufacturer Part Number" "3511396AFSS1BNA1" (id 7) (at 172.085 26.67 0)
+      (effects (font (size 1.27 1.27)) hide)
+    )
     (pin "10a")
     (pin "11a")
@@
       (effects (font (size 1.27 1.27)) hide)
     )
+    (property "Alternative Manufacturer Part Number" "3511396AFSS1BNA1" (id 7) (at 172.085 129.54 0)
+      (effects (font (size 1.27 1.27)) hide)
+    )
     (pin "10a")
     (pin "11a")
@@
       (effects (font (size 1.27 1.27)) hide)
     )
+    (property "Alternative Manufacturer Part Number" "3511396AFSS1BNA1" (id 7) (at 172.085 232.41 0)
+      (effects (font (size 1.27 1.27)) hide)
+    )
     (pin "10a")
     (pin "11a")
@@
       (effects (font (size 1.27 1.27)) hide)
     )
+    (property "Alternative Manufacturer Part Number" "3511396AFSS1BNA1" (id 7) (at 217.805 26.035 0)
+      (effects (font (size 1.27 1.27)) hide)
+    )
     (pin "10a")
     (pin "11a")
@@
       (effects (font (size 1.27 1.27)) hide)
     )
+    (property "Alternative Manufacturer Part Number" "3511396AFSS1BNA1" (id 7) (at 217.805 128.905 0)
+      (effects (font (size 1.27 1.27)) hide)
+    )
     (pin "10a")
     (pin "11a")
@@
       (effects (font (size 1.27 1.27)) hide)
     )
+    (property "Alternative Manufacturer Part Number" "3511396AFSS1BNA1" (id 7) (at 217.805 231.775 0)
+      (effects (font (size 1.27 1.27)) hide)
+    )
     (pin "10a")
     (pin "11a")
@@
       (effects (font (size 1.27 1.27)) hide)
     )
+    (property "Alternative Manufacturer Part Number" "3511396AFSS1BNA1" (id 7) (at 462.915 128.905 0)
+      (effects (font (size 1.27 1.27)) hide)
+    )
     (pin "10a")
     (pin "11a")
@@
       (effects (font (size 1.27 1.27)) hide)
     )
+    (property "Alternative Manufacturer Part Number" "3511396AFSS1BNA1" (id 7) (at 417.195 232.41 0)
+      (effects (font (size 1.27 1.27)) hide)
+    )
     (pin "10a")
     (pin "11a")
@@
       (effects (font (size 1.27 1.27)) hide)
     )
+    (property "Alternative Manufacturer Part Number" "3511396AFSS1BNA1" (id 7) (at 462.915 26.035 0)
+      (effects (font (size 1.27 1.27)) hide)
+    )
     (pin "10a")
     (pin "11a")
@@
       (effects (font (size 1.27 1.27)) hide)
     )
+    (property "Alternative Manufacturer Part Number" "3511396AFSS1BNA1" (id 7) (at 370.205 26.67 0)
+      (effects (font (size 1.27 1.27)) hide)
+    )
     (pin "10a")
     (pin "11a")
@@
       (effects (font (size 1.27 1.27)) hide)
     )
+    (property "Alternative Manufacturer Part Number" "3511396AFSS1BNA1" (id 7) (at 417.195 26.67 0)
+      (effects (font (size 1.27 1.27)) hide)
+    )
     (pin "10a")
     (pin "11a")
@@
       (effects (font (size 1.27 1.27)) hide)
     )
+    (property "Alternative Manufacturer Part Number" "3511396AFSS1BNA1" (id 7) (at 370.205 232.41 0)
+      (effects (font (size 1.27 1.27)) hide)
+    )
     (pin "10a")
     (pin "11a")
@@
       (effects (font (size 1.27 1.27)) hide)
     )
+    (property "Alternative Manufacturer Part Number" "3511396AFSS1BNA1" (id 7) (at 370.205 129.54 0)
+      (effects (font (size 1.27 1.27)) hide)
+    )
     (pin "10a")
     (pin "11a")
@@
       (effects (font (size 1.27 1.27)) hide)
     )
+    (property "Alternative Manufacturer Part Number" "3511396AFSS1BNA1" (id 7) (at 462.915 231.775 0)
+      (effects (font (size 1.27 1.27)) hide)
+    )
     (pin "10a")
     (pin "11a")
@@
       (effects (font (size 1.27 1.27)) hide)
     )
+    (property "Alternative Manufacturer Part Number" "3511396AFSS1BNA1" (id 7) (at 417.195 129.54 0)
+      (effects (font (size 1.27 1.27)) hide)
+    )
